File: analog_pm10_to_3V3.sch (KiCad schematic (older format))
At the start: 7 parts

Commit message: AD7321 integrated
Parts:
- gave numbers to parts that had none: 7
Changed lines of the file:
@@
 $Descr A4 11693 8268
 encoding utf-8
-Sheet 11 12
+Sheet 11 13
 Title ""
 Date ""
@@
 U 1 1 5C02928C
 P 5800 3300
-F 0 "U?" H 5900 3450 50  0000 L CNN
+AR Path="/5C02928C" Ref="U?"  Part="1"
+AR Path="/5C01FF52/5C02928C" Ref="U7"  Part="1"
+F 0 "U7" H 5900 3450 50  0000 L CNN
 F 1 "OPAMP" H 5900 3600 50  0000 L CNN
 F 2 "" H 5800 3300 50  0001 C CNN
@@
 U 1 1 5C029299
 P 5100 3200
-F 0 "R?" V 4895 3200 50  0000 C CNN
+AR Path="/5C029299" Ref="R?"  Part="1"
+AR Path="/5C01FF52/5C029299" Ref="R24"  Part="1"
+F 0 "R24" V 4895 3200 50  0000 C CNN
 F 1 "15K" V 4986 3200 50  0000 C CNN
 F 2 "" H 5100 3200 50  0001 C CNN
@@
 U 1 1 5C0292A0
 P 5950 2800
-F 0 "R?" V 5745 2800 50  0000 C CNN
+AR Path="/5C0292A0" Ref="R?"  Part="1"
+AR Path="/5C01FF52/5C0292A0" Ref="R26"  Part="1"
+F 0 "R26" V 5745 2800 50  0000 C CNN
 F 1 "2K" V 5836 2800 50  0000 C CNN
 F 2 "" H 5950 2800 50  0001 C CNN
@@
 P 5000 3400
 AR Path="/5C0292A7" Ref="R?"  Part="1"
-AR Path="/5C01FF52/5C0292A7" Ref="R?"  Part="1"
-F 0 "R?" V 4800 3400 50  0000 C CNN
+AR Path="/5C01FF52/5C0292A7" Ref="R23"  Part="1"
+F 0 "R23" V 4800 3400 50  0000 C CNN
 F 1 "15K" V 4900 3400 50  0000 C CNN
 F 2 "" H 5000 3400 50  0001 C CNN
@@
 U 1 1 5C0292AE
 P 5250 3800
-F 0 "R?" H 5182 3754 50  0000 R CNN
+AR Path="/5C0292AE" Ref="R?"  Part="1"
+AR Path="/5C01FF52/5C0292AE" Ref="R25"  Part="1"
+F 0 "R25" H 5182 3754 50  0000 R CNN
 F 1 "2K" H 5182 3845 50  0000 R CNN
 F 2 "" H 5250 3800 50  0001 C CNN
@@
 P 5250 3900
 AR Path="/5C0292B5" Ref="#PWR?"  Part="1"
-AR Path="/5C01FF52/5C0292B5" Ref="#PWR?"  Part="1"
-F 0 "#PWR?" H 5250 3650 50  0001 C CNN
+AR Path="/5C01FF52/5C0292B5" Ref="#PWR0116"  Part="1"
+F 0 "#PWR0116" H 5250 3650 50  0001 C CNN
 F 1 "GND" H 5255 3727 50  0000 C CNN
 F 2 "" H 5250 3900 50  0001 C CNN
@@
 P 5550 2500
 AR Path="/5C0292C5" Ref="#PWR?"  Part="1"
-AR Path="/5C01FF52/5C0292C5" Ref="#PWR?"  Part="1"
-F 0 "#PWR?" H 5550 2250 50  0001 C CNN
+AR Path="/5C01FF52/5C0292C5" Ref="#PWR0117"  Part="1"
+F 0 "#PWR0117" H 5550 2250 50  0001 C CNN
 F 1 "GND" H 5555 2327 50  0000 C CNN
 F 2 "" H 5550 2500 50  0001 C CNN
@@
 P 5550 4000
 AR Path="/5C0292CD" Ref="#PWR?"  Part="1"
-AR Path="/5C01FF52/5C0292CD" Ref="#PWR?"  Part="1"
-F 0 "#PWR?" H 5550 3850 50  0001 C CNN
+AR Path="/5C01FF52/5C0292CD" Ref="#PWR0118"  Part="1"
+F 0 "#PWR0118" H 5550 3850 50  0001 C CNN
 F 1 "+3V3" H 5565 4173 50  0000 C CNN
 F 2 "" H 5550 4000 50  0001 C CNN
@@
 U 1 1 5C0292D5
 P 4300 4050
-F 0 "#PWR?" H 4300 3900 50  0001 C CNN
+AR Path="/5C0292D5" Ref="#PWR?"  Part="1"
+AR Path="/5C01FF52/5C0292D5" Ref="#PWR0119"  Part="1"
+F 0 "#PWR0119" H 4300 3900 50  0001 C CNN
 F 1 "+3V3" H 4315 4223 50  0000 C CNN
 F 2 "" H 4300 4050 50  0001 C CNN
@@
 U 1 1 5C0292DB
 P 4300 4650
-F 0 "#PWR?" H 4300 4400 50  0001 C CNN
+AR Path="/5C0292DB" Ref="#PWR?"  Part="1"
+AR Path="/5C01FF52/5C0292DB" Ref="#PWR0120"  Part="1"
+F 0 "#PWR0120" H 4300 4400 50  0001 C CNN
 F 1 "GND" H 4305 4477 50  0000 C CNN
 F 2 "" H 4300 4650 50  0001 C CNN
@@
 U 1 1 5C0292E1
 P 4300 4500
-F 0 "R?" H 4232 4546 50  0000 R CNN
+AR Path="/5C0292E1" Ref="R?"  Part="1"
+AR Path="/5C01FF52/5C0292E1" Ref="R22"  Part="1"
+F 0 "R22" H 4232 4546 50  0000 R CNN
 F 1 "1K" H 4232 4455 50  0000 R CNN
 F 2 "" H 4300 4500 50  0001 C CNN
@@
 U 1 1 5C0292E8
 P 4300 4150
-F 0 "R?" H 4368 4196 50  0000 L CNN
+AR Path="/5C0292E8" Ref="R?"  Part="1"
+AR Path="/5C01FF52/5C0292E8" Ref="R21"  Part="1"
+F 0 "R21" H 4368 4196 50  0000 L CNN
 F 1 "1K" H 4368 4105 50  0000 L CNN
 F 2 "" H 4300 4150 50  0001 C CNN
