File: mech_enc_3V3.sch (KiCad schematic (older format))
At the start: 3 parts

Commit message: added mechanical encoder debouncing schematic
Parts:
- added C?: 1U, symbol Device:C
- added R?: 6.8K, symbol Device:R_US
- added R?: 15K, symbol Device:R_US
Connections:
- net labels added: A, B, C, ~A~, ~B~
- net labels removed: SW+, SW-, ~SW~
- wire segments 13 -> 26
Changed lines of the file:
@@
 $Descr A4 11693 8268
 encoding utf-8
-Sheet 9 9
+Sheet 10 9
 Title ""
 Date ""
@@
 $EndDescr
 Text HLabel 3300 3250 0    50   Input ~ 0
-SW+
+A
 Text HLabel 3300 3350 0    50   Input ~ 0
-SW-
+C
 $Comp
 L Device:R_US R13
@@
 AR Path="/5BF0BEE3/5BEFC0B0" Ref="R?"  Part="1"
 AR Path="/5BF0DB73/5BEFC0B0" Ref="R?"  Part="1"
-AR Path="/5BF1AF42/5BEFC0B0" Ref="R?"  Part="1"
 F 0 "R?" H 3532 2896 50  0000 R CNN
 F 1 "6.8K" H 3532 2805 50  0000 R CNN
@@
 AR Path="/5BF0BEE3/5BEFC134" Ref="R?"  Part="1"
 AR Path="/5BF0DB73/5BEFC134" Ref="R?"  Part="1"
-AR Path="/5BF1AF42/5BEFC134" Ref="R?"  Part="1"
 F 0 "R?" V 3900 3150 50  0000 C CNN
 F 1 "15K" V 3900 3350 50  0000 C CNN
@@
 AR Path="/5BF0BEE3/5BEFC1B8" Ref="C?"  Part="1"
 AR Path="/5BF0DB73/5BEFC1B8" Ref="C?"  Part="1"
-AR Path="/5BF1AF42/5BEFC1B8" Ref="C?"  Part="1"
 F 0 "C?" H 4515 3546 50  0000 L CNN
 F 1 "1U" H 4515 3455 50  0000 L CNN
@@
 Target debounce time is 20ms, which has been empirically shown to be \nsufficiently long for normal switches. \n(http://www.ganssle.com/debouncing-pt2.htm)\n\nWe will solve for 2 conditions, one where the switch is closed, \nand one where it is opened.  \n\nWe the voltage is rising, we want to keep voltage below \nthe minimum CMOS HIGH input voltage (VIH) for 20ms \n(i.e. until debouncing has finished).  \n\nWe want to do the reverse when the voltage is dropping, i.e. keep it above\nVIL.\n\nFor 3V3 CMOS logic, VIH := 2V and VIL := 0.8V
 Text HLabel 4650 3250 2    50   Output ~ 0
-~SW~
+~A~
 Wire Wire Line
 	4400 3250 4650 3250
@@
 Wire Wire Line
 	3300 3750 3600 3750
+Text HLabel 3300 4650 0    50   Input ~ 0
+B
+Text HLabel 3300 4750 0    50   Input ~ 0
+C
+$Comp
+L Device:R_US R?
+U 1 1 5BF0E835
+P 3600 4250
+AR Path="/5BEF83E4/5BF0E835" Ref="R?"  Part="1"
+AR Path="/5BEFB3AE/5BF0E835" Ref="R?"  Part="1"
+AR Path="/5BF0BEE3/5BF0E835" Ref="R?"  Part="1"
+AR Path="/5BF0DB73/5BF0E835" Ref="R?"  Part="1"
+F 0 "R?" H 3532 4296 50  0000 R CNN
+F 1 "6.8K" H 3532 4205 50  0000 R CNN
+F 2 "" V 3640 4240 50  0001 C CNN
+F 3 "~" H 3600 4250 50  0001 C CNN
+	1    3600 4250
+	-1   0    0    -1
+$EndComp
+$Comp
+L Device:R_US R?
+U 1 1 5BF0E83B
+P 4000 4650
+AR Path="/5BEF83E4/5BF0E83B" Ref="R?"  Part="1"
+AR Path="/5BEFB3AE/5BF0E83B" Ref="R?"  Part="1"
+AR Path="/5BF0BEE3/5BF0E83B" Ref="R?"  Part="1"
+AR Path="/5BF0DB73/5BF0E83B" Ref="R?"  Part="1"
+F 0 "R?" V 3900 4550 50  0000 C CNN
+F 1 "15K" V 3900 4750 50  0000 C CNN
+F 2 "" V 4040 4640 50  0001 C CNN
+F 3 "~" H 4000 4650 50  0001 C CNN
+	1    4000 4650
+	0    1    -1   0
+$EndComp
+$Comp
+L Device:C C?
+U 1 1 5BF0E841
+P 4400 4900
+AR Path="/5BEF83E4/5BF0E841" Ref="C?"  Part="1"
+AR Path="/5BEFB3AE/5BF0E841" Ref="C?"  Part="1"
+AR Path="/5BF0BEE3/5BF0E841" Ref="C?"  Part="1"
+AR Path="/5BF0DB73/5BF0E841" Ref="C?"  Part="1"
+F 0 "C?" H 4515 4946 50  0000 L CNN
+F 1 "1U" H 4515 4855 50  0000 L CNN
+F 2 "" H 4438 4750 50  0001 C CNN
+F 3 "~" H 4400 4900 50  0001 C CNN
+	1    4400 4900
+	1    0    0    -1
+$EndComp
+Text HLabel 3300 4000 0    50   Input ~ 0
+3V3
+Wire Wire Line
+	3600 4000 3600 4100
+Text HLabel 3300 5150 0    50   Input ~ 0
+GND
+Wire Wire Line
+	3600 5150 3600 4750
+Wire Wire Line
+	3850 4650 3600 4650
+Connection ~ 3600 4650
+Wire Wire Line
+	4400 4750 4400 4650
+Wire Wire Line
+	4400 4650 4150 4650
+Connection ~ 4400 4650
+Wire Wire Line
+	4400 5050 4400 5150
+Wire Wire Line
+	4400 5150 3600 5150
+Connection ~ 3600 5150
+Text HLabel 4650 4650 2    50   Output ~ 0
+~B~
+Wire Wire Line
+	4400 4650 4650 4650
+Wire Wire Line
+	3600 4400 3600 4650
+Wire Wire Line
+	3300 4650 3600 4650
+Wire Wire Line
+	3300 4750 3600 4750
+Wire Wire Line
+	3300 4000 3600 4000
+Wire Wire Line
+	3300 5150 3600 5150
 $EndSCHEMATC

Commit message: AD7321 integrated
Parts:
- gave numbers to parts that had none: 3
Changed lines of the file:
@@
 $Comp
 L Device:R_US R13
-U 1 1 5BEFC0B0
+U 1 1 5C04B397
 P 3600 2850
-AR Path="/5BEF83E4/5BEFC0B0" Ref="R13"  Part="1"
-AR Path="/5BEFB3AE/5BEFC0B0" Ref="R15"  Part="1"
-AR Path="/5BF0BEE3/5BEFC0B0" Ref="R?"  Part="1"
-AR Path="/5BF0DB73/5BEFC0B0" Ref="R?"  Part="1"
-F 0 "R?" H 3532 2896 50  0000 R CNN
+AR Path="/5BEF83E4/5C04B397" Ref="R13"  Part="1"
+AR Path="/5BEFB3AE/5C04B397" Ref="R15"  Part="1"
+AR Path="/5BF0BEE3/5C04B397" Ref="R?"  Part="1"
+AR Path="/5BF0DB73/5C04B397" Ref="R12"  Part="1"
+F 0 "R12" H 3532 2896 50  0000 R CNN
 F 1 "6.8K" H 3532 2805 50  0000 R CNN
 F 2 "" V 3640 2840 50  0001 C CNN
@@
 $Comp
 L Device:R_US R14
-U 1 1 5BEFC134
+U 1 1 5C04B398
 P 4000 3250
-AR Path="/5BEF83E4/5BEFC134" Ref="R14"  Part="1"
-AR Path="/5BEFB3AE/5BEFC134" Ref="R16"  Part="1"
-AR Path="/5BF0BEE3/5BEFC134" Ref="R?"  Part="1"
-AR Path="/5BF0DB73/5BEFC134" Ref="R?"  Part="1"
-F 0 "R?" V 3900 3150 50  0000 C CNN
+AR Path="/5BEF83E4/5C04B398" Ref="R14"  Part="1"
+AR Path="/5BEFB3AE/5C04B398" Ref="R16"  Part="1"
+AR Path="/5BF0BEE3/5C04B398" Ref="R?"  Part="1"
+AR Path="/5BF0DB73/5C04B398" Ref="R16"  Part="1"
+F 0 "R16" V 3900 3150 50  0000 C CNN
 F 1 "15K" V 3900 3350 50  0000 C CNN
 F 2 "" V 4040 3240 50  0001 C CNN
@@
 $Comp
 L Device:C C3
-U 1 1 5BEFC1B8
+U 1 1 5C04B399
 P 4400 3500
-AR Path="/5BEF83E4/5BEFC1B8" Ref="C3"  Part="1"
-AR Path="/5BEFB3AE/5BEFC1B8" Ref="C4"  Part="1"
-AR Path="/5BF0BEE3/5BEFC1B8" Ref="C?"  Part="1"
-AR Path="/5BF0DB73/5BEFC1B8" Ref="C?"  Part="1"
-F 0 "C?" H 4515 3546 50  0000 L CNN
+AR Path="/5BEF83E4/5C04B399" Ref="C3"  Part="1"
+AR Path="/5BEFB3AE/5C04B399" Ref="C4"  Part="1"
+AR Path="/5BF0BEE3/5C04B399" Ref="C?"  Part="1"
+AR Path="/5BF0DB73/5C04B399" Ref="C2"  Part="1"
+F 0 "C2" H 4515 3546 50  0000 L CNN
 F 1 "1U" H 4515 3455 50  0000 L CNN
 F 2 "" H 4438 3350 50  0001 C CNN
@@
 AR Path="/5BEFB3AE/5BF0E835" Ref="R?"  Part="1"
 AR Path="/5BF0BEE3/5BF0E835" Ref="R?"  Part="1"
-AR Path="/5BF0DB73/5BF0E835" Ref="R?"  Part="1"
-F 0 "R?" H 3532 4296 50  0000 R CNN
+AR Path="/5BF0DB73/5BF0E835" Ref="R15"  Part="1"
+F 0 "R15" H 3532 4296 50  0000 R CNN
 F 1 "6.8K" H 3532 4205 50  0000 R CNN
 F 2 "" V 3640 4240 50  0001 C CNN
@@
 AR Path="/5BEFB3AE/5BF0E83B" Ref="R?"  Part="1"
 AR Path="/5BF0BEE3/5BF0E83B" Ref="R?"  Part="1"
-AR Path="/5BF0DB73/5BF0E83B" Ref="R?"  Part="1"
-F 0 "R?" V 3900 4550 50  0000 C CNN
+AR Path="/5BF0DB73/5BF0E83B" Ref="R17"  Part="1"
+F 0 "R17" V 3900 4550 50  0000 C CNN
 F 1 "15K" V 3900 4750 50  0000 C CNN
 F 2 "" V 4040 4640 50  0001 C CNN
@@
 AR Path="/5BEFB3AE/5BF0E841" Ref="C?"  Part="1"
 AR Path="/5BF0BEE3/5BF0E841" Ref="C?"  Part="1"
-AR Path="/5BF0DB73/5BF0E841" Ref="C?"  Part="1"
-F 0 "C?" H 4515 4946 50  0000 L CNN
+AR Path="/5BF0DB73/5BF0E841" Ref="C4"  Part="1"
+F 0 "C4" H 4515 4946 50  0000 L CNN
 F 1 "1U" H 4515 4855 50  0000 L CNN
 F 2 "" H 4438 4750 50  0001 C CNN

Commit message: reorganized
Parts:
- removed C3, C4: 1U, symbol Device:C
- removed R13, R15: 6.8K, symbol Device:R_US
- removed R14, R17: 15K, symbol Device:R_US
Connections:
- wire segments 26 -> 16
Other:
- note removed: "Substituting Vil and Vih for their respective switching voltages\nand\nLet C = 1uF and t = 20ms\n\nWhen discharging (i.e. switch open -> closed):\nR2 = -t / (C ln(Vil/ Vcc) )\nR2 = 14K use 15K\n\nWhen charging (i.e. switch closed -> opened):\nR1 + R2 = -t / (C ln(1 - Vih/ Vcc) )\nR1 + R2 = 21.5K\nR1 = 21.5K - 15K = 6.5K use 6.8K"
- note removed: "Target debounce time is 20ms, which has been empirically shown to be \nsufficiently long for normal switches. \n(http://www.ganssle.com/debouncing-pt2.htm)\n\nWe will solve for 2 conditions, one where the switch is closed, \nand one where it is opened. \n\nWe the voltage is rising, we want to keep voltage below \nthe minimum CMOS HIGH input voltage (VIH) for 20ms \n(i.e. until debouncing has fini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"
- note removed: "When cap is charging (i.e. switch is open)\nVsw := Vcc * exp(t/RC)\n\nWhen cap is discharging after being fully charged (i.e. switch is closed)\nVsw := Vcc - Vcc * exp(t/RC)\n\nR2 := resistor in discharge\nR1 := additional resistor in charge (i.e. pullup to Vcc)\n\nSo the equations become:\nVsw := 0 + Vcc * exp(t/((R1 + R2)*C)) [charging]\nand\nVsw := Vcc - Vcc * exp(t/(R2*C)) [discharging]"
Changed lines of the file:
@@
 $Descr A4 11693 8268
 encoding utf-8
-Sheet 9 12
+Sheet 9 14
 Title ""
 Date ""
@@
 Comment4 ""
 $EndDescr
-Text HLabel 3300 3250 0    50   Input ~ 0
+Text HLabel 4750 3250 2    50   Output ~ 0
+~B~
+$Sheet
+S 3450 1950 1200 600
+U 5C4840A6
+F0 "A Debounce" 50
+F1 "../subs/debounce_3V3.sch" 50
+F2 "SW+" I L 3450 2200 50
+F3 "SW-" I L 3450 2300 50
+F4 "3V3" I L 3450 2050 50
+F5 "GND" I L 3450 2450 50
+F6 "~SW~" O R 4650 2250 50
+$EndSheet
+Text HLabel 3150 1850 0    50   Input ~ 0
+3V3
+Text HLabel 3150 2200 0    50   Input ~ 0
 A
-Text HLabel 3300 3350 0    50   Input ~ 0
+Text HLabel 3150 2300 0    50   Input ~ 0
 C
-$Comp
-L Device:R_US R13
-U 1 1 5C04B397
-P 3600 2850
-AR Path="/5BEF83E4/5C04B397" Ref="R13"  Part="1"
-AR Path="/5BEFB3AE/5C04B397" Ref="R15"  Part="1"
-AR Path="/5BF0BEE3/5C04B397" Ref="R?"  Part="1"
-AR Path="/5BF0DB73/5C04B397" Ref="R12"  Part="1"
-F 0 "R12" H 3532 2896 50  0000 R CNN
-F 1 "6.8K" H 3532 2805 50  0000 R CNN
-F 2 "" V 3640 2840 50  0001 C CNN
-F 3 "~" H 3600 2850 50  0001 C CNN
-	1    3600 2850
-	-1   0    0    -1
-$EndComp
-$Comp
-L Device:R_US R14
-U 1 1 5C04B398
-P 4000 3250
-AR Path="/5BEF83E4/5C04B398" Ref="R14"  Part="1"
-AR Path="/5BEFB3AE/5C04B398" Ref="R16"  Part="1"
-AR Path="/5BF0BEE3/5C04B398" Ref="R?"  Part="1"
-AR Path="/5BF0DB73/5C04B398" Ref="R16"  Part="1"
-F 0 "R16" V 3900 3150 50  0000 C CNN
-F 1 "15K" V 3900 3350 50  0000 C CNN
-F 2 "" V 4040 3240 50  0001 C CNN
-F 3 "~" H 4000 3250 50  0001 C CNN
-	1    4000 3250
-	0    1    -1   0
-$EndComp
-$Comp
-L Device:C C3
-U 1 1 5C04B399
-P 4400 3500
-AR Path="/5BEF83E4/5C04B399" Ref="C3"  Part="1"
-AR Path="/5BEFB3AE/5C04B399" Ref="C4"  Part="1"
-AR Path="/5BF0BEE3/5C04B399" Ref="C?"  Part="1"
-AR Path="/5BF0DB73/5C04B399" Ref="C2"  Part="1"
-F 0 "C2" H 4515 3546 50  0000 L CNN
-F 1 "1U" H 4515 3455 50  0000 L CNN
-F 2 "" H 4438 3350 50  0001 C CNN
-F 3 "~" H 4400 3500 50  0001 C CNN
-	1    4400 3500
-	1    0    0    -1
-$EndComp
-Text HLabel 3300 2600 0    50   Input ~ 0
-3V3
-Wire Wire Line
-	3600 2600 3600 2700
-Text HLabel 3300 3750 0    50   Input ~ 0
-GND
-Wire Wire Line
-	3600 3750 3600 3350
-Wire Wire Line
-	3850 3250 3600 3250
-Connection ~ 3600 3250
-Wire Wire Line
-	4400 3350 4400 3250
-Wire Wire Line
-	4400 3250 4150 3250
-Connection ~ 4400 3250
-Wire Wire Line
-	4400 3650 4400 3750
-Wire Wire Line
-	4400 3750 3600 3750
-Connection ~ 3600 3750
-Text Notes 5100 2900 0    50   ~ 0
-Target debounce time is 20ms, which has been empirically shown to be \nsufficiently long for normal switches. \n(http://www.ganssle.com/debouncing-pt2.htm)\n\nWe will solve for 2 conditions, one where the switch is closed, \nand one where it is opened.  \n\nWe the voltage is rising, we want to keep voltage below \nthe minimum CMOS HIGH input voltage (VIH) for 20ms \n(i.e. until debouncing has finished).  \n\nWe want to do the reverse when the voltage is dropping, i.e. keep it above\nVIL.\n\nFor 3V3 CMOS logic, VIH := 2V and VIL := 0.8V
-Text HLabel 4650 3250 2    50   Output ~ 0
+Text HLabel 4750 2250 2    50   Output ~ 0
 ~A~
 Wire Wire Line
-	4400 3250 4650 3250
-Text Notes 5100 4300 0    50   ~ 0
-When cap is charging (i.e. switch is open)\nVsw := Vcc * exp(t/RC)\n\nWhen cap is discharging after being fully charged (i.e. switch is closed)\nVsw := Vcc - Vcc * exp(t/RC)\n\nR2 := resistor in discharge\nR1 := additional resistor in charge (i.e. pullup to Vcc)\n\nSo the equations become:\nVsw := 0 + Vcc * exp(t/((R1 + R2)*C)) [charging]\nand\nVsw := Vcc - Vcc * exp(t/(R2*C)) [discharging]
+	4750 2250 4650 2250
+Text HLabel 3150 3700 0    50   Input ~ 0
+GND
+Text HLabel 3150 3200 0    50   Input ~ 0
+B
+Text HLabel 3150 3300 0    50   Input ~ 0
+C
+$Sheet
+S 3450 2950 1200 600
+U 5C485D0D
+F0 "B Debounce" 50
+F1 "../subs/debounce_3V3.sch" 50
+F2 "SW+" I L 3450 3200 50
+F3 "SW-" I L 3450 3300 50
+F4 "3V3" I L 3450 3050 50
+F5 "GND" I L 3450 3450 50
+F6 "~SW~" O R 4650 3250 50
+$EndSheet
 Wire Wire Line
-	3600 3000 3600 3250
-Text Notes 5100 5600 0    50   ~ 0
-Substituting Vil and Vih for their respective switching voltages\nand\nLet C = 1uF and t = 20ms\n\nWhen discharging (i.e. switch open -> closed):\nR2 = -t / (C ln(Vil/ Vcc) )\nR2 = 14K use 15K\n\nWhen charging (i.e. switch closed -> opened):\nR1 + R2 = -t / (C ln(1 - Vih/ Vcc) )\nR1 + R2 = 21.5K\nR1 =  21.5K - 15K = 6.5K use 6.8K
+	4750 3250 4650 3250
 Wire Wire Line
-	3300 3250 3600 3250
+	3150 3700 3350 3700
 Wire Wire Line
-	3300 3350 3600 3350
+	3350 3700 3350 3450
 Wire Wire Line
-	3300 2600 3600 2600
+	3350 3450 3450 3450
 Wire Wire Line
-	3300 3750 3600 3750
-Text HLabel 3300 4650 0    50   Input ~ 0
-B
-Text HLabel 3300 4750 0    50   Input ~ 0
-C
-$Comp
-L Device:R_US R?
-U 1 1 5BF0E835
-P 3600 4250
-AR Path="/5BEF83E4/5BF0E835" Ref="R?"  Part="1"
-AR Path="/5BEFB3AE/5BF0E835" Ref="R?"  Part="1"
-AR Path="/5BF0BEE3/5BF0E835" Ref="R?"  Part="1"
-AR Path="/5BF0DB73/5BF0E835" Ref="R15"  Part="1"
-F 0 "R15" H 3532 4296 50  0000 R CNN
-F 1 "6.8K" H 3532 4205 50  0000 R CNN
-F 2 "" V 3640 4240 50  0001 C CNN
-F 3 "~" H 3600 4250 50  0001 C CNN
-	1    3600 4250
-	-1   0    0    -1
-$EndComp
-$Comp
-L Device:R_US R?
-U 1 1 5BF0E83B
-P 4000 4650
-AR Path="/5BEF83E4/5BF0E83B" Ref="R?"  Part="1"
-AR Path="/5BEFB3AE/5BF0E83B" Ref="R?"  Part="1"
-AR Path="/5BF0BEE3/5BF0E83B" Ref="R?"  Part="1"
-AR Path="/5BF0DB73/5BF0E83B" Ref="R17"  Part="1"
-F 0 "R17" V 3900 4550 50  0000 C CNN
-F 1 "15K" V 3900 4750 50  0000 C CNN
-F 2 "" V 4040 4640 50  0001 C CNN
-F 3 "~" H 4000 4650 50  0001 C CNN
-	1    4000 4650
-	0    1    -1   0
-$EndComp
-$Comp
-L Device:C C?
-U 1 1 5BF0E841
-P 4400 4900
-AR Path="/5BEF83E4/5BF0E841" Ref="C?"  Part="1"
-AR Path="/5BEFB3AE/5BF0E841" Ref="C?"  Part="1"
-AR Path="/5BF0BEE3/5BF0E841" Ref="C?"  Part="1"
-AR Path="/5BF0DB73/5BF0E841" Ref="C4"  Part="1"
-F 0 "C4" H 4515 4946 50  0000 L CNN
-F 1 "1U" H 4515 4855 50  0000 L CNN
-F 2 "" H 4438 4750 50  0001 C CNN
-F 3 "~" H 4400 4900 50  0001 C CNN
-	1    4400 4900
-	1    0    0    -1
-$EndComp
-Text HLabel 3300 4000 0    50   Input ~ 0
-3V3
+	3450 2450 3350 2450
 Wire Wire Line
-	3600 4000 3600 4100
-Text HLabel 3300 5150 0    50   Input ~ 0
-GND
+	3350 2450 3350 3450
+Connection ~ 3350 3450
 Wire Wire Line
-	3600 5150 3600 4750
+	3150 1850 3250 1850
 Wire Wire Line
-	3850 4650 3600 4650
-Connection ~ 3600 4650
+	3250 1850 3250 2050
 Wire Wire Line
-	4400 4750 4400 4650
+	3250 2050 3450 2050
 Wire Wire Line
-	4400 4650 4150 4650
-Connection ~ 4400 4650
+	3250 2050 3250 3050
 Wire Wire Line
-	4400 5050 4400 5150
+	3250 3050 3450 3050
+Connection ~ 3250 2050
 Wire Wire Line
-	4400 5150 3600 5150
-Connection ~ 3600 5150
-Text HLabel 4650 4650 2    50   Output ~ 0
-~B~
+	3150 2200 3450 2200
 Wire Wire Line
-	4400 4650 4650 4650
+	3450 2300 3150 2300
 Wire Wire Line
-	3600 4400 3600 4650
+	3150 3200 3450 3200
 Wire Wire Line
-	3300 4650 3600 4650
-Wire Wire Line
-	3300 4750 3600 4750
-Wire Wire Line
-	3300 4000 3600 4000
-Wire Wire Line
-	3300 5150 3600 5150
+	3450 3300 3150 3300
 $EndSCHEMATC
