File: 5V_to_3V3_divider.sch (KiCad schematic (older format))
At the start: 3 parts

Commit message: added ADS8887 adc
Connections:
- net labels added: SIG_3V3, SIG_5V
- net labels removed: 3V3, 5V
Changed lines of the file:
@@
 $Descr A4 11693 8268
 encoding utf-8
-Sheet 20 24
+Sheet 21 24
 Title ""
 Date ""
@@
 $EndComp
 Text HLabel 6050 2750 0    50   Input ~ 0
-5V
+SIG_5V
 Text HLabel 6050 4050 0    50   Input ~ 0
 GND
 Text HLabel 6300 3200 2    50   Output ~ 0
-3V3
+SIG_3V3
 Wire Wire Line
 	6050 2750 6150 2750
