File: usb_otg_tvs.sch (KiCad schematic (older format))
At the start: 1 part, among them U13 TPD3E001DRLR

Commit message: added ADS8887 adc
Parts:
- removed U13: TPD3E001DRLR, Package_TO_SOT_SMD:SOT-543, symbol Power_Protection:TPD3E001DRLR
- added U10: TPD3E001DRLR, Package_TO_SOT_SMD:SOT-553, symbol william_usb:TPD3E001DRLR
Changed lines of the file:
@@
 $Descr A4 11693 8268
 encoding utf-8
-Sheet 19 24
+Sheet 18 24
 Title ""
 Date ""
@@
 Comment4 ""
 $EndDescr
-$Comp
-L Power_Protection:TPD3E001DRLR U?
-U 1 1 5C7A07F6
-P 5350 3400
-AR Path="/5C6A983A/5C7A07F6" Ref="U?"  Part="1"
-AR Path="/5C6A983A/5C7A05F9/5C7A07F6" Ref="U13"  Part="1"
-F 0 "U13" H 5350 3767 50  0000 C CNN
-F 1 "TPD3E001DRLR" H 5350 3676 50  0000 C CNN
-F 2 "Package_TO_SOT_SMD:SOT-543" H 4650 3100 50  0001 C CNN
-F 3 "http://www.ti.com/lit/ds/symlink/tpd3e001.pdf" H 5150 3650 50  0001 C CNN
-	1    5350 3400
-	1    0    0    -1
-$EndComp
 Text HLabel 5750 3300 2    50   Input ~ 0
 D+
@@
 Text HLabel 5750 3500 2    50   Input ~ 0
 ID
+$Comp
+L william_usb:TPD3E001DRLR U10
+U 1 1 5C8D42B1
+P 5350 3400
+F 0 "U10" H 5350 3767 50  0000 C CNN
+F 1 "TPD3E001DRLR" H 5350 3676 50  0000 C CNN
+F 2 "Package_TO_SOT_SMD:SOT-553" H 4650 3100 50  0001 C CNN
+F 3 "http://www.ti.com/lit/ds/symlink/tpd3e001.pdf" H 5150 3650 50  0001 C CNN
+	1    5350 3400
+	1    0    0    -1
+$EndComp
 $EndSCHEMATC
