File: opto_in_noPD.sch (KiCad schematic (older format))
At the start: 5 parts, among them U6 EL3H7-G

Commit message: added NPN sensor interface, changed tagconnect, added some optoisolated options
Parts:
- removed R12: 10K, Resistor_SMD:R_0603_1608Metric, symbol Device:R
Connections:
- wire segments 23 -> 19
Changed lines of the file:
@@
 $Descr A4 11693 8268
 encoding utf-8
-Sheet 5 18
+Sheet 19 19
 Title ""
 Date ""
@@
 $Comp
 L william_optoisolators:EL3H7-G U?
-U 1 1 5DD57F44
+U 1 1 5BF4DC50
 P 5550 3450
-AR Path="/5DD57F44" Ref="U?"  Part="1"
-AR Path="/5BBAEA3B/5DD57F44" Ref="U?"  Part="1"
-AR Path="/5BBE2F4A/5DD57F44" Ref="U?"  Part="1"
-AR Path="/5BC81FD3/5DD57F44" Ref="U?"  Part="1"
-AR Path="/5BFB4598/5DD57F44" Ref="U?"  Part="1"
-AR Path="/5BEC9D5D/5DD57F44" Ref="U6"  Part="1"
-AR Path="/5BEC9D88/5DD57F44" Ref="U?"  Part="1"
-AR Path="/5BECA926/5DD57F44" Ref="U?"  Part="1"
-AR Path="/5BF2E294/5DD57F44" Ref="U7"  Part="1"
-AR Path="/5D934E77/5DD57F44" Ref="U3"  Part="1"
-AR Path="/5D93BBB8/5DD57F44" Ref="U4"  Part="1"
-AR Path="/5D93C499/5DD57F44" Ref="U5"  Part="1"
-AR Path="/5D93C4A2/5DD57F44" Ref="U6"  Part="1"
-AR Path="/5DC22088/5DD57F44" Ref="U?"  Part="1"
-F 0 "U5" H 5400 3650 50  0000 C CNN
+AR Path="/5BF4DC50" Ref="U?"  Part="1"
+AR Path="/5BBAEA3B/5BF4DC50" Ref="U?"  Part="1"
+AR Path="/5BBE2F4A/5BF4DC50" Ref="U?"  Part="1"
+AR Path="/5BC81FD3/5BF4DC50" Ref="U?"  Part="1"
+AR Path="/5BFB4598/5BF4DC50" Ref="U?"  Part="1"
+AR Path="/5BEC9D5D/5BF4DC50" Ref="U6"  Part="1"
+AR Path="/5BEC9D88/5BF4DC50" Ref="U?"  Part="1"
+AR Path="/5BECA926/5BF4DC50" Ref="U?"  Part="1"
+AR Path="/5BF2E294/5BF4DC50" Ref="U7"  Part="1"
+AR Path="/5D934E77/5BF4DC50" Ref="U3"  Part="1"
+AR Path="/5D93BBB8/5BF4DC50" Ref="U4"  Part="1"
+AR Path="/5D93C499/5BF4DC50" Ref="U5"  Part="1"
+AR Path="/5D93C4A2/5BF4DC50" Ref="U6"  Part="1"
+AR Path="/5DC22088/5BF4DC50" Ref="U?"  Part="1"
+F 0 "U?" H 5400 3650 50  0000 C CNN
 F 1 "EL3H7-G" H 5550 3250 50  0000 C CNN
 F 2 "Package_SO:SOP-4_4.4x2.8mm_P1.27mm" H 5550 3450 50  0001 C CNN
@@
 AR Path="/5D93C4A2/5BBB1F6D" Ref="R11"  Part="1"
 AR Path="/5DC22088/5BBB1F6D" Ref="R?"  Part="1"
-F 0 "R8" V 4254 3650 50  0000 C CNN
+F 0 "R?" V 4254 3650 50  0000 C CNN
 F 1 "4K3" V 4345 3650 50  0000 C CNN
 F 2 "Resistor_SMD:R_0603_1608Metric" H 4450 3650 50  0001 C CNN
@@
 AR Path="/5D93C4A2/5BF4DC51" Ref="R12"  Part="1"
 AR Path="/5DC22088/5BF4DC51" Ref="R?"  Part="1"
-F 0 "R9" H 6059 3796 50  0000 L CNN
+F 0 "R?" H 6059 3796 50  0000 L CNN
 F 1 "10K" H 6059 3705 50  0000 L CNN
 F 2 "Resistor_SMD:R_0603_1608Metric" H 6000 3750 50  0001 C CNN
@@
 Vf := 1.2V (typ)\nImax := 50mA\nIled := 5mA\n\nVin - Vf = Vres\n24V - 1.2V = 22.8V\n\nVres/Iled = Rres\n22.8V/ .005A = 4.6K\n\nWe'll just use 4.3K
 $Comp
-L Device:R R?
-U 1 1 5BBE68CB
-P 4200 3450
-AR Path="/5BBE68CB" Ref="R?"  Part="1"
-AR Path="/5BBAEA3B/5BBE68CB" Ref="R?"  Part="1"
-AR Path="/5BBE2F4A/5BBE68CB" Ref="R?"  Part="1"
-AR Path="/5BC81FD3/5BBE68CB" Ref="R?"  Part="1"
-AR Path="/5BFB4598/5BBE68CB" Ref="R?"  Part="1"
-AR Path="/5BEC9D5D/5BBE68CB" Ref="R12"  Part="1"
-AR Path="/5BEC9D88/5BBE68CB" Ref="R?"  Part="1"
-AR Path="/5BECA926/5BBE68CB" Ref="R?"  Part="1"
-AR Path="/5BF2E294/5BBE68CB" Ref="R23"  Part="1"
-AR Path="/5D934E77/5BBE68CB" Ref="R1"  Part="1"
-AR Path="/5D93BBB8/5BBE68CB" Ref="R4"  Part="1"
-AR Path="/5D93C499/5BBE68CB" Ref="R7"  Part="1"
-AR Path="/5D93C4A2/5BBE68CB" Ref="R10"  Part="1"
-AR Path="/5DC22088/5BBE68CB" Ref="R?"  Part="1"
-F 0 "R7" H 4141 3496 50  0000 R CNN
-F 1 "10K" H 4141 3405 50  0000 R CNN
-F 2 "Resistor_SMD:R_0603_1608Metric" H 4200 3450 50  0001 C CNN
-F 3 "~" H 4200 3450 50  0001 C CNN
-	1    4200 3450
-	1    0    0    -1
-$EndComp
-Wire Wire Line
-	4150 3650 4200 3650
-$Comp
 L william_diodes:BAS21LT1G D?
 U 1 1 5BBEB592
@@
 AR Path="/5D93C4A2/5BBEB592" Ref="D4"  Part="1"
 AR Path="/5DC22088/5BBEB592" Ref="D?"  Part="1"
-F 0 "D3" V 4704 3529 50  0000 L CNN
+F 0 "D?" V 4704 3529 50  0000 L CNN
 F 1 "BAS21LT1G" V 4795 3529 50  0000 L CNN
 F 2 "Package_TO_SOT_SMD:SOT-23" H 4700 3600 50  0001 C CNN
@@
 	4200 2850 4200 3150
 Wire Wire Line
-	4200 3600 4200 3650
-Connection ~ 4200 3650
-Wire Wire Line
-	4200 3650 4300 3650
-Wire Wire Line
 	5850 3350 6350 3350
 Wire Wire Line
@@
 	6000 3550 6350 3550
 Wire Wire Line
-	4150 3250 4200 3250
-Wire Wire Line
-	4200 3300 4200 3250
-Connection ~ 4200 3250
-Wire Wire Line
 	4750 3250 4750 3300
-Wire Wire Line
-	4200 3250 4750 3250
 Wire Wire Line
 	4750 3250 5000 3250
@@
 Wire Wire Line
 	5000 3250 5000 3350
+Wire Wire Line
+	4150 3250 4750 3250
+Wire Wire Line
+	4150 3650 4300 3650
 $EndSCHEMATC
