File: Nfet_PWR_noPD.sch (KiCad schematic (older format))
At the start: 3 parts, among them Q11 IRF7458TRPBF

Commit message: modified opto-isolated NFET schematic - needed PU resistor
Parts:
- removed R5: 10K, Resistor_SMD:R_0603_1608Metric, symbol Device:R
Connections:
- wire segments 13 -> 9
Changed lines of the file:
@@
 $Descr A4 11693 8268
 encoding utf-8
-Sheet 9 18
+Sheet 10 18
 Title ""
 Date ""
@@
 Wire Wire Line
 	6250 3850 6250 3650
-Wire Wire Line
-	5250 3450 5450 3450
-Wire Wire Line
-	5250 3850 5450 3850
-Wire Wire Line
-	5450 3500 5450 3450
-Connection ~ 5450 3450
-Wire Wire Line
-	5450 3450 5600 3450
-Wire Wire Line
-	5450 3800 5450 3850
-Connection ~ 5450 3850
-Wire Wire Line
-	5450 3850 6250 3850
 Text HLabel 6450 3050 2    50   Input ~ 0
 LOAD-
@@
 $EndComp
 $Comp
-L Device:R R5
-U 1 1 5BE5AA7F
-P 5450 3650
-AR Path="/5BE5A530/5BE5AA7F" Ref="R5"  Part="1"
-AR Path="/5BE5D36F/5BE5AA7F" Ref="R7"  Part="1"
-AR Path="/5BE5D37A/5BE5AA7F" Ref="R9"  Part="1"
-AR Path="/5BE5D381/5BE5AA7F" Ref="R?"  Part="1"
-AR Path="/5C3B8390/5BE5AA7F" Ref="R?"  Part="1"
-AR Path="/5C3C14B8/5BE5AA7F" Ref="R?"  Part="1"
-AR Path="/5C4D1AE2/5BE5AA7F" Ref="R?"  Part="1"
-AR Path="/5C4E4A9C/5BE5AA7F" Ref="R1"  Part="1"
-AR Path="/5C4EE84B/5BE5AA7F" Ref="R27"  Part="1"
-AR Path="/5D986736/5BE5AA7F" Ref="R?"  Part="1"
-AR Path="/5D98C5E1/5BE5AA7F" Ref="R?"  Part="1"
-AR Path="/5DD45A74/5DD45DBE/5BE5AA7F" Ref="R49"  Part="1"
-F 0 "R49" H 5520 3696 50  0000 L CNN
-F 1 "10K" H 5520 3605 50  0000 L CNN
-F 2 "Resistor_SMD:R_0603_1608Metric" V 5380 3650 50  0001 C CNN
-F 3 "~" H 5450 3650 50  0001 C CNN
-	1    5450 3650
-	1    0    0    -1
-$EndComp
-$Comp
 L william_fets:IRF7458TRPBF Q11
 U 1 1 5DD46952
@@
 	1    0    0    -1
 $EndComp
+Wire Wire Line
+	5250 3450 5600 3450
+Wire Wire Line
+	5250 3850 6250 3850
 $EndSCHEMATC

Commit message: CORRECTED NPN & PNP optoisolated schematics, added some others (apparently)
Parts:
- Q11: footprint Package_SO:SO-8_3.9x4.9mm_P1.27mm -> william_mosfet:SO-8_3.9x4.9mm_P1.27mm
Changed lines of the file:
@@
 EESchema Schematic File Version 4
-LIBS:main-cache
 EELAYER 30 0
 EELAYER END
 $Descr A4 11693 8268
 encoding utf-8
-Sheet 10 18
+Sheet 9 19
 Title ""
 Date ""
@@
 F 0 "Q11" H 6356 3496 50  0000 L CNN
 F 1 "IRF7458TRPBF" H 6356 3405 50  0000 L CNN
-F 2 "Package_SO:SO-8_3.9x4.9mm_P1.27mm" H 6000 3650 50  0001 C CNN
+F 2 "william_mosfet:SO-8_3.9x4.9mm_P1.27mm" H 6000 3650 50  0001 C CNN
 F 3 "https://www.infineon.com/dgdl/irf7458pbf.pdf?fileId=5546d462533600a4015355fecb231bfe" H 6150 3450 50  0001 C CNN
 	1    6150 3450
