File: stm32f373cctx.sch (KiCad schematic (older format))
At the start: 12 parts, among them J18 SWD, U2 STM32F373CCTx

Commit message: added stm32f373 and fixed optoisolated output
Parts:
- removed J18: SWD, Connector_PinHeader_2.54mm:PinHeader_1x06_P2.54mm_Vertical, symbol Connector_Generic:Conn_01x06
- added J18: TC2030-IDC, Connector:Tag-Connect_TC2030-IDC-FP_2x03_P1.27mm_Vertical, symbol william_connectors:TC2030-IDC
Connections:
- no-connect marks 13 -> 17
Changed lines of the file:
@@
 	1    0    0    -1
 $EndComp
-$Comp
-L Connector_Generic:Conn_01x06 J18
-U 1 1 5D8E98BD
-P 1100 1850
-F 0 "J18" H 1018 2267 50  0000 C CNN
-F 1 "SWD" H 1018 2176 50  0000 C CNN
-F 2 "Connector_PinHeader_2.54mm:PinHeader_1x06_P2.54mm_Vertical" H 1100 1850 50  0001 C CNN
-F 3 "~" H 1100 1850 50  0001 C CNN
-	1    1100 1850
-	-1   0    0    -1
-$EndComp
-Text Label 1600 1650 0    50   ~ 0
+Text Label 1900 1600 0    50   ~ 0
 VCC
-Text Label 1600 1750 0    50   ~ 0
+Text Label 1900 1900 0    50   ~ 0
 SWCLK
-Text Label 1600 1850 0    50   ~ 0
+Text Label 1900 2000 0    50   ~ 0
 GND
-Text Label 1600 1950 0    50   ~ 0
+Text Label 1900 1700 0    50   ~ 0
 SWDIO
-Text Label 1600 2050 0    50   ~ 0
+Text Label 1900 1800 0    50   ~ 0
 ~RST
-Text Label 1600 2150 0    50   ~ 0
+Text Label 1900 2100 0    50   ~ 0
 SWO
 Wire Wire Line
-	1600 1650 1300 1650
-Wire Wire Line
-	1300 1750 1600 1750
-Wire Wire Line
-	1300 1850 1600 1850
-Wire Wire Line
-	1600 1950 1300 1950
-Wire Wire Line
-	1300 2050 1600 2050
-Wire Wire Line
-	1600 2150 1300 2150
+	1900 1600 1600 1600
+Wire Wire Line
+	1600 1900 1900 1900
+Wire Wire Line
+	1600 2000 1900 2000
+Wire Wire Line
+	1900 1700 1600 1700
+Wire Wire Line
+	1600 1800 1900 1800
+Wire Wire Line
+	1900 2100 1600 2100
 Text Label 6800 3900 0    50   ~ 0
 SWCLK
@@
 Text HLabel 6800 3000 2    50   Input ~ 0
 START_L
+NoConn ~ 6800 2900
+NoConn ~ 6800 4800
+NoConn ~ 6800 5000
+NoConn ~ 6800 5100
+$Comp
+L william_connectors:TC2030-IDC J18
+U 1 1 5D9984C0
+P 1300 1850
+F 0 "J18" H 1293 2448 50  0000 C CNN
+F 1 "TC2030-IDC" H 1293 2357 50  0000 C CNN
+F 2 "Connector:Tag-Connect_TC2030-IDC-FP_2x03_P1.27mm_Vertical" H 1150 1950 50  0001 C CNN
+F 3 "http://www.tag-connect.com/Materials/TC2030-IDC.pdf" H 1150 1950 50  0001 C CNN
+	1    1300 1850
+	-1   0    0    -1
+$EndComp
 $EndSCHEMATC

Commit message: removing backup files
Parts:
- J18: footprint Connector:Tag-Connect_TC2030-IDC-FP_2x03_P1.27mm_Vertical -> Connector:Tag-Connect_TC2030-IDC-NL_2x03_P1.27mm_Vertical
Changed lines of the file:
@@
 F 0 "J18" H 1293 2448 50  0000 C CNN
 F 1 "TC2030-IDC" H 1293 2357 50  0000 C CNN
-F 2 "Connector:Tag-Connect_TC2030-IDC-FP_2x03_P1.27mm_Vertical" H 1150 1950 50  0001 C CNN
+F 2 "Connector:Tag-Connect_TC2030-IDC-NL_2x03_P1.27mm_Vertical" H 1150 1950 50  0001 C CNN
 F 3 "http://www.tag-connect.com/Materials/TC2030-IDC.pdf" H 1150 1950 50  0001 C CNN
 	1    1300 1850

Commit message: fixed opto out schematic (updated footprints), added new fet schematics
Connections:
- net labels added: CLUTCH_ON, MTR_ON
- no-connect marks 17 -> 15
Changed lines of the file:
@@
 $Descr A4 11693 8268
 encoding utf-8
-Sheet 2 14
+Sheet 2 18
 Title ""
 Date ""
@@
 NoConn ~ 6800 5300
 NoConn ~ 6800 5200
-NoConn ~ 6800 4900
 NoConn ~ 6800 4400
 NoConn ~ 6800 4000
@@
 START_L
 NoConn ~ 6800 2900
-NoConn ~ 6800 4800
 NoConn ~ 6800 5000
 NoConn ~ 6800 5100
@@
 	-1   0    0    -1
 $EndComp
+Text HLabel 6800 4800 2    50   Output ~ 0
+MTR_ON
+Text HLabel 6800 4900 2    50   Output ~ 0
+CLUTCH_ON
 $EndSCHEMATC

Commit message: modified opto-isolated NFET schematic - needed PU resistor
Connections:
- net labels added: ADJUST
- no-connect marks 15 -> 14
Changed lines of the file:
@@
 Text Label 3500 3050 0    50   ~ 0
 VSS
+Text HLabel 6800 3700 2    50   Output ~ 0
+LED_ERR
 Text HLabel 6800 3600 2    50   Output ~ 0
-LED_ERR
-Text HLabel 6800 3700 2    50   Output ~ 0
 LED_RDY
 Text HLabel 4600 5300 0    50   Output ~ 0
@@
 Text HLabel 6800 3100 2    50   Input ~ 0
 MISC_IN_1
-NoConn ~ 4600 4300
 NoConn ~ 4600 4400
 NoConn ~ 4600 4600
@@
 NoConn ~ 6800 5200
 NoConn ~ 6800 4400
-NoConn ~ 6800 4000
 NoConn ~ 6800 3300
-NoConn ~ 6800 2600
 Text Label 900  7550 0    50   ~ 0
 VREFSD
@@
 Text HLabel 6800 3000 2    50   Input ~ 0
 START_L
-NoConn ~ 6800 2900
 NoConn ~ 6800 5000
 NoConn ~ 6800 5100
@@
 	-1   0    0    -1
 $EndComp
-Text HLabel 6800 4800 2    50   Output ~ 0
+Text HLabel 6800 2900 2    50   Output ~ 0
 MTR_ON
-Text HLabel 6800 4900 2    50   Output ~ 0
+Text HLabel 4600 4300 0    50   Output ~ 0
 CLUTCH_ON
+NoConn ~ 6800 4800
+NoConn ~ 6800 4900
+Text HLabel 6800 2600 2    50   Input ~ 0
+ADJUST
+NoConn ~ 6800 4000
 $EndSCHEMATC

Commit message: added NPN sensor interface, changed tagconnect, added some optoisolated options
Parts:
- J18: footprint Connector:Tag-Connect_TC2030-IDC-NL_2x03_P1.27mm_Vertical -> Connector:Tag-Connect_TC2030-IDC-FP_2x03_P1.27mm_Vertical
Changed lines of the file:
@@
 F 0 "J18" H 1293 2448 50  0000 C CNN
 F 1 "TC2030-IDC" H 1293 2357 50  0000 C CNN
-F 2 "Connector:Tag-Connect_TC2030-IDC-NL_2x03_P1.27mm_Vertical" H 1150 1950 50  0001 C CNN
+F 2 "Connector:Tag-Connect_TC2030-IDC-FP_2x03_P1.27mm_Vertical" H 1150 1950 50  0001 C CNN
 F 3 "http://www.tag-connect.com/Materials/TC2030-IDC.pdf" H 1150 1950 50  0001 C CNN
 	1    1300 1850
