File: MAX11270.sch (KiCad schematic (older format))
At the start: 7 parts, among them U5 MAX11270

Commit message: updated max11270
Parts:
- C?: renamed from C8; symbol device:C -> Device:C
- C?: renamed from C9; symbol device:C -> Device:C
- C?: renamed from C6; symbol device:C -> Device:C
- C?: renamed from C7; symbol device:C -> Device:C
- C?: renamed from C11; symbol device:C -> Device:C
- C?: renamed from C10; symbol device:C -> Device:C
- renumbered U5 to U?
Connections:
- wire segments 44 -> 40
Changed lines of the file:
@@
 EESchema Schematic File Version 4
-LIBS:strain_gauge_485-cache
+LIBS:main-cache
 EELAYER 26 0
 EELAYER END
 $Descr A4 11693 8268
 encoding utf-8
-Sheet 3 4
+Sheet 11 11
 Title ""
 Date ""
@@
 $EndDescr
 $Comp
-L william:MAX11270 U5
+L william:MAX11270 U?
 U 1 1 5B2E54B9
 P 5850 3750
-F 0 "U5" H 5300 4550 50  0000 C CNN
+F 0 "U?" H 5300 4550 50  0000 C CNN
 F 1 "MAX11270" H 6250 4550 50  0000 C CNN
 F 2 "Housings_SSOP:TSSOP-24_4.4x7.8mm_Pitch0.65mm" H 5700 3800 50  0001 C CNN
@@
 $EndComp
 $Comp
-L device:C C8
+L Device:C C?
 U 1 1 5B2E54C5
 P 5550 2600
-F 0 "C8" H 5350 2650 50  0000 L CNN
+F 0 "C?" H 5350 2650 50  0000 L CNN
 F 1 "1U" H 5350 2550 50  0000 L CNN
 F 2 "Capacitors_SMD:C_0402" H 5588 2450 50  0001 C CNN
@@
 $EndComp
 $Comp
-L device:C C9
+L Device:C C?
 U 1 1 5B2E54CC
 P 6150 2600
-F 0 "C9" H 6265 2646 50  0000 L CNN
+F 0 "C?" H 6265 2646 50  0000 L CNN
 F 1 "1U" H 6265 2555 50  0000 L CNN
 F 2 "Capacitors_SMD:C_0402" H 6188 2450 50  0001 C CNN
@@
 	5950 2400 6150 2400
 $Comp
-L device:C C6
+L Device:C C?
 U 1 1 5B2E6585
 P 4650 3100
-F 0 "C6" H 4450 3150 50  0000 L CNN
+F 0 "C?" H 4450 3150 50  0000 L CNN
 F 1 "10N" H 4400 3050 50  0000 L CNN
 F 2 "Capacitors_SMD:C_0402" H 4688 2950 50  0001 C CNN
@@
 $EndComp
 $Comp
-L device:C C7
+L Device:C C?
 U 1 1 5B2E66DA
 P 4650 3550
-F 0 "C7" H 4450 3600 50  0000 L CNN
+F 0 "C?" H 4450 3600 50  0000 L CNN
 F 1 "10N" H 4400 3500 50  0000 L CNN
 F 2 "Capacitors_SMD:C_0402" H 4688 3400 50  0001 C CNN
@@
 $EndComp
 Wire Wire Line
-	4650 3700 4850 3700
-Wire Wire Line
 	4850 3500 5150 3500
 Wire Wire Line
@@
 Wire Wire Line
 	4850 3150 4850 2950
-Wire Wire Line
-	4850 2950 4650 2950
-Wire Wire Line
-	4650 3250 5150 3250
 Wire Wire Line
 	4850 3500 4850 3700
@@
 Text HLabel 4350 3250 0    50   Input ~ 0
 AIN-
-Wire Wire Line
-	4350 3250 4650 3250
-Connection ~ 4650 3250
-Wire Wire Line
-	4350 2950 4650 2950
-Connection ~ 4650 2950
-$Comp
-L device:C C11
+$Comp
+L Device:C C?
 U 1 1 5B2E9EF3
 P 6900 4050
-F 0 "C11" H 6650 4100 50  0000 L CNN
+F 0 "C?" H 6650 4100 50  0000 L CNN
 F 1 "10N" H 6650 4000 50  0000 L CNN
 F 2 "Capacitors_SMD:C_0402" H 6938 3900 50  0001 C CNN
@@
 	6600 4000 6550 4000
 $Comp
-L device:C C10
+L Device:C C?
 U 1 1 5B2EAA13
 P 6900 4450
-F 0 "C10" H 6650 4500 50  0000 L CNN
+F 0 "C?" H 6650 4500 50  0000 L CNN
 F 1 "10U" H 6650 4400 50  0000 L CNN
 F 2 "Capacitors_SMD:C_0805" H 6938 4300 50  0001 C CNN
@@
 Text HLabel 4350 3400 0    50   Input ~ 0
 3V3
-Wire Wire Line
-	4350 3400 4650 3400
-Connection ~ 4650 3400
 Text Label 4350 3700 2    50   ~ 0
 AGND
 Wire Wire Line
-	4350 3700 4650 3700
-Connection ~ 4650 3700
-Wire Wire Line
-	4650 3400 5150 3400
-Wire Wire Line
 	6900 4300 6900 4250
 Wire Wire Line
@@
 Wire Wire Line
 	6600 4100 6550 4100
+Wire Wire Line
+	4350 3700 4850 3700
+Wire Wire Line
+	4350 2950 4850 2950
+Wire Wire Line
+	4350 3250 5150 3250
+Wire Wire Line
+	4350 3400 5150 3400
 $EndSCHEMATC

Commit message: AD7321 integrated
Parts:
- gave numbers to parts that had none: 7
Changed lines of the file:
@@
 $Descr A4 11693 8268
 encoding utf-8
-Sheet 11 11
+Sheet 13 14
 Title ""
 Date ""
@@
 $EndDescr
 $Comp
-L william:MAX11270 U?
+L william:MAX11270 U9
 U 1 1 5B2E54B9
 P 5850 3750
-F 0 "U?" H 5300 4550 50  0000 C CNN
+F 0 "U9" H 5300 4550 50  0000 C CNN
 F 1 "MAX11270" H 6250 4550 50  0000 C CNN
 F 2 "Housings_SSOP:TSSOP-24_4.4x7.8mm_Pitch0.65mm" H 5700 3800 50  0001 C CNN
@@
 $EndComp
 $Comp
-L Device:C C?
+L Device:C C17
 U 1 1 5B2E54C5
 P 5550 2600
-F 0 "C?" H 5350 2650 50  0000 L CNN
+F 0 "C17" H 5350 2650 50  0000 L CNN
 F 1 "1U" H 5350 2550 50  0000 L CNN
 F 2 "Capacitors_SMD:C_0402" H 5588 2450 50  0001 C CNN
@@
 $EndComp
 $Comp
-L Device:C C?
+L Device:C C18
 U 1 1 5B2E54CC
 P 6150 2600
-F 0 "C?" H 6265 2646 50  0000 L CNN
+F 0 "C18" H 6265 2646 50  0000 L CNN
 F 1 "1U" H 6265 2555 50  0000 L CNN
 F 2 "Capacitors_SMD:C_0402" H 6188 2450 50  0001 C CNN
@@
 	5950 2400 6150 2400
 $Comp
-L Device:C C?
+L Device:C C15
 U 1 1 5B2E6585
 P 4650 3100
-F 0 "C?" H 4450 3150 50  0000 L CNN
+F 0 "C15" H 4450 3150 50  0000 L CNN
 F 1 "10N" H 4400 3050 50  0000 L CNN
 F 2 "Capacitors_SMD:C_0402" H 4688 2950 50  0001 C CNN
@@
 $EndComp
 $Comp
-L Device:C C?
+L Device:C C16
 U 1 1 5B2E66DA
 P 4650 3550
-F 0 "C?" H 4450 3600 50  0000 L CNN
+F 0 "C16" H 4450 3600 50  0000 L CNN
 F 1 "10N" H 4400 3500 50  0000 L CNN
 F 2 "Capacitors_SMD:C_0402" H 4688 3400 50  0001 C CNN
@@
 AIN-
 $Comp
-L Device:C C?
+L Device:C C19
 U 1 1 5B2E9EF3
 P 6900 4050
-F 0 "C?" H 6650 4100 50  0000 L CNN
+F 0 "C19" H 6650 4100 50  0000 L CNN
 F 1 "10N" H 6650 4000 50  0000 L CNN
 F 2 "Capacitors_SMD:C_0402" H 6938 3900 50  0001 C CNN
@@
 	6600 4000 6550 4000
 $Comp
-L Device:C C?
+L Device:C C20
 U 1 1 5B2EAA13
 P 6900 4450
-F 0 "C?" H 6650 4500 50  0000 L CNN
+F 0 "C20" H 6650 4500 50  0000 L CNN
 F 1 "10U" H 6650 4400 50  0000 L CNN
 F 2 "Capacitors_SMD:C_0805" H 6938 4300 50  0001 C CNN

Commit message: add DHT22 & MAX11254 schematics
Parts:
- added NT1, NT2: Net-Tie_2, symbol Device:Net-Tie_2
- renumbered C15 to C18, C16 to C20, C17 to C21, C18 to C22, C19 to C23, C20 to C24, U9 to U3
Connections:
- net labels added: VCC
- net labels removed: 3V3
- wire segments 40 -> 35
Changed lines of the file:
@@
 $Descr A4 11693 8268
 encoding utf-8
-Sheet 13 14
+Sheet 5 8
 Title ""
 Date ""
@@
 $EndDescr
 $Comp
-L william:MAX11270 U9
+L william:MAX11270 U3
 U 1 1 5B2E54B9
 P 5850 3750
-F 0 "U9" H 5300 4550 50  0000 C CNN
+F 0 "U3" H 5300 4550 50  0000 C CNN
 F 1 "MAX11270" H 6250 4550 50  0000 C CNN
 F 2 "Housings_SSOP:TSSOP-24_4.4x7.8mm_Pitch0.65mm" H 5700 3800 50  0001 C CNN
@@
 $EndComp
 $Comp
-L Device:C C17
+L Device:C C21
 U 1 1 5B2E54C5
 P 5550 2600
-F 0 "C17" H 5350 2650 50  0000 L CNN
+F 0 "C21" H 5350 2650 50  0000 L CNN
 F 1 "1U" H 5350 2550 50  0000 L CNN
 F 2 "Capacitors_SMD:C_0402" H 5588 2450 50  0001 C CNN
@@
 $EndComp
 $Comp
-L Device:C C18
+L Device:C C22
 U 1 1 5B2E54CC
 P 6150 2600
-F 0 "C18" H 6265 2646 50  0000 L CNN
+F 0 "C22" H 6265 2646 50  0000 L CNN
 F 1 "1U" H 6265 2555 50  0000 L CNN
 F 2 "Capacitors_SMD:C_0402" H 6188 2450 50  0001 C CNN
@@
 Text HLabel 6550 3750 2    50   Output ~ 0
 ~DATA_READY~
-Text HLabel 5750 2200 0    50   Input ~ 0
-3V3
+Text HLabel 5450 2250 0    50   Input ~ 0
+VCC
 Text Label 5750 4700 2    50   ~ 0
 AGND
@@
 	5950 2900 5950 2400
 Wire Wire Line
-	5750 2300 5750 2400
-Connection ~ 5750 2400
-Wire Wire Line
-	5750 2300 5850 2300
-Wire Wire Line
-	5950 2300 5950 2400
-Connection ~ 5950 2400
-Wire Wire Line
 	5950 2400 6150 2400
 $Comp
-L Device:C C15
+L Device:C C18
 U 1 1 5B2E6585
 P 4650 3100
-F 0 "C15" H 4450 3150 50  0000 L CNN
+F 0 "C18" H 4450 3150 50  0000 L CNN
 F 1 "10N" H 4400 3050 50  0000 L CNN
 F 2 "Capacitors_SMD:C_0402" H 4688 2950 50  0001 C CNN
@@
 $EndComp
 $Comp
-L Device:C C16
+L Device:C C20
 U 1 1 5B2E66DA
 P 4650 3550
-F 0 "C16" H 4450 3600 50  0000 L CNN
+F 0 "C20" H 4450 3600 50  0000 L CNN
 F 1 "10N" H 4400 3500 50  0000 L CNN
 F 2 "Capacitors_SMD:C_0402" H 4688 3400 50  0001 C CNN
@@
 AIN-
 $Comp
-L Device:C C19
+L Device:C C23
 U 1 1 5B2E9EF3
 P 6900 4050
-F 0 "C19" H 6650 4100 50  0000 L CNN
+F 0 "C23" H 6650 4100 50  0000 L CNN
 F 1 "10N" H 6650 4000 50  0000 L CNN
 F 2 "Capacitors_SMD:C_0402" H 6938 3900 50  0001 C CNN
@@
 	6600 4000 6550 4000
 $Comp
-L Device:C C20
+L Device:C C24
 U 1 1 5B2EAA13
 P 6900 4450
-F 0 "C20" H 6650 4500 50  0000 L CNN
+F 0 "C24" H 6650 4500 50  0000 L CNN
 F 1 "10U" H 6650 4400 50  0000 L CNN
 F 2 "Capacitors_SMD:C_0805" H 6938 4300 50  0001 C CNN
@@
 Wire Wire Line
 	6900 4600 6900 4700
-Connection ~ 5950 4700
-Wire Wire Line
-	5750 2200 5850 2200
-Wire Wire Line
-	5850 2200 5850 2300
-Connection ~ 5850 2300
-Wire Wire Line
-	5850 2300 5950 2300
 NoConn ~ 6550 3400
 NoConn ~ 6550 3500
@@
 	4850 4100 5000 4100
 Wire Wire Line
-	5950 4700 5750 4700
-Connection ~ 5750 4700
-Wire Wire Line
 	5750 4700 5750 4600
 Wire Wire Line
@@
 	5500 4700 5750 4700
 Text HLabel 4350 3400 0    50   Input ~ 0
-3V3
+VCC
 Text Label 4350 3700 2    50   ~ 0
 AGND
@@
 Wire Wire Line
 	4350 3400 5150 3400
+$Comp
+L Device:Net-Tie_2 NT1
+U 1 1 5C19759F
+P 5850 2400
+F 0 "NT1" H 5850 2578 50  0000 C CNN
+F 1 "Net-Tie_2" H 5850 2487 50  0000 C CNN
+F 2 "" H 5850 2400 50  0001 C CNN
+F 3 "~" H 5850 2400 50  0001 C CNN
+	1    5850 2400
+	1    0    0    -1
+$EndComp
+Connection ~ 5750 2400
+Connection ~ 5950 2400
+$Comp
+L Device:Net-Tie_2 NT2
+U 1 1 5C1982C7
+P 5850 4700
+F 0 "NT2" H 5850 4878 50  0000 C CNN
+F 1 "Net-Tie_2" H 5850 4787 50  0000 C CNN
+F 2 "" H 5850 4700 50  0001 C CNN
+F 3 "~" H 5850 4700 50  0001 C CNN
+	1    5850 4700
+	-1   0    0    1
+$EndComp
+Connection ~ 5750 4700
+Connection ~ 5950 4700
+Wire Wire Line
+	5450 2250 5550 2250
+Wire Wire Line
+	5550 2250 5550 2400
+Connection ~ 5550 2400
 $EndSCHEMATC

Commit message: fixes, updates, new things for datlogger v2
Parts:
- removed NT1, NT2: Net-Tie_2, symbol Device:Net-Tie_2
- C18: footprint Capacitors_SMD:C_0402 -> Capacitor_SMD:C_0603_1608Metric
- C19: renamed from C20; footprint Capacitors_SMD:C_0402 -> Capacitor_SMD:C_0603_1608Metric
- C20: renamed from C21; footprint Capacitors_SMD:C_0402 -> Capacitor_SMD:C_0603_1608Metric
- C21: renamed from C22; footprint Capacitors_SMD:C_0402 -> Capacitor_SMD:C_0603_1608Metric
- C22: renamed from C23; footprint Capacitors_SMD:C_0402 -> Capacitor_SMD:C_0603_1608Metric
- C23: renamed from C24; footprint Capacitors_SMD:C_0805 -> Capacitor_SMD:C_0805_2012Metric
- U6: renamed from U3; footprint Housings_SSOP:TSSOP-24_4.4x7.8mm_Pitch0.65mm -> Package_SO:TSSOP-24_4.4x7.8mm_P0.65mm; symbol william:MAX11270 -> william_adc:MAX11270EUG+
Connections:
- wire segments 35 -> 41
Changed lines of the file:
@@
 EESchema Schematic File Version 4
-LIBS:main-cache
-EELAYER 26 0
+EELAYER 30 0
 EELAYER END
 $Descr A4 11693 8268
 encoding utf-8
-Sheet 5 8
+Sheet 7 13
 Title ""
 Date ""
@@
 $EndDescr
 $Comp
-L william:MAX11270 U3
+L william_adc:MAX11270EUG+ U6
 U 1 1 5B2E54B9
 P 5850 3750
-F 0 "U3" H 5300 4550 50  0000 C CNN
+F 0 "U6" H 5300 4550 50  0000 C CNN
 F 1 "MAX11270" H 6250 4550 50  0000 C CNN
-F 2 "Housings_SSOP:TSSOP-24_4.4x7.8mm_Pitch0.65mm" H 5700 3800 50  0001 C CNN
+F 2 "Package_SO:TSSOP-24_4.4x7.8mm_P0.65mm" H 5700 3800 50  0001 C CNN
 F 3 "" H 5700 3800 50  0001 C CNN
 	1    5850 3750
@@
 $EndComp
 $Comp
-L Device:C C21
+L Device:C C20
 U 1 1 5B2E54C5
 P 5550 2600
-F 0 "C21" H 5350 2650 50  0000 L CNN
+F 0 "C20" H 5350 2650 50  0000 L CNN
 F 1 "1U" H 5350 2550 50  0000 L CNN
-F 2 "Capacitors_SMD:C_0402" H 5588 2450 50  0001 C CNN
+F 2 "Capacitor_SMD:C_0603_1608Metric" H 5588 2450 50  0001 C CNN
 F 3 "" H 5550 2600 50  0001 C CNN
 	1    5550 2600
@@
 $EndComp
 $Comp
-L Device:C C22
+L Device:C C21
 U 1 1 5B2E54CC
 P 6150 2600
-F 0 "C22" H 6265 2646 50  0000 L CNN
+F 0 "C21" H 6265 2646 50  0000 L CNN
 F 1 "1U" H 6265 2555 50  0000 L CNN
-F 2 "Capacitors_SMD:C_0402" H 6188 2450 50  0001 C CNN
+F 2 "Capacitor_SMD:C_0603_1608Metric" H 6188 2450 50  0001 C CNN
 F 3 "" H 6150 2600 50  0001 C CNN
 	1    6150 2600
@@
 F 0 "C18" H 4450 3150 50  0000 L CNN
 F 1 "10N" H 4400 3050 50  0000 L CNN
-F 2 "Capacitors_SMD:C_0402" H 4688 2950 50  0001 C CNN
+F 2 "Capacitor_SMD:C_0603_1608Metric" H 4688 2950 50  0001 C CNN
 F 3 "" H 4650 3100 50  0001 C CNN
 	1    4650 3100
@@
 $EndComp
 $Comp
-L Device:C C20
+L Device:C C19
 U 1 1 5B2E66DA
 P 4650 3550
-F 0 "C20" H 4450 3600 50  0000 L CNN
+F 0 "C19" H 4450 3600 50  0000 L CNN
 F 1 "10N" H 4400 3500 50  0000 L CNN
-F 2 "Capacitors_SMD:C_0402" H 4688 3400 50  0001 C CNN
+F 2 "Capacitor_SMD:C_0603_1608Metric" H 4688 3400 50  0001 C CNN
 F 3 "" H 4650 3550 50  0001 C CNN
 	1    4650 3550
@@
 AIN-
 $Comp
-L Device:C C23
+L Device:C C22
 U 1 1 5B2E9EF3
 P 6900 4050
-F 0 "C23" H 6650 4100 50  0000 L CNN
+F 0 "C22" H 6650 4100 50  0000 L CNN
 F 1 "10N" H 6650 4000 50  0000 L CNN
-F 2 "Capacitors_SMD:C_0402" H 6938 3900 50  0001 C CNN
+F 2 "Capacitor_SMD:C_0603_1608Metric" H 6938 3900 50  0001 C CNN
 F 3 "" H 6900 4050 50  0001 C CNN
 	1    6900 4050
@@
 	6600 4000 6550 4000
 $Comp
-L Device:C C24
+L Device:C C23
 U 1 1 5B2EAA13
 P 6900 4450
-F 0 "C24" H 6650 4500 50  0000 L CNN
+F 0 "C23" H 6650 4500 50  0000 L CNN
 F 1 "10U" H 6650 4400 50  0000 L CNN
-F 2 "Capacitors_SMD:C_0805" H 6938 4300 50  0001 C CNN
+F 2 "Capacitor_SMD:C_0805_2012Metric" H 6938 4300 50  0001 C CNN
 F 3 "" H 6900 4450 50  0001 C CNN
 	1    6900 4450
@@
 	6600 4100 6550 4100
 Wire Wire Line
-	4350 3700 4850 3700
-Wire Wire Line
-	4350 2950 4850 2950
-Wire Wire Line
-	4350 3250 5150 3250
-Wire Wire Line
-	4350 3400 5150 3400
-$Comp
-L Device:Net-Tie_2 NT1
-U 1 1 5C19759F
-P 5850 2400
-F 0 "NT1" H 5850 2578 50  0000 C CNN
-F 1 "Net-Tie_2" H 5850 2487 50  0000 C CNN
-F 2 "" H 5850 2400 50  0001 C CNN
-F 3 "~" H 5850 2400 50  0001 C CNN
-	1    5850 2400
-	1    0    0    -1
-$EndComp
+	4350 3700 4650 3700
+Wire Wire Line
+	4350 2950 4650 2950
+Wire Wire Line
+	4350 3250 4650 3250
+Wire Wire Line
+	4350 3400 4650 3400
+Wire Wire Line
+	5450 2250 5550 2250
+Wire Wire Line
+	5550 2250 5550 2400
+Connection ~ 5550 2400
+Connection ~ 4650 3400
+Wire Wire Line
+	4650 3400 5150 3400
+Connection ~ 4650 3700
+Wire Wire Line
+	4650 3700 4850 3700
+Connection ~ 4650 2950
+Wire Wire Line
+	4650 2950 4850 2950
+Connection ~ 4650 3250
+Wire Wire Line
+	4650 3250 5150 3250
+Wire Wire Line
+	5750 4700 5950 4700
+Connection ~ 5750 4700
+Connection ~ 5950 4700
+Wire Wire Line
+	5750 2400 5950 2400
 Connection ~ 5750 2400
 Connection ~ 5950 2400
-$Comp
-L Device:Net-Tie_2 NT2
-U 1 1 5C1982C7
-P 5850 4700
-F 0 "NT2" H 5850 4878 50  0000 C CNN
-F 1 "Net-Tie_2" H 5850 4787 50  0000 C CNN
-F 2 "" H 5850 4700 50  0001 C CNN
-F 3 "~" H 5850 4700 50  0001 C CNN
-	1    5850 4700
-	-1   0    0    1
-$EndComp
-Connection ~ 5750 4700
-Connection ~ 5950 4700
-Wire Wire Line
-	5450 2250 5550 2250
-Wire Wire Line
-	5550 2250 5550 2400
-Connection ~ 5550 2400
 $EndSCHEMATC
