File: ICM-20948.sch (KiCad schematic (older format))
At the start: 4 parts, among them U2 ICM-20948

Commit message: add DHT22 & MAX11254 schematics
Parts:
- U2: symbol william_imu:ICM-20948 -> main-rescue:ICM-20948-william_imu
Changed lines of the file:
@@
 $Descr A4 11693 8268
 encoding utf-8
-Sheet 3 4
+Sheet 3 8
 Title ""
 Date ""
@@
 $EndDescr
 $Comp
-L william_imu:ICM-20948 U2
+L main-rescue:ICM-20948-william_imu U2
 U 1 1 5C0145EA
 P 5650 3350
+AR Path="/5C0145EA" Ref="U2"  Part="1"
+AR Path="/5BFF1ADC/5C0145EA" Ref="U2"  Part="1"
 F 0 "U2" H 6200 4000 50  0000 C CNN
 F 1 "ICM-20948" H 5650 3250 50  0000 C CNN

Commit message: changes to STBB1Axx bucks
Parts:
- C2: renamed from C12; footprint (none) -> Capacitor_SMD:C_0603_1608Metric
- C3: renamed from C13; footprint (none) -> Capacitor_SMD:C_0603_1608Metric
- C4: renamed from C14; footprint (none) -> Capacitor_SMD:C_0603_1608Metric
- U2: symbol main-rescue:ICM-20948-william_imu -> william_imu:ICM-20948
Other:
- note added: "7 MHz SPI or 400 kHz Fast Mode I²C"
- note added: "FSYNC := Frame synchronization digital input. Connect to GND if unused"
- note added: "INT1 := Can be push-pull or open drain\nInterrupt Source can be:\nDMP Interrupt\nWake on Motion Interrupt\nPLL RDY Interrupt\nI2C Master Interrupt\nRaw Data Ready Interrupt\nFIFO Overflow Interrupt\nFIFO Watermark Interrupt"
Changed lines of the file:
@@
 EESchema Schematic File Version 4
-LIBS:main-cache
+LIBS:v1-cache
 EELAYER 26 0
 EELAYER END
 $Descr A4 11693 8268
 encoding utf-8
-Sheet 3 9
+Sheet 3 6
 Title ""
 Date ""
@@
 $EndDescr
 $Comp
-L main-rescue:ICM-20948-william_imu U2
+L william_imu:ICM-20948 U?
 U 1 1 5C0145EA
 P 5650 3350
-AR Path="/5C0145EA" Ref="U2"  Part="1"
+AR Path="/5C0145EA" Ref="U?"  Part="1"
 AR Path="/5BFF1ADC/5C0145EA" Ref="U2"  Part="1"
+AR Path="/5C3EEBD8/5C0145EA" Ref="U2"  Part="1"
 F 0 "U2" H 6200 4000 50  0000 C CNN
 F 1 "ICM-20948" H 5650 3250 50  0000 C CNN
@@
 GND
 $Comp
-L Device:C_Small C14
+L Device:C_Small C4
 U 1 1 5C0150F1
 P 6400 4000
-F 0 "C14" H 6309 3954 50  0000 R CNN
+F 0 "C4" H 6309 3954 50  0000 R CNN
 F 1 "100N" H 6309 4045 50  0000 R CNN
-F 2 "" H 6400 4000 50  0001 C CNN
+F 2 "Capacitor_SMD:C_0603_1608Metric" H 6400 4000 50  0001 C CNN
 F 3 "~" H 6400 4000 50  0001 C CNN
 	1    6400 4000
@@
 $EndComp
 $Comp
-L Device:C_Small C12
+L Device:C_Small C2
 U 1 1 5C0151BB
 P 5350 2400
-F 0 "C12" H 5258 2446 50  0000 R CNN
+F 0 "C2" H 5258 2446 50  0000 R CNN
 F 1 "100N" H 5258 2355 50  0000 R CNN
-F 2 "" H 5350 2400 50  0001 C CNN
+F 2 "Capacitor_SMD:C_0603_1608Metric" H 5350 2400 50  0001 C CNN
 F 3 "~" H 5350 2400 50  0001 C CNN
 	1    5350 2400
@@
 1V8
 $Comp
-L Device:C_Small C13
+L Device:C_Small C3
 U 1 1 5C018283
 P 5900 2400
-F 0 "C13" H 5808 2446 50  0000 R CNN
+F 0 "C3" H 5808 2446 50  0000 R CNN
 F 1 "100N" H 5808 2355 50  0000 R CNN
-F 2 "" H 5900 2400 50  0001 C CNN
+F 2 "Capacitor_SMD:C_0603_1608Metric" H 5900 2400 50  0001 C CNN
 F 3 "~" H 5900 2400 50  0001 C CNN
 	1    5900 2400
@@
 Text HLabel 4800 2250 0    50   Input ~ 0
 1V8
+Text Notes 2700 3250 0    50   ~ 0
+7 MHz SPI or 400 kHz Fast Mode I²C
+Text Notes 1500 3550 0    50   ~ 0
+FSYNC := Frame synchronization digital input. Connect to GND if unused
+Text Notes 7400 3200 0    50   ~ 0
+INT1 := Can be push-pull or open drain\nInterrupt Source can be:\nDMP Interrupt\nWake on Motion Interrupt\nPLL RDY Interrupt\nI2C Master Interrupt\nRaw Data Ready Interrupt\nFIFO Overflow Interrupt\nFIFO Watermark Interrupt
 $EndSCHEMATC

Commit message: fixes, updates, new things for datlogger v2
Parts:
- renumbered C3 to C10, C4 to C11, C2 to C9, U2 to U3
Connections:
- net labels added: REG
Changed lines of the file:
@@
 EESchema Schematic File Version 4
-LIBS:v1-cache
-EELAYER 26 0
+EELAYER 30 0
 EELAYER END
 $Descr A4 11693 8268
 encoding utf-8
-Sheet 3 6
+Sheet 6 13
 Title ""
 Date ""
@@
 P 5650 3350
 AR Path="/5C0145EA" Ref="U?"  Part="1"
-AR Path="/5BFF1ADC/5C0145EA" Ref="U2"  Part="1"
-AR Path="/5C3EEBD8/5C0145EA" Ref="U2"  Part="1"
-F 0 "U2" H 6200 4000 50  0000 C CNN
+AR Path="/5BFF1ADC/5C0145EA" Ref="U?"  Part="1"
+AR Path="/5C3EEBD8/5C0145EA" Ref="U?"  Part="1"
+AR Path="/5EC590AF/5C0145EA" Ref="U3"  Part="1"
+AR Path="/5EC729B7/5C0145EA" Ref="U?"  Part="1"
+AR Path="/5EC732C7/5C0145EA" Ref="U?"  Part="1"
+AR Path="/5EC8743F/5C0145EA" Ref="U4"  Part="1"
+AR Path="/5EC8EDA5/5C0145EA" Ref="U5"  Part="1"
+F 0 "U5" H 6200 4000 50  0000 C CNN
 F 1 "ICM-20948" H 5650 3250 50  0000 C CNN
 F 2 "Sensor_Motion:InvenSense_QFN-24_3x3mm_P0.4mm" H 5700 2900 50  0001 C CNN
@@
 GND
 $Comp
-L Device:C_Small C4
+L Device:C_Small C11
 U 1 1 5C0150F1
 P 6400 4000
-F 0 "C4" H 6309 3954 50  0000 R CNN
+AR Path="/5EC590AF/5C0150F1" Ref="C11"  Part="1"
+AR Path="/5EC729B7/5C0150F1" Ref="C?"  Part="1"
+AR Path="/5EC732C7/5C0150F1" Ref="C?"  Part="1"
+AR Path="/5EC8743F/5C0150F1" Ref="C14"  Part="1"
+AR Path="/5EC8EDA5/5C0150F1" Ref="C17"  Part="1"
+F 0 "C17" H 6309 3954 50  0000 R CNN
 F 1 "100N" H 6309 4045 50  0000 R CNN
 F 2 "Capacitor_SMD:C_0603_1608Metric" H 6400 4000 50  0001 C CNN
@@
 $EndComp
 $Comp
-L Device:C_Small C2
+L Device:C_Small C9
 U 1 1 5C0151BB
 P 5350 2400
-F 0 "C2" H 5258 2446 50  0000 R CNN
+AR Path="/5EC590AF/5C0151BB" Ref="C9"  Part="1"
+AR Path="/5EC729B7/5C0151BB" Ref="C?"  Part="1"
+AR Path="/5EC732C7/5C0151BB" Ref="C?"  Part="1"
+AR Path="/5EC8743F/5C0151BB" Ref="C12"  Part="1"
+AR Path="/5EC8EDA5/5C0151BB" Ref="C15"  Part="1"
+F 0 "C15" H 5258 2446 50  0000 R CNN
 F 1 "100N" H 5258 2355 50  0000 R CNN
 F 2 "Capacitor_SMD:C_0603_1608Metric" H 5350 2400 50  0001 C CNN
@@
 1V8
 $Comp
-L Device:C_Small C3
+L Device:C_Small C10
 U 1 1 5C018283
 P 5900 2400
-F 0 "C3" H 5808 2446 50  0000 R CNN
+AR Path="/5EC590AF/5C018283" Ref="C10"  Part="1"
+AR Path="/5EC729B7/5C018283" Ref="C?"  Part="1"
+AR Path="/5EC732C7/5C018283" Ref="C?"  Part="1"
+AR Path="/5EC8743F/5C018283" Ref="C13"  Part="1"
+AR Path="/5EC8EDA5/5C018283" Ref="C16"  Part="1"
+F 0 "C16" H 5808 2446 50  0000 R CNN
 F 1 "100N" H 5808 2355 50  0000 R CNN
 F 2 "Capacitor_SMD:C_0603_1608Metric" H 5900 2400 50  0001 C CNN
@@
 Text Notes 7400 3200 0    50   ~ 0
 INT1 := Can be push-pull or open drain\nInterrupt Source can be:\nDMP Interrupt\nWake on Motion Interrupt\nPLL RDY Interrupt\nI2C Master Interrupt\nRaw Data Ready Interrupt\nFIFO Overflow Interrupt\nFIFO Watermark Interrupt
+Text Label 6400 3800 0    50   ~ 0
+REG
 $EndSCHEMATC

Commit message: fixed some footprints
Parts:
- U3: footprint Sensor_Motion:InvenSense_QFN-24_3x3mm_P0.4mm -> william_imu:ICM-20948
Changed lines of the file:
@@
 F 0 "U5" H 6200 4000 50  0000 C CNN
 F 1 "ICM-20948" H 5650 3250 50  0000 C CNN
-F 2 "Sensor_Motion:InvenSense_QFN-24_3x3mm_P0.4mm" H 5700 2900 50  0001 C CNN
+F 2 "william_imu:ICM-20948" H 5700 2900 50  0001 C CNN
 F 3 "" H 5700 2900 50  0001 C CNN
 	1    5650 3350
