File: STBB1Axx_1V8.sch (KiCad schematic (older format))
At the start: 10 parts, among them U4 STBB1-Axx

Commit message: fixes, updates, new things for datlogger v2
Parts:
- removed NT3, NT4: ~, NetTie:NetTie-2_SMD_Pad0.5mm, symbol Device:Net-Tie_2
- L2: footprint Inductor_SMD:L_Taiyo-Yuden_MD-4040 -> william_inductor:L_Taiyo-Yuden_MD-4040
- renumbered C12 to C5, C13 to C6, C14 to C7, C15 to C8, R7 to R6, R8 to R7, U4 to U2
Connections:
- wire segments 41 -> 40
Changed lines of the file:
@@
 EESchema Schematic File Version 4
-LIBS:v1-cache
-EELAYER 26 0
+EELAYER 30 0
 EELAYER END
 $Descr A4 11693 8268
 encoding utf-8
-Sheet 5 6
+Sheet 3 13
 Title ""
 Date ""
@@
 AR Path="/5C3F7E47/5C42D59C" Ref="U?"  Part="1"
 AR Path="/5C3FDE71/5C42D59C" Ref="U?"  Part="1"
-AR Path="/5C3FF9CB/5C42D59C" Ref="U4"  Part="1"
-F 0 "U4" H 6050 3050 50  0000 L CNN
+AR Path="/5C3FF9CB/5C42D59C" Ref="U?"  Part="1"
+AR Path="/5EC44D2D/5C42D59C" Ref="U2"  Part="1"
+AR Path="/5ED128B8/5C42D59C" Ref="U?"  Part="1"
+F 0 "U2" H 6050 3050 50  0000 L CNN
 F 1 "STBB1-Axx" H 5400 2550 50  0000 L CNN
 F 2 "Package_DFN_QFN:DFN-10-1EP_2x3mm_P0.5mm_EP0.64x2.4mm" H 5250 2700 50  0001 C CNN
@@
 AR Path="/5C3F7E47/5C42D5A4" Ref="L?"  Part="1"
 AR Path="/5C3FDE71/5C42D5A4" Ref="L?"  Part="1"
-AR Path="/5C3FF9CB/5C42D5A4" Ref="L2"  Part="1"
+AR Path="/5C3FF9CB/5C42D5A4" Ref="L?"  Part="1"
+AR Path="/5EC44D2D/5C42D5A4" Ref="L2"  Part="1"
+AR Path="/5ED128B8/5C42D5A4" Ref="L?"  Part="1"
 F 0 "L2" H 4709 2304 50  0000 R CNN
 F 1 "2U2" H 4709 2395 50  0000 R CNN
-F 2 "Inductor_SMD:L_Taiyo-Yuden_MD-4040" H 4750 2350 50  0001 C CNN
+F 2 "william_inductor:L_Taiyo-Yuden_MD-4040" H 4750 2350 50  0001 C CNN
 F 3 "~" H 4750 2350 50  0001 C CNN
 	1    4750 2350
@@
 	6350 2550 6250 2550
 Wire Wire Line
-	5650 3250 5650 3100
+	5650 3250 5650 3200
 Wire Wire Line
 	3700 1900 4000 1900
@@
 AR Path="/5C3F7E47/5C42D5B3" Ref="C?"  Part="1"
 AR Path="/5C3FDE71/5C42D5B3" Ref="C?"  Part="1"
-AR Path="/5C3FF9CB/5C42D5B3" Ref="C14"  Part="1"
-F 0 "C14" H 6965 2696 50  0000 L CNN
+AR Path="/5C3FF9CB/5C42D5B3" Ref="C?"  Part="1"
+AR Path="/5EC44D2D/5C42D5B3" Ref="C7"  Part="1"
+AR Path="/5ED128B8/5C42D5B3" Ref="C?"  Part="1"
+F 0 "C7" H 6965 2696 50  0000 L CNN
 F 1 "22U" H 6965 2605 50  0000 L CNN
 F 2 "Capacitor_SMD:C_0805_2012Metric" H 6888 2500 50  0001 C CNN
@@
 P 6350 2400
 AR Path="/5C3F7E47/5C42D5C3" Ref="R?"  Part="1"
-AR Path="/5C3FF9CB/5C42D5C3" Ref="R7"  Part="1"
-F 0 "R7" H 6418 2446 50  0000 L CNN
+AR Path="/5C3FF9CB/5C42D5C3" Ref="R?"  Part="1"
+AR Path="/5EC44D2D/5C42D5C3" Ref="R6"  Part="1"
+AR Path="/5ED128B8/5C42D5C3" Ref="R?"  Part="1"
+F 0 "R6" H 6418 2446 50  0000 L CNN
 F 1 "270K" H 6418 2355 50  0000 L CNN
 F 2 "Resistor_SMD:R_0603_1608Metric" V 6390 2390 50  0001 C CNN
@@
 P 6350 3050
 AR Path="/5C3F7E47/5C42D5CA" Ref="R?"  Part="1"
-AR Path="/5C3FF9CB/5C42D5CA" Ref="R8"  Part="1"
-F 0 "R8" H 6418 3096 50  0000 L CNN
+AR Path="/5C3FF9CB/5C42D5CA" Ref="R?"  Part="1"
+AR Path="/5EC44D2D/5C42D5CA" Ref="R7"  Part="1"
+AR Path="/5ED128B8/5C42D5CA" Ref="R?"  Part="1"
+F 0 "R7" H 6418 3096 50  0000 L CNN
 F 1 "100K" H 6418 3005 50  0000 L CNN
 F 2 "Resistor_SMD:R_0603_1608Metric" V 6390 3040 50  0001 C CNN
@@
 AR Path="/5C3F7E47/5C42D5D4" Ref="C?"  Part="1"
 AR Path="/5C3FDE71/5C42D5D4" Ref="C?"  Part="1"
-AR Path="/5C3FF9CB/5C42D5D4" Ref="C13"  Part="1"
-F 0 "C13" H 4315 2696 50  0000 L CNN
+AR Path="/5C3FF9CB/5C42D5D4" Ref="C?"  Part="1"
+AR Path="/5EC44D2D/5C42D5D4" Ref="C6"  Part="1"
+AR Path="/5ED128B8/5C42D5D4" Ref="C?"  Part="1"
+F 0 "C6" H 4315 2696 50  0000 L CNN
 F 1 "10U" H 4315 2605 50  0000 L CNN
 F 2 "Capacitor_SMD:C_0805_2012Metric" H 4238 2500 50  0001 C CNN
@@
 Text Notes 6600 1950 0    50   ~ 0
 Vout from 1V2 to 5V5
-$Comp
-L Device:Net-Tie_2 NT?
-U 1 1 5C42D5DD
-P 5550 3250
-AR Path="/5C3F7E47/5C42D5DD" Ref="NT?"  Part="1"
-AR Path="/5C3FF9CB/5C42D5DD" Ref="NT4"  Part="1"
-F 0 "NT4" H 5550 3164 50  0000 C CNN
-F 1 "~" H 5550 3337 50  0000 C CNN
-F 2 "NetTie:NetTie-2_SMD_Pad0.5mm" H 5550 3250 50  0001 C CNN
-F 3 "~" H 5550 3250 50  0001 C CNN
-	1    5550 3250
-	1    0    0    -1
-$EndComp
-Text HLabel 5800 3250 2    50   Input ~ 0
+Text HLabel 3700 3250 0    50   Input ~ 0
 GND
-$Comp
-L Device:Net-Tie_2 NT?
-U 1 1 5C42D5E5
-P 5550 1900
-AR Path="/5C3F7E47/5C42D5E5" Ref="NT?"  Part="1"
-AR Path="/5C3FF9CB/5C42D5E5" Ref="NT3"  Part="1"
-F 0 "NT3" H 5550 1986 50  0000 C CNN
-F 1 "~" H 5550 1987 50  0000 C CNN
-F 2 "NetTie:NetTie-2_SMD_Pad0.5mm" H 5550 1900 50  0001 C CNN
-F 3 "~" H 5550 1900 50  0001 C CNN
-	1    5550 1900
-	1    0    0    -1
-$EndComp
 Wire Wire Line
 	4500 1900 5450 1900
@@
 Connection ~ 5450 3250
 Wire Wire Line
-	5450 3100 5450 3250
+	5450 3200 5450 3250
 Wire Wire Line
 	6350 2550 6350 2900
@@
 AR Path="/5C3F7E47/5C42D5F9" Ref="C?"  Part="1"
 AR Path="/5C3FDE71/5C42D5F9" Ref="C?"  Part="1"
-AR Path="/5C3FF9CB/5C42D5F9" Ref="C15"  Part="1"
-F 0 "C15" H 7165 2696 50  0000 L CNN
+AR Path="/5C3FF9CB/5C42D5F9" Ref="C?"  Part="1"
+AR Path="/5EC44D2D/5C42D5F9" Ref="C8"  Part="1"
+AR Path="/5ED128B8/5C42D5F9" Ref="C?"  Part="1"
+F 0 "C8" H 7165 2696 50  0000 L CNN
 F 1 "100N" H 7165 2605 50  0000 L CNN
 F 2 "Capacitor_SMD:C_0603_1608Metric" H 7088 2500 50  0001 C CNN
@@
 AR Path="/5C3F7E47/5C42D607" Ref="C?"  Part="1"
 AR Path="/5C3FDE71/5C42D607" Ref="C?"  Part="1"
-AR Path="/5C3FF9CB/5C42D607" Ref="C12"  Part="1"
-F 0 "C12" H 4115 2696 50  0000 L CNN
+AR Path="/5C3FF9CB/5C42D607" Ref="C?"  Part="1"
+AR Path="/5EC44D2D/5C42D607" Ref="C5"  Part="1"
+AR Path="/5ED128B8/5C42D607" Ref="C?"  Part="1"
+F 0 "C5" H 4115 2696 50  0000 L CNN
 F 1 "100N" H 4115 2605 50  0000 L CNN
 F 2 "Capacitor_SMD:C_0603_1608Metric" H 4038 2500 50  0001 C CNN
@@
 $EndComp
 Connection ~ 4000 1900
-Connection ~ 5450 1900
 Wire Wire Line
 	4000 2500 4000 1900
@@
 	4200 2800 4200 3250
 Wire Wire Line
-	4200 3250 4600 3250
-Wire Wire Line
-	4000 2800 4000 3250
-Wire Wire Line
 	4000 3250 4200 3250
 Connection ~ 4200 3250
@@
 Connection ~ 6350 3500
 Wire Wire Line
-	5800 3250 5650 3250
-Connection ~ 5650 3250
-Wire Wire Line
 	6850 2200 7050 2200
-$Comp
-L v1-rescue:PWR_FLAG-v1-rescue #FLG?
-U 1 1 5C5843D1
-P 5850 1800
-AR Path="/5C5843D1" Ref="#FLG?"  Part="1"
-AR Path="/5C3FF9CB/5C5843D1" Ref="#FLG0108"  Part="1"
-F 0 "#FLG0108" H 5850 1875 50  0001 C CNN
-F 1 "PWR_FLAG" H 5850 1950 50  0000 C CNN
-F 2 "" H 5850 1800 50  0001 C CNN
-F 3 "" H 5850 1800 50  0001 C CNN
-	1    5850 1800
-	1    0    0    -1
-$EndComp
-Wire Wire Line
-	5850 1800 5850 1900
-Wire Wire Line
-	5850 1900 5650 1900
-Connection ~ 5650 1900
-$Comp
-L v1-rescue:PWR_FLAG-v1-rescue #FLG?
-U 1 1 5C5866EA
-P 4600 3200
-AR Path="/5C5866EA" Ref="#FLG?"  Part="1"
-AR Path="/5C3FF9CB/5C5866EA" Ref="#FLG0109"  Part="1"
-F 0 "#FLG0109" H 4600 3275 50  0001 C CNN
-F 1 "PWR_FLAG" H 4600 3350 50  0000 C CNN
-F 2 "" H 4600 3200 50  0001 C CNN
-F 3 "" H 4600 3200 50  0001 C CNN
-	1    4600 3200
-	1    0    0    -1
-$EndComp
-Wire Wire Line
-	4600 3200 4600 3250
-Connection ~ 4600 3250
-Wire Wire Line
-	4600 3250 5450 3250
+Wire Wire Line
+	4200 3250 5450 3250
+Wire Wire Line
+	3700 3250 4000 3250
+Connection ~ 4000 3250
+Wire Wire Line
+	5650 1900 5450 1900
+Connection ~ 5450 1900
+Wire Wire Line
+	4000 3200 4000 3250
+Wire Wire Line
+	4000 2800 4000 3250
+Wire Wire Line
+	5650 3250 5450 3250
 $EndSCHEMATC

Commit message: fixed some footprints
Parts:
- U2: footprint Package_DFN_QFN:DFN-10-1EP_2x3mm_P0.5mm_EP0.64x2.4mm -> Package_DFN_QFN:DFN-10-1EP_3x3mm_P0.5mm_EP1.7x2.5mm
Changed lines of the file:
@@
 F 0 "U2" H 6050 3050 50  0000 L CNN
 F 1 "STBB1-Axx" H 5400 2550 50  0000 L CNN
-F 2 "Package_DFN_QFN:DFN-10-1EP_2x3mm_P0.5mm_EP0.64x2.4mm" H 5250 2700 50  0001 C CNN
+F 2 "Package_DFN_QFN:DFN-10-1EP_3x3mm_P0.5mm_EP1.7x2.5mm" H 5250 2700 50  0001 C CNN
 F 3 "http://www.st.com/content/ccc/resource/technical/document/datasheet/20/a6/10/e0/63/85/43/c1/DM00037824.pdf/files/DM00037824.pdf/jcr:content/translations/en.DM00037824.pdf" H 5250 2700 50  0001 C CNN
 	1    5550 2550
