File: MCP73831-2-OT.sch (KiCad schematic (older format))
At the start: 6 parts, among them U3 MCP73831-2-OT

Commit message: changed max schematics
Other:
- note added: "Blue pref, for low current consumption"
- note removed: "Blue"
Changed lines of the file:
@@
-EESchema Schematic File Version 5
-EELAYER 31 0
+EESchema Schematic File Version 4
+EELAYER 30 0
 EELAYER END
 $Descr A4 11693 8268
@@
 Comment3 ""
 Comment4 ""
-Comment5 ""
-Comment6 ""
-Comment7 ""
-Comment8 ""
-Comment9 ""
 $EndDescr
 Connection ~ 5900 3100
@@
 LOW ON CHARGING\nHIGH Z OTHERWISE \n(OPEN DRAIN)
 Text Notes 7100 2600 0    50   ~ 0
-Blue
+Blue pref, for low current consumption
 Text HLabel 2300 2900 0    50   Input ~ 0
 VIN

Commit message: schematics for milad board v0
Parts:
- renumbered C10 to C1, C11 to C2, D4 to D1, R10 to R1, R11 to R2, U3 to U2
Changed lines of the file:
@@
 $Descr A4 11693 8268
 encoding utf-8
-Sheet 2 10
+Sheet 2 6
 Title ""
 Date ""
@@
 VIN
 $Comp
-L Device:R R10
+L Device:R R1
 U 1 1 5E20F2A0
 P 4850 3350
-F 0 "R10" H 4920 3396 50  0000 L CNN
+F 0 "R1" H 4920 3396 50  0000 L CNN
 F 1 "1K" H 4920 3305 50  0000 L CNN
 F 2 "Resistor_SMD:R_0603_1608Metric" V 4780 3350 50  0001 C CNN
@@
 $EndComp
 $Comp
-L Device:R R11
+L Device:R R2
 U 1 1 5E2112C7
 P 6750 2850
-F 0 "R11" H 6820 2896 50  0000 L CNN
+F 0 "R2" H 6820 2896 50  0000 L CNN
 F 1 "1K" H 6820 2805 50  0000 L CNN
 F 2 "Resistor_SMD:R_0603_1608Metric" V 6680 2850 50  0001 C CNN
@@
 $EndComp
 $Comp
-L Device:LED D4
+L Device:LED D1
 U 1 1 5E20FC43
 P 6750 2550
-F 0 "D4" V 6789 2433 50  0000 R CNN
+F 0 "D1" V 6789 2433 50  0000 R CNN
 F 1 "LED" V 6698 2433 50  0000 R CNN
 F 2 "LED_SMD:LED_0603_1608Metric" H 6750 2550 50  0001 C CNN
@@
 $EndComp
 $Comp
-L Device:C C10
+L Device:C C1
 U 1 1 5E216D79
 P 2400 3150
-F 0 "C10" H 2285 3104 50  0000 R CNN
+F 0 "C1" H 2285 3104 50  0000 R CNN
 F 1 "4U7" H 2285 3195 50  0000 R CNN
 F 2 "Capacitor_SMD:C_0603_1608Metric" H 2438 3000 50  0001 C CNN
@@
 $EndComp
 $Comp
-L Device:C C11
+L Device:C C2
 U 1 1 5E2164A5
 P 3100 3150
-F 0 "C11" H 3215 3196 50  0000 L CNN
+F 0 "C2" H 3215 3196 50  0000 L CNN
 F 1 "4U7" H 3215 3105 50  0000 L CNN
 F 2 "Capacitor_SMD:C_0603_1608Metric" H 3138 3000 50  0001 C CNN
@@
 $EndComp
 $Comp
-L Battery_Management:MCP73831-2-OT U3
+L Battery_Management:MCP73831-2-OT U2
 U 1 1 5E205A54
 P 5350 3000
-F 0 "U3" H 5600 3250 50  0000 C CNN
+F 0 "U2" H 5600 3250 50  0000 C CNN
 F 1 "MCP73831-2-OT" H 5350 3700 50  0000 C CNN
 F 2 "Package_TO_SOT_SMD:SOT-23-5" H 5400 2750 50  0001 L CIN

Commit message: adding milad subs
Parts:
- renumbered D1 to D2, R1 to R2, R2 to R3, U2 to U1
Changed lines of the file:
@@
 $Descr A4 11693 8268
 encoding utf-8
-Sheet 2 6
+Sheet 2 10
 Title ""
 Date ""
@@
 VIN
 $Comp
-L Device:R R1
+L Device:R R2
 U 1 1 5E20F2A0
 P 4850 3350
-F 0 "R1" H 4920 3396 50  0000 L CNN
+F 0 "R2" H 4920 3396 50  0000 L CNN
 F 1 "1K" H 4920 3305 50  0000 L CNN
 F 2 "Resistor_SMD:R_0603_1608Metric" V 4780 3350 50  0001 C CNN
@@
 $EndComp
 $Comp
-L Device:R R2
+L Device:R R3
 U 1 1 5E2112C7
 P 6750 2850
-F 0 "R2" H 6820 2896 50  0000 L CNN
+F 0 "R3" H 6820 2896 50  0000 L CNN
 F 1 "1K" H 6820 2805 50  0000 L CNN
 F 2 "Resistor_SMD:R_0603_1608Metric" V 6680 2850 50  0001 C CNN
@@
 $EndComp
 $Comp
-L Device:LED D1
+L Device:LED D2
 U 1 1 5E20FC43
 P 6750 2550
-F 0 "D1" V 6789 2433 50  0000 R CNN
+F 0 "D2" V 6789 2433 50  0000 R CNN
 F 1 "LED" V 6698 2433 50  0000 R CNN
 F 2 "LED_SMD:LED_0603_1608Metric" H 6750 2550 50  0001 C CNN
@@
 $EndComp
 $Comp
-L Battery_Management:MCP73831-2-OT U2
+L Battery_Management:MCP73831-2-OT U1
 U 1 1 5E205A54
 P 5350 3000
-F 0 "U2" H 5600 3250 50  0000 C CNN
+F 0 "U1" H 5600 3250 50  0000 C CNN
 F 1 "MCP73831-2-OT" H 5350 3700 50  0000 C CNN
 F 2 "Package_TO_SOT_SMD:SOT-23-5" H 5400 2750 50  0001 L CIN
