File: cp2102.sch (KiCad schematic (older format))
At the start: 5 parts

Commit message: adding milad subs
Parts:
- C12: renamed from C?; footprint (none) -> Capacitor_SMD:C_0603_1608Metric
- J4: renamed from J?; footprint (none) -> william_usb:USB_Micro_B_Female_10118194-0001LF
- R15, R16: renamed from R?; footprint (none) -> Resistor_SMD:R_0603_1608Metric
- gave numbers to parts that had none: 1
Changed lines of the file:
@@
 $Descr A4 11693 8268
 encoding utf-8
-Sheet 6 6
+Sheet 6 10
 Title ""
 Date ""
@@
 P 5800 3750
 AR Path="/5F789CB7/5F79DC9C" Ref="U?"  Part="1"
-AR Path="/5F789CB7/5F79B8DA/5F79DC9C" Ref="U?"  Part="1"
-F 0 "U?" H 6000 5150 50  0000 C CNN
+AR Path="/5F789CB7/5F79B8DA/5F79DC9C" Ref="U3"  Part="1"
+F 0 "U3" H 6000 5150 50  0000 C CNN
 F 1 "CP2102N-A01-GQFN28" H 6400 5050 50  0000 C CNN
 F 2 "Package_DFN_QFN:QFN-28-1EP_5x5mm_P0.5mm_EP3.35x3.35mm" H 6250 2550 50  0001 L CNN
@@
 P 7000 2850
 AR Path="/5F789CB7/5F79DCB7" Ref="R?"  Part="1"
-AR Path="/5F789CB7/5F79B8DA/5F79DCB7" Ref="R?"  Part="1"
-F 0 "R?" V 6793 2850 50  0000 C CNN
+AR Path="/5F789CB7/5F79B8DA/5F79DCB7" Ref="R15"  Part="1"
+F 0 "R15" V 6793 2850 50  0000 C CNN
 F 1 "100R" V 6884 2850 50  0000 C CNN
-F 2 "" V 6930 2850 50  0001 C CNN
+F 2 "Resistor_SMD:R_0603_1608Metric" V 6930 2850 50  0001 C CNN
 F 3 "~" H 7000 2850 50  0001 C CNN
 	1    7000 2850
@@
 P 7000 2950
 AR Path="/5F789CB7/5F79DCBD" Ref="R?"  Part="1"
-AR Path="/5F789CB7/5F79B8DA/5F79DCBD" Ref="R?"  Part="1"
-F 0 "R?" V 7207 2950 50  0000 C CNN
+AR Path="/5F789CB7/5F79B8DA/5F79DCBD" Ref="R16"  Part="1"
+F 0 "R16" V 7207 2950 50  0000 C CNN
 F 1 "100R" V 7116 2950 50  0000 C CNN
-F 2 "" V 6930 2950 50  0001 C CNN
+F 2 "Resistor_SMD:R_0603_1608Metric" V 6930 2950 50  0001 C CNN
 F 3 "~" H 7000 2950 50  0001 C CNN
 	1    7000 2950
@@
 P 3850 3150
 AR Path="/5F79DCC7" Ref="J?"  Part="1"
-AR Path="/5F789CB7/5F79B8DA/5F79DCC7" Ref="J?"  Part="1"
-F 0 "J?" H 3907 3617 50  0000 C CNN
+AR Path="/5F789CB7/5F79B8DA/5F79DCC7" Ref="J4"  Part="1"
+F 0 "J4" H 3907 3617 50  0000 C CNN
 F 1 "USB_B_Micro" H 3907 3526 50  0000 C CNN
-F 2 "" H 4000 3100 50  0001 C CNN
+F 2 "william_usb:USB_Micro_B_Female_10118194-0001LF" H 4000 3100 50  0001 C CNN
 F 3 "~" H 4000 3100 50  0001 C CNN
 	1    3850 3150
 	1    0    0    -1
 $EndComp
-$Comp
-L power:GND #PWR?
-U 1 1 5F79DCCD
-P 3850 3650
-AR Path="/5F79DCCD" Ref="#PWR?"  Part="1"
-AR Path="/5F789CB7/5F79B8DA/5F79DCCD" Ref="#PWR?"  Part="1"
-F 0 "#PWR?" H 3850 3400 50  0001 C CNN
-F 1 "GND" H 3855 3477 50  0000 C CNN
-F 2 "" H 3850 3650 50  0001 C CNN
-F 3 "" H 3850 3650 50  0001 C CNN
-	1    3850 3650
-	1    0    0    -1
-$EndComp
-Wire Wire Line
-	3850 3650 3850 3600
 NoConn ~ 5300 2850
-Text HLabel 4750 2850 2    50   Output ~ 0
+Text HLabel 4550 2850 0    50   Output ~ 0
 VBUS
 Wire Wire Line
@@
 Wire Wire Line
 	3750 3600 3850 3600
-Connection ~ 3850 3600
 Wire Wire Line
 	3850 3600 3850 3550
@@
 	4650 3050 5300 3050
 Wire Wire Line
-	4750 2850 4650 2850
+	4550 2850 4650 2850
 Wire Wire Line
 	4650 2850 4650 2950
@@
 VBUS
 $Comp
-L Device:C C?
+L Device:C C12
 U 1 1 5F7C0359
 P 2350 3150
-F 0 "C?" H 2465 3196 50  0000 L CNN
+F 0 "C12" H 2465 3196 50  0000 L CNN
 F 1 "100N" H 2465 3105 50  0000 L CNN
-F 2 "" H 2388 3000 50  0001 C CNN
+F 2 "Capacitor_SMD:C_0603_1608Metric" H 2388 3000 50  0001 C CNN
 F 3 "~" H 2350 3150 50  0001 C CNN
 	1    2350 3150
@@
 Wire Wire Line
 	2250 3400 2350 3400
+Text HLabel 3650 3600 0    50   Input ~ 0
+GND
+Wire Wire Line
+	3650 3600 3750 3600
+Connection ~ 3750 3600
 $EndSCHEMATC

Commit message: updated esp32
Parts:
- renumbered U3 to U4
Changed lines of the file:
@@
 P 5800 3750
 AR Path="/5F789CB7/5F79DC9C" Ref="U?"  Part="1"
-AR Path="/5F789CB7/5F79B8DA/5F79DC9C" Ref="U3"  Part="1"
-F 0 "U3" H 6000 5150 50  0000 C CNN
+AR Path="/5F789CB7/5F79B8DA/5F79DC9C" Ref="U4"  Part="1"
+F 0 "U4" H 6000 5150 50  0000 C CNN
 F 1 "CP2102N-A01-GQFN28" H 6400 5050 50  0000 C CNN
 F 2 "Package_DFN_QFN:QFN-28-1EP_5x5mm_P0.5mm_EP3.35x3.35mm" H 6250 2550 50  0001 L CNN
