File: pam2421_6V3.sch (KiCad schematic (older format))
At the start: 14 parts, among them U4 PAM2423AECADJR

Commit message: updated esp32
Parts:
- renumbered U4 to U5
Changed lines of the file:
@@
 $EndDescr
 $Comp
-L william_dc_dc:PAM2423AECADJR U4
+L william_dc_dc:PAM2423AECADJR U5
 U 1 1 5F859E56
 P 5350 3350
-F 0 "U4" H 5350 3817 50  0000 C CNN
+F 0 "U5" H 5350 3817 50  0000 C CNN
 F 1 "PAM2423AECADJR" H 5350 3726 50  0000 C CNN
 F 2 "Package_SO:HTSOP-8-1EP_3.9x4.9mm_P1.27mm_EP2.4x3.2mm_ThermalVias" H 4750 3950 50  0001 L CNN
@@
 > 1.4V
 $Comp
-L power:PWR_FLAG #FLG0101
+L power:PWR_FLAG #FLG01
 U 1 1 5F8A657A
 P 7600 2700
-F 0 "#FLG0101" H 7600 2775 50  0001 C CNN
+F 0 "#FLG01" H 7600 2775 50  0001 C CNN
 F 1 "PWR_FLAG" H 7600 2873 50  0000 C CNN
 F 2 "" H 7600 2700 50  0001 C CNN
