File: STM32F446RETx.sch (KiCad schematic (older format))
At the start: 13 parts, among them J4 SWD_PROG_HEADER, U3 STM32F446RETx, Y1 ABM3-8.000MHZ-D2Y-T

Commit message: updated STM32F446RETx
Parts:
- C?: renamed from C18; symbol device:C_Small -> Device:C_Small
- C?: renamed from C19; symbol device:C -> Device:C
- C?: renamed from C20; symbol device:C -> Device:C
- C?: renamed from C21; symbol device:C -> Device:C
- C?: renamed from C22; symbol device:C -> Device:C
- C?: renamed from C23; symbol device:C -> Device:C
- C?: renamed from C24; symbol device:C -> Device:C
- C?: renamed from C25; symbol device:C -> Device:C
- C?: renamed from C26; symbol device:C -> Device:C
- C?: renamed from C27; symbol device:C -> Device:C
- J?: renamed from J4; symbol conn:Conn_01x06 -> Connector_Generic:Conn_01x06
- Y?: renamed from Y1; symbol device:Crystal -> Device:Crystal
- renumbered U3 to U?
Changed lines of the file:
@@
 EESchema Schematic File Version 4
-LIBS:strain_gauge_485-cache
+LIBS:main-cache
 EELAYER 26 0
 EELAYER END
 $Descr A4 11693 8268
 encoding utf-8
-Sheet 4 4
+Sheet 12 12
 Title ""
 Date ""
@@
 3V3
 $Comp
-L device:C_Small C18
+L Device:C_Small C?
 U 1 1 5B322B70
 P 900 1950
-F 0 "C18" H 992 1996 50  0000 L CNN
+F 0 "C?" H 992 1996 50  0000 L CNN
 F 1 "2U2" H 992 1905 50  0000 L CNN
 F 2 "Capacitors_SMD:C_0402" H 900 1950 50  0001 C CNN
@@
 3V3
 $Comp
-L device:C C19
+L Device:C C?
 U 1 1 5B32459A
 P 3850 6000
-F 0 "C19" H 3965 6046 50  0000 L CNN
+F 0 "C?" H 3965 6046 50  0000 L CNN
 F 1 "10U" H 3965 5955 50  0000 L CNN
 F 2 "Capacitors_SMD:C_0805" H 3888 5850 50  0001 C CNN
@@
 $EndComp
 $Comp
-L device:C C20
+L Device:C C?
 U 1 1 5B324834
 P 4350 6000
-F 0 "C20" H 4465 6046 50  0000 L CNN
+F 0 "C?" H 4465 6046 50  0000 L CNN
 F 1 "100N" H 4465 5955 50  0000 L CNN
 F 2 "Capacitors_SMD:C_0402" H 4388 5850 50  0001 C CNN
@@
 $EndComp
 $Comp
-L device:C C21
+L Device:C C?
 U 1 1 5B32486E
 P 4800 6000
-F 0 "C21" H 4915 6046 50  0000 L CNN
+F 0 "C?" H 4915 6046 50  0000 L CNN
 F 1 "100N" H 4915 5955 50  0000 L CNN
 F 2 "Capacitors_SMD:C_0402" H 4838 5850 50  0001 C CNN
@@
 $EndComp
 $Comp
-L device:C C22
+L Device:C C?
 U 1 1 5B324896
 P 5200 6000
-F 0 "C22" H 5315 6046 50  0000 L CNN
+F 0 "C?" H 5315 6046 50  0000 L CNN
 F 1 "100N" H 5315 5955 50  0000 L CNN
 F 2 "Capacitors_SMD:C_0402" H 5238 5850 50  0001 C CNN
@@
 $EndComp
 $Comp
-L device:C C23
+L Device:C C?
 U 1 1 5B3248C6
 P 5650 6000
-F 0 "C23" H 5765 6046 50  0000 L CNN
+F 0 "C?" H 5765 6046 50  0000 L CNN
 F 1 "100N" H 5765 5955 50  0000 L CNN
 F 2 "Capacitors_SMD:C_0402" H 5688 5850 50  0001 C CNN
@@
 $EndComp
 $Comp
-L device:C C24
+L Device:C C?
 U 1 1 5B3248F2
 P 6150 6000
-F 0 "C24" H 6265 6046 50  0000 L CNN
+F 0 "C?" H 6265 6046 50  0000 L CNN
 F 1 "100N" H 6265 5955 50  0000 L CNN
 F 2 "Capacitors_SMD:C_0402" H 6188 5850 50  0001 C CNN
@@
 	1    0    0    -1
 $EndComp
-Wire Wire Line
-	4350 6150 3850 6150
-Connection ~ 3850 6150
-Wire Wire Line
-	4350 6150 4800 6150
-Connection ~ 4350 6150
-Wire Wire Line
-	4800 6150 5200 6150
-Wire Wire Line
-	5200 6150 5650 6150
-Connection ~ 4800 6150
-Connection ~ 5200 6150
-Wire Wire Line
-	5650 6150 6150 6150
-Connection ~ 5650 6150
-Wire Wire Line
-	6150 5850 5650 5850
-Wire Wire Line
-	5650 5850 5200 5850
-Connection ~ 5650 5850
-Wire Wire Line
-	5200 5850 4800 5850
-Connection ~ 5200 5850
-Wire Wire Line
-	4800 5850 4350 5850
-Connection ~ 4800 5850
-Wire Wire Line
-	4350 5850 3850 5850
-Connection ~ 4350 5850
 Text Label 8100 5900 2    50   ~ 0
 OSC_IN
@@
 OSC_OUT
 $Comp
-L device:Crystal Y1
+L Device:Crystal Y?
 U 1 1 5B3297A2
 P 8400 5900
-F 0 "Y1" H 8400 6168 50  0000 C CNN
+F 0 "Y?" H 8400 6168 50  0000 C CNN
 F 1 "ABM3-8.000MHZ-D2Y-T" H 8400 6077 50  0000 C CNN
 F 2 "kicad libraries:ABM3-8.000MHZ-D2Y-T" H 8400 5900 50  0001 C CNN
@@
 $EndComp
 $Comp
-L device:C C25
+L Device:C C?
 U 1 1 5B329872
 P 8150 6050
-F 0 "C25" H 7900 6100 50  0000 L CNN
+F 0 "C?" H 7900 6100 50  0000 L CNN
 F 1 "18P" H 7900 6000 50  0000 L CNN
 F 2 "Capacitors_SMD:C_0402" H 8188 5900 50  0001 C CNN
@@
 	1    0    0    -1
 $EndComp
-Wire Wire Line
-	8100 5900 8150 5900
-Wire Wire Line
-	8150 5900 8250 5900
-Connection ~ 8150 5900
-$Comp
-L device:C C26
+$Comp
+L Device:C C?
 U 1 1 5B32AB55
 P 8650 6050
-F 0 "C26" H 8765 6096 50  0000 L CNN
+F 0 "C?" H 8765 6096 50  0000 L CNN
 F 1 "18P" H 8765 6005 50  0000 L CNN
 F 2 "Capacitors_SMD:C_0402" H 8688 5900 50  0001 C CNN
@@
 $EndComp
 Wire Wire Line
-	8550 5900 8650 5900
-Wire Wire Line
-	8750 5900 8650 5900
-Connection ~ 8650 5900
-Wire Wire Line
 	8150 6200 8150 6250
 Wire Wire Line
 	8650 6250 8650 6200
 $Comp
-L conn:Conn_01x06 J4
+L Connector_Generic:Conn_01x06 J?
 U 1 1 5B334DD4
 P 1400 6050
-F 0 "J4" H 1320 6467 50  0000 C CNN
+F 0 "J?" H 1320 6467 50  0000 C CNN
 F 1 "SWD_PROG_HEADER" H 1320 6376 50  0000 C CNN
 F 2 "Pin_Headers:Pin_Header_Straight_1x06_Pitch2.54mm" H 1400 6050 50  0001 C CNN
@@
 $EndComp
 $Comp
-L power:+5V #PWR0113
+L power:+5V #PWR?
 U 1 1 5B334DDB
 P 2000 5750
-F 0 "#PWR0113" H 2000 5600 50  0001 C CNN
+F 0 "#PWR?" H 2000 5600 50  0001 C CNN
 F 1 "+5V" H 2015 5923 50  0000 C CNN
 F 2 "" H 2000 5750 50  0001 C CNN
@@
 	1600 6050 2000 6050
 $Comp
-L device:C C27
+L Device:C C?
 U 1 1 5B3391D6
 P 3450 6000
-F 0 "C27" H 3565 6046 50  0000 L CNN
+F 0 "C?" H 3565 6046 50  0000 L CNN
 F 1 "10U" H 3565 5955 50  0000 L CNN
 F 2 "Capacitors_SMD:C_0805" H 3488 5850 50  0001 C CNN
@@
 	1    0    0    -1
 $EndComp
-Wire Wire Line
-	3350 5850 3450 5850
-Wire Wire Line
-	3450 5850 3850 5850
-Connection ~ 3450 5850
-Connection ~ 3850 5850
-Wire Wire Line
-	3850 6150 3450 6150
 Text HLabel 10200 2000 2    50   Output ~ 0
 MOSI
@@
 Wire Wire Line
 	3450 6250 3450 6150
-Connection ~ 3450 6150
 Text HLabel 5500 4900 0    50   Input ~ 0
 GND
@@
 GND
 $Comp
-L stm32:STM32F446RETx U3
+L stm32:STM32F446RETx U?
 U 1 1 5B3B9C8D
 P 5700 2900
-F 0 "U3" H 9550 4950 50  0000 C CNN
+F 0 "U?" H 9550 4950 50  0000 C CNN
 F 1 "STM32F446RETx" H 9800 4850 50  0000 C CNN
 F 2 "Housings_QFP:LQFP-64_10x10mm_Pitch0.5mm" H 10100 4775 50  0001 R TNN
@@
 Wire Wire Line
 	10200 2500 10850 2500
+Wire Wire Line
+	8100 5900 8150 5900
+Wire Wire Line
+	8550 5900 8650 5900
+Wire Wire Line
+	3450 6150 3850 6150
+Wire Wire Line
+	3350 5850 3450 5850
+Connection ~ 8150 5900
+Wire Wire Line
+	8150 5900 8250 5900
+Connection ~ 8650 5900
+Wire Wire Line
+	8650 5900 8750 5900
+Connection ~ 3450 5850
+Wire Wire Line
+	3450 5850 3850 5850
+Connection ~ 3450 6150
+Connection ~ 3850 5850
+Wire Wire Line
+	3850 5850 4350 5850
+Connection ~ 3850 6150
+Wire Wire Line
+	3850 6150 4350 6150
+Connection ~ 4350 5850
+Wire Wire Line
+	4350 5850 4800 5850
+Connection ~ 4350 6150
+Wire Wire Line
+	4350 6150 4800 6150
+Connection ~ 4800 5850
+Wire Wire Line
+	4800 5850 5200 5850
+Connection ~ 4800 6150
+Wire Wire Line
+	4800 6150 5200 6150
+Connection ~ 5200 5850
+Wire Wire Line
+	5200 5850 5650 5850
+Connection ~ 5200 6150
+Wire Wire Line
+	5200 6150 5650 6150
+Connection ~ 5650 5850
+Wire Wire Line
+	5650 5850 6150 5850
+Connection ~ 5650 6150
+Wire Wire Line
+	5650 6150 6150 6150
 $EndSCHEMATC

Commit message: updated stm32f446rex schematic, normalized
Parts:
- removed C? (x4): 100N, Capacitors_SMD:C_0402, symbol Device:C
- removed C? (x2): 18P, Capacitors_SMD:C_0402, symbol Device:C
- removed Y?: ABM3-8.000MHZ-D2Y-T, kicad libraries:ABM3-8.000MHZ-D2Y-T, symbol Device:Crystal
- added C?: 10N, Capacitor_SMD:C_0402_1005Metric, symbol Device:C_Small
- added C? (x4): 100N, Capacitor_SMD:C_0402_1005Metric, symbol Device:C
- added NT? (x2): Net-Tie_2, symbol Device:Net-Tie_2
- C?: footprint Capacitors_SMD:C_0402 -> Capacitor_SMD:C_0805_2012Metric
- C? (x2): footprint Capacitors_SMD:C_0805 -> Capacitor_SMD:C_0805_2012Metric
- C?: footprint Capacitors_SMD:C_0402 -> Capacitor_SMD:C_0402_1005Metric
- J?: footprint Pin_Headers:Pin_Header_Straight_1x06_Pitch2.54mm -> Connector_PinHeader_2.54mm:PinHeader_1x06_P2.54mm_Vertical
- U?: footprint Housings_QFP:LQFP-64_10x10mm_Pitch0.5mm -> Package_QFP:LQFP-64_10x10mm_P0.5mm
Connections:
- net labels added: VBAT, VCC, V_USB
- net labels removed: +5V, CLK, D+, D-, D_+, D_-, MISO, MOSI, RX, TX, VBUS, ~CS~_ADC, ~CS~_EEPROM, ~DATA_READY~, ~RESET~_ADC
- wire segments 49 -> 98
- no-connect marks 35 -> 0
Other:
- moved on the sheet: C?

Commit message: fixes, updates, new things for datlogger v2
Parts:
- removed NT? (x2): Net-Tie_2, symbol Device:Net-Tie_2
- removed U?: STM32F446RETx, Package_QFP:LQFP-64_10x10mm_P0.5mm, symbol stm32:STM32F446RETx
- added U?: STM32F446RCTx, Package_QFP:LQFP-64_10x10mm_P0.5mm, symbol MCU_ST_STM32F4:STM32F446RCTx
Connections:
- net labels added: VCAP1
- wire segments 98 -> 106
Changed lines of the file:
@@
 EESchema Schematic File Version 4
-LIBS:main-cache
-EELAYER 26 0
+EELAYER 30 0
 EELAYER END
 $Descr A4 11693 8268
 encoding utf-8
-Sheet 2 8
+Sheet 12 13
 Title ""
 Date ""
@@
 Comment4 ""
 $EndDescr
-Text Label 1200 3000 2    50   ~ 0
+Text Label 4400 2800 0    50   ~ 0
 OSC_IN
-Text Label 1200 3100 2    50   ~ 0
+Text Label 4400 2900 0    50   ~ 0
 OSC_OUT
 Wire Wire Line
-	5500 5400 5500 5500
-Wire Wire Line
-	5500 5500 5600 5500
-Wire Wire Line
-	5600 5500 5600 5400
-Wire Wire Line
-	5600 5500 5700 5500
-Wire Wire Line
-	5700 5500 5700 5400
-Connection ~ 5600 5500
-Wire Wire Line
-	5700 5500 5800 5500
-Wire Wire Line
-	5800 5500 5800 5400
-Connection ~ 5700 5500
-Wire Wire Line
-	5900 5600 5900 5400
-Text HLabel 1200 2300 0    50   Input ~ 0
+	5400 5000 5400 5100
+Wire Wire Line
+	5400 5100 5500 5100
+Wire Wire Line
+	5500 5100 5500 5000
+Wire Wire Line
+	5500 5100 5600 5100
+Wire Wire Line
+	5600 5100 5600 5000
+Connection ~ 5500 5100
+Wire Wire Line
+	5600 5100 5700 5100
+Wire Wire Line
+	5700 5100 5700 5000
+Connection ~ 5600 5100
+Text HLabel 5300 1400 0    50   Input ~ 0
 VBAT
 $Comp
@@
 	800  2400 1200 2400
 Wire Wire Line
-	5400 1400 5500 1400
+	5500 1250 5500 1400
 Wire Wire Line
 	5500 1400 5500 1500
@@
 Text Label 10550 3200 2    50   ~ 0
 SWDIO
-Text Label 1200 1900 2    50   ~ 0
+Text Label 1200 1900 0    50   ~ 0
 ~RST~
 Text HLabel 1700 6300 2    50   Input ~ 0
@@
 Wire Wire Line
 	3600 7100 3700 7100
-Text HLabel 5500 5500 0    50   Input ~ 0
+Text HLabel 5400 5100 0    50   Input ~ 0
 GND
 Text HLabel 750  2750 0    50   Input ~ 0
 GND
-Text HLabel 1200 2100 0    50   Input ~ 0
-GND
-$Comp
-L stm32:STM32F446RETx U?
-U 1 1 5B3B9C8D
-P 5700 3500
-F 0 "U?" H 9550 5550 50  0000 C CNN
-F 1 "STM32F446RETx" H 9800 5450 50  0000 C CNN
-F 2 "Package_QFP:LQFP-64_10x10mm_P0.5mm" H 10100 5375 50  0001 R TNN
-F 3 "http://www.st.com/st-web-ui/static/active/en/resource/technical/document/datasheet/DM00141306.pdf" H 5700 3500 50  0001 C CNN
-	1    5700 3500
-	1    0    0    -1
-$EndComp
+Text HLabel 2250 2400 0    50   Input ~ 0
+GND
 Wire Wire Line
 	3700 7100 4100 7100
@@
 Text Label 10550 3400 2    50   ~ 0
 SWO
-Text HLabel 5400 1400 0    50   Input ~ 0
+Text HLabel 5300 1250 0    50   Input ~ 0
 VCC
 Wire Wire Line
@@
 U 5C241710
 F0 "crystal" 50
-F1 "../subs/24MHz_4pin.sch" 50
+F1 "../subs/../subs/24MHz_4pin.sch" 50
 F2 "GND" I L 1050 7400 50
 F3 "OSC_IN" I L 1050 7050 50
@@
 	1    0    0    -1
 $EndComp
-$Comp
-L Device:Net-Tie_2 NT?
-U 1 1 5C25AB07
-P 5800 5600
-F 0 "NT?" H 5800 5778 50  0000 C CNN
-F 1 "Net-Tie_2" H 5800 5687 50  0000 C CNN
-F 2 "" H 5800 5600 50  0001 C CNN
-F 3 "~" H 5800 5600 50  0001 C CNN
-	1    5800 5600
-	1    0    0    1
-$EndComp
-$Comp
-L Device:Net-Tie_2 NT?
-U 1 1 5C25AC41
-P 5800 1300
-F 0 "NT?" H 5800 1478 50  0000 C CNN
-F 1 "Net-Tie_2" H 5800 1387 50  0000 C CNN
-F 2 "" H 5800 1300 50  0001 C CNN
-F 3 "~" H 5800 1300 50  0001 C CNN
-	1    5800 1300
-	1    0    0    -1
-$EndComp
-Wire Wire Line
-	5900 1300 5900 1500
-Wire Wire Line
-	5700 1300 5700 1400
-Wire Wire Line
-	5700 5600 5700 5500
 Wire Wire Line
 	750  2250 800  2250
@@
 Wire Wire Line
 	1200 5000 850  5000
+$Comp
+L MCU_ST_STM32F4:STM32F446RCTx U?
+U 1 1 5EE908A1
+P 5600 3200
+F 0 "U?" H 6150 4900 50  0000 C CNN
+F 1 "STM32F446RCTx" H 5600 3200 50  0000 C CNN
+F 2 "Package_QFP:LQFP-64_10x10mm_P0.5mm" H 5000 1500 50  0001 R CNN
+F 3 "http://www.st.com/st-web-ui/static/active/en/resource/technical/document/datasheet/DM00141306.pdf" H 5600 3200 50  0001 C CNN
+	1    5600 3200
+	1    0    0    -1
+$EndComp
+Wire Wire Line
+	5700 5100 5800 5100
+Wire Wire Line
+	5800 5100 5800 5000
+Connection ~ 5700 5100
+Wire Wire Line
+	5800 1400 5900 1400
+Wire Wire Line
+	5900 1400 5900 1500
+Connection ~ 5800 1400
+Wire Wire Line
+	5500 1250 5300 1250
+Wire Wire Line
+	5300 1400 5400 1400
+Wire Wire Line
+	5400 1400 5400 1500
+Text Label 4400 1700 0    50   ~ 0
+~RST~
+Wire Wire Line
+	4400 1700 4900 1700
+Text Label 1200 2400 0    50   ~ 0
+VCAP1
+Text Label 4400 2100 0    50   ~ 0
+VCAP1
+Wire Wire Line
+	4400 2100 4900 2100
+$Sheet
+S 2750 5350 1000 550
+U 5EECCCAE
+F0 "sheet5EECCCAE" 50
+F1 "../subs/../subs/24MHz_4pin.sch" 50
+F2 "GND" I L 2750 5800 50
+F3 "OSC_IN" I L 2750 5450 50
+F4 "OSC_OUT" O L 2750 5550 50
+$EndSheet
+Text Label 2300 5450 0    50   ~ 0
+OSC_IN
+Text Label 2300 5550 0    50   ~ 0
+OSC_OUT
+Text HLabel 2500 5800 0    50   Input ~ 0
+GND
+Wire Wire Line
+	2300 5450 2750 5450
+Wire Wire Line
+	2500 5800 2750 5800
+Wire Wire Line
+	2300 5550 2750 5550
 $EndSCHEMATC

Commit message: parts for grease board &displays
Changed lines of the file:
@@
 U 5C241710
 F0 "crystal" 50
-F1 "../subs/../subs/24MHz_4pin.sch" 50
+F1 "../subs/../subs/../subs/24MHz_4pin.sch" 50
 F2 "GND" I L 1050 7400 50
 F3 "OSC_IN" I L 1050 7050 50
@@
 U 5EECCCAE
 F0 "sheet5EECCCAE" 50
-F1 "../subs/../subs/24MHz_4pin.sch" 50
+F1 "../subs/../subs/../subs/24MHz_4pin.sch" 50
 F2 "GND" I L 2750 5800 50
 F3 "OSC_IN" I L 2750 5450 50
