File: debounce_3V3.sch (KiCad schematic (older format))
At the start: 3 parts

Commit message: updating
Changed lines of the file:
@@
 $Descr A4 11693 8268
 encoding utf-8
-Sheet 10 14
+Sheet 10 18
 Title ""
 Date ""
@@
 AR Path="/5BF0DB73/5C4840A6/5BEFC0B0" Ref="R19"  Part="1"
 AR Path="/5BF0DB73/5C485D0D/5BEFC0B0" Ref="R21"  Part="1"
-F 0 "R19" H 3532 3046 50  0000 R CNN
+F 0 "R21" H 3532 3046 50  0000 R CNN
 F 1 "6.8K" H 3532 2955 50  0000 R CNN
 F 2 "Resistor_SMD:R_0603_1608Metric" V 3640 2990 50  0001 C CNN
@@
 AR Path="/5BF0DB73/5C4840A6/5BEFC134" Ref="R20"  Part="1"
 AR Path="/5BF0DB73/5C485D0D/5BEFC134" Ref="R22"  Part="1"
-F 0 "R20" V 3900 3150 50  0000 C CNN
+F 0 "R22" V 3900 3150 50  0000 C CNN
 F 1 "15K" V 3900 3350 50  0000 C CNN
 F 2 "Resistor_SMD:R_0603_1608Metric" V 4040 3240 50  0001 C CNN
@@
 AR Path="/5BF0DB73/5C4840A6/5BEFC1B8" Ref="C13"  Part="1"
 AR Path="/5BF0DB73/5C485D0D/5BEFC1B8" Ref="C14"  Part="1"
-F 0 "C13" H 4515 3546 50  0000 L CNN
+F 0 "C14" H 4515 3546 50  0000 L CNN
 F 1 "1U" H 4515 3455 50  0000 L CNN
 F 2 "Capacitor_SMD:C_0603_1608Metric" H 4438 3350 50  0001 C CNN

Commit message: some changes
Parts:
- R15: value 6.8K -> 6K8; symbol Device:R_US -> Device:R
- R16: symbol Device:R_US -> Device:R
Changed lines of the file:
@@
 $Descr A4 11693 8268
 encoding utf-8
-Sheet 10 18
+Sheet 7 24
 Title ""
 Date ""
@@
 SW-
 $Comp
-L Device:R_US R15
+L Device:R R15
 U 1 1 5BEFC0B0
 P 3600 3000
@@
 AR Path="/5BF0DB73/5C485D0D/5BEFC0B0" Ref="R21"  Part="1"
 F 0 "R21" H 3532 3046 50  0000 R CNN
-F 1 "6.8K" H 3532 2955 50  0000 R CNN
+F 1 "6K8" H 3532 2955 50  0000 R CNN
 F 2 "Resistor_SMD:R_0603_1608Metric" V 3640 2990 50  0001 C CNN
 F 3 "~" H 3600 3000 50  0001 C CNN
@@
 $EndComp
 $Comp
-L Device:R_US R16
+L Device:R R16
 U 1 1 5BEFC134
 P 4000 3250

Commit message: stm32f405 for lora
Changed lines of the file:
@@
 EESchema Schematic File Version 4
-LIBS:main-cache
-EELAYER 29 0
+EELAYER 30 0
 EELAYER END
 $Descr A4 11693 8268
 encoding utf-8
-Sheet 7 23
+Sheet 12 14
 Title ""
 Date ""
@@
 AR Path="/5BF0DB73/5C4840A6/5BEFC0B0" Ref="R19"  Part="1"
 AR Path="/5BF0DB73/5C485D0D/5BEFC0B0" Ref="R21"  Part="1"
-F 0 "R21" H 3532 3046 50  0000 R CNN
+AR Path="/5FCF2B04/5FD83231/5C4840A6/5BEFC0B0" Ref="R18"  Part="1"
+AR Path="/5FCF2B04/5FD83231/5C485D0D/5BEFC0B0" Ref="R20"  Part="1"
+F 0 "R20" H 3532 3046 50  0000 R CNN
 F 1 "6K8" H 3532 2955 50  0000 R CNN
 F 2 "Resistor_SMD:R_0603_1608Metric" V 3640 2990 50  0001 C CNN
@@
 AR Path="/5BF0DB73/5C4840A6/5BEFC134" Ref="R20"  Part="1"
 AR Path="/5BF0DB73/5C485D0D/5BEFC134" Ref="R22"  Part="1"
-F 0 "R22" V 3900 3150 50  0000 C CNN
+AR Path="/5FCF2B04/5FD83231/5C4840A6/5BEFC134" Ref="R19"  Part="1"
+AR Path="/5FCF2B04/5FD83231/5C485D0D/5BEFC134" Ref="R21"  Part="1"
+F 0 "R21" V 3900 3150 50  0000 C CNN
 F 1 "15K" V 3900 3350 50  0000 C CNN
 F 2 "Resistor_SMD:R_0603_1608Metric" V 4040 3240 50  0001 C CNN
@@
 AR Path="/5BF0DB73/5C4840A6/5BEFC1B8" Ref="C13"  Part="1"
 AR Path="/5BF0DB73/5C485D0D/5BEFC1B8" Ref="C14"  Part="1"
-F 0 "C14" H 4515 3546 50  0000 L CNN
+AR Path="/5FCF2B04/5FD83231/5C4840A6/5BEFC1B8" Ref="C25"  Part="1"
+AR Path="/5FCF2B04/5FD83231/5C485D0D/5BEFC1B8" Ref="C26"  Part="1"
+F 0 "C26" H 4515 3546 50  0000 L CNN
 F 1 "1U" H 4515 3455 50  0000 L CNN
 F 2 "Capacitor_SMD:C_0603_1608Metric" H 4438 3350 50  0001 C CNN
