File: 12V_polarity_protection.sch (KiCad schematic (older format))
At the start: 2 parts, among them Q1 SI7615ADN-T1-GE3

Commit message: adding milad subs
Parts:
- renumbered R3 to R4
Changed lines of the file:
@@
 $Descr A4 11693 8268
 encoding utf-8
-Sheet 3 6
+Sheet 3 10
 Title ""
 Date ""
@@
 	3900 2500 4350 2500
 $Comp
-L Device:R R3
+L Device:R R4
 U 1 1 5F76696E
 P 4550 3000
-F 0 "R3" H 4620 3046 50  0000 L CNN
+F 0 "R4" H 4620 3046 50  0000 L CNN
 F 1 "10K" H 4620 2955 50  0000 L CNN
 F 2 "Resistor_SMD:R_0603_1608Metric" V 4480 3000 50  0001 C CNN

Commit message: polarity protection updated
Parts:
- Q1: MPN (none) -> SI7615ADN-T1-GE3
Changed lines of the file:
@@
 F 2 "Package_SO:Vishay_PowerPAK_1212-8_Single" H 4750 2700 50  0001 C CNN
 F 3 "https://www.vishay.com/docs/62667/si7615adn.pdf" H 4550 2600 50  0001 C CNN
+F 4 "SI7615ADN-T1-GE3" V 4550 2600 50  0001 C CNN "MPN"
 	1    4550 2600
 	0    -1   -1   0

Commit message: chevelle adds
Parts:
- removed Q1: SI7615ADN-T1-GE3, Package_SO:Vishay_PowerPAK_1212-8_Single, symbol william_fets:SI7615ADN-T1-GE3
- removed R4: 10K, Resistor_SMD:R_0603_1608Metric, symbol Device:R
- added C?: 2U2, Capacitor_SMD:C_0805_2012Metric, symbol Device:C
- added D?: SMBJ22CAQ-13-F, Diode_SMD:D_SMB, symbol Device:D_TVS
- added Q?: AON7524, william_mosfet:AlphaOmega_DFN-8_EP_3x3mm_0.65pitch_1.75x2.35mmEP, symbol william_fets:AON7524
- added U?: LM74610, Package_SO:SSOP-8_2.95x2.8mm_P0.65mm, symbol william_batteries:LM74610
Connections:
- wire segments 5 -> 13
Changed lines of the file:
@@
 $Descr A4 11693 8268
 encoding utf-8
-Sheet 3 10
+Sheet 9 10
 Title ""
 Date ""
@@
 Comment4 ""
 $EndDescr
-$Comp
-L william_fets:SI7615ADN-T1-GE3 Q?
-U 1 1 5F75C8D6
-P 4550 2600
-AR Path="/5F75C8D6" Ref="Q?"  Part="1"
-AR Path="/5F75BE24/5F75C8D6" Ref="Q1"  Part="1"
-F 0 "Q1" V 4892 2600 50  0000 C CNN
-F 1 "SI7615ADN-T1-GE3" V 4801 2600 50  0000 C CNN
-F 2 "Package_SO:Vishay_PowerPAK_1212-8_Single" H 4750 2700 50  0001 C CNN
-F 3 "https://www.vishay.com/docs/62667/si7615adn.pdf" H 4550 2600 50  0001 C CNN
-F 4 "SI7615ADN-T1-GE3" V 4550 2600 50  0001 C CNN "MPN"
-	1    4550 2600
-	0    -1   -1   0
-$EndComp
 Text HLabel 3900 2500 0    50   Input ~ 0
 VIN
-Text HLabel 3900 3300 0    50   Input ~ 0
-GND
 Text HLabel 5200 2500 2    50   Input ~ 0
 VPROT
 Wire Wire Line
-	4750 2500 5200 2500
+	4750 2500 5100 2500
 Wire Wire Line
 	4550 2800 4550 2850
 Wire Wire Line
-	4550 3300 3900 3300
-Wire Wire Line
-	3900 2500 4350 2500
+	3900 2500 3950 2500
+Text Notes 5000 1950 0    50   ~ 0
+Rds_on = appx 9mΩ @ -3V Vgs
 $Comp
-L Device:R R4
-U 1 1 5F76696E
-P 4550 3000
-F 0 "R4" H 4620 3046 50  0000 L CNN
-F 1 "10K" H 4620 2955 50  0000 L CNN
-F 2 "Resistor_SMD:R_0603_1608Metric" V 4480 3000 50  0001 C CNN
-F 3 "~" H 4550 3000 50  0001 C CNN
-	1    4550 3000
+L william_batteries:LM74610 U?
+U 1 1 6012E65A
+P 4600 3300
+F 0 "U?" H 4500 2877 50  0000 C CNN
+F 1 "LM74610" H 4500 2786 50  0000 C CNN
+F 2 "Package_SO:SSOP-8_2.95x2.8mm_P0.65mm" H 4600 3300 50  0001 C CNN
+F 3 "https://www.ti.com/lit/ds/symlink/lm74610-q1.pdf?ts=1607451864730&ref_url=https%253A%252F%252Fwww.ti.com%252Fproduct%252FLM74610-Q1" H 4600 3300 50  0001 C CNN
+	1    4600 3300
 	1    0    0    -1
 $EndComp
+$Comp
+L william_fets:AON7524 Q?
+U 1 1 6012ED64
+P 4550 2600
+F 0 "Q?" V 4893 2600 50  0000 C CNN
+F 1 "AON7524" V 4802 2600 50  0000 C CNN
+F 2 "william_mosfet:AlphaOmega_DFN-8_EP_3x3mm_0.65pitch_1.75x2.35mmEP" H 4400 2800 50  0001 C CNN
+F 3 "http://aosmd.com/res/data_sheets/AON7524.pdf" H 4550 2600 50  0001 C CNN
+	1    4550 2600
+	0    1    -1   0
+$EndComp
 Wire Wire Line
-	4550 3150 4550 3300
-Text Notes 5000 1950 0    50   ~ 0
-Rds_on = appx 9mΩ @ -3V Vgs
+	4100 3050 4100 2500
+Connection ~ 4100 2500
+Wire Wire Line
+	4100 2500 4350 2500
+Wire Wire Line
+	5100 3050 5100 2500
+Connection ~ 5100 2500
+Wire Wire Line
+	5100 2500 5200 2500
+Wire Wire Line
+	4650 2850 4650 2800
+Wire Wire Line
+	4650 2800 4550 2800
+Connection ~ 4550 2800
+$Comp
+L Device:C C?
+U 1 1 60132667
+P 5100 3400
+F 0 "C?" H 5215 3446 50  0000 L CNN
+F 1 "2U2" H 5215 3355 50  0000 L CNN
+F 2 "Capacitor_SMD:C_0805_2012Metric" H 5138 3250 50  0001 C CNN
+F 3 "~" H 5100 3400 50  0001 C CNN
+	1    5100 3400
+	1    0    0    -1
+$EndComp
+$Comp
+L Device:D_TVS D?
+U 1 1 6013F73A
+P 3950 3100
+F 0 "D?" V 3996 3020 50  0000 R CNN
+F 1 "SMBJ22CAQ-13-F" V 3905 3020 50  0000 R CNN
+F 2 "Diode_SMD:D_SMB" H 3950 3100 50  0001 C CNN
+F 3 "~" H 3950 3100 50  0001 C CNN
+F 4 "SMBJ22CAQ-13-F" V 3950 3100 50  0001 C CNN "MPN"
+	1    3950 3100
+	0    1    -1   0
+$EndComp
+Text HLabel 3850 3500 0    50   Input ~ 0
+GND
+Wire Wire Line
+	3950 2950 3950 2500
+Connection ~ 3950 2500
+Wire Wire Line
+	3950 2500 4100 2500
+Wire Wire Line
+	3950 3250 3950 3500
+Wire Wire Line
+	3950 3500 3850 3500
 $EndSCHEMATC
