File: 3V3_atmega32u4.sch (KiCad schematic (older format))
At the start: 17 parts, among them J8 AVR-ISP-6, U2 ATmega32U4-AU, Y1 NX5032GA-8MHZ-EXS00A-CG07039

Commit message: changed max schematics
Parts:
- removed C3: 100N, Capacitor_SMD:C_0603_1608Metric, symbol Device:C
Connections:
- wire segments 104 -> 99
- no-connect marks 0 -> 1
Changed lines of the file:
@@
-EESchema Schematic File Version 5
-EELAYER 31 0
+EESchema Schematic File Version 4
+EELAYER 30 0
 EELAYER END
 $Descr A4 11693 8268
 encoding utf-8
-Sheet 6 7
+Sheet 5 10
 Title ""
 Date ""
@@
 Comment3 ""
 Comment4 ""
-Comment5 ""
-Comment6 ""
-Comment7 ""
-Comment8 ""
-Comment9 ""
 $EndDescr
 Connection ~ 7700 1650
@@
 Connection ~ 2400 1100
 Connection ~ 2000 3950
-Connection ~ 2400 2100
 Connection ~ 8100 1150
-Connection ~ 5600 1800
 Connection ~ 8100 1650
 Connection ~ 2450 3350
 Connection ~ 2000 3450
-Connection ~ 2400 2600
 Connection ~ 2400 1500
 Connection ~ 2850 3250
@@
 	2400 1500 2800 1500
 Wire Wire Line
-	2400 2100 2750 2100
-Wire Wire Line
 	2400 2200 2400 2100
 Wire Wire Line
@@
 	2450 3950 2850 3950
 Wire Wire Line
-	2750 2100 2750 2200
-Wire Wire Line
-	2750 2500 2750 2600
-Wire Wire Line
-	2750 2600 2400 2600
-Wire Wire Line
 	2800 1100 2750 1100
 Wire Wire Line
@@
 	4600 4000 4700 4000
 Wire Wire Line
-	4700 1800 5600 1800
-Wire Wire Line
 	4700 2200 5100 2200
 Wire Wire Line
@@
 Wire Wire Line
 	5100 3500 4700 3500
-Wire Wire Line
-	5600 1800 5600 1900
-Wire Wire Line
-	5600 1800 5700 1800
 Wire Wire Line
 	5600 5600 5600 5500
@@
 $EndComp
 $Comp
-L Device:C C3
-U 1 1 5E275A45
-P 2750 2350
-F 0 "C3" H 2865 2396 50  0000 L CNN
-F 1 "100N" H 2865 2305 50  0000 L CNN
-F 2 "Capacitor_SMD:C_0603_1608Metric" H 2788 2200 50  0001 C CNN
-F 3 "~" H 2750 2350 50  0001 C CNN
-	1    2750 2350
-	1    0    0    -1
-$EndComp
-$Comp
 L Device:C C4
 U 1 1 5E2F1C0C
@@
 	1    0    0    -1
 $EndComp
+Text HLabel 4550 3500 0    50   Input ~ 0
+3V3
+Wire Wire Line
+	4550 3500 4700 3500
+Connection ~ 4700 3500
+Wire Wire Line
+	4700 1800 5700 1800
+NoConn ~ 5600 1900
 $EndSCHEMATC

Commit message: chevelle adds
Parts:
- added C3: 100N, Capacitor_SMD:C_0603_1608Metric, symbol Device:C
Connections:
- wire segments 99 -> 104
- no-connect marks 1 -> 0
Changed lines of the file:
@@
 $Descr A4 11693 8268
 encoding utf-8
-Sheet 5 10
+Sheet 7 10
 Title ""
 Date ""
@@
 Comment4 ""
 $EndDescr
+Connection ~ 7700 1150
 Connection ~ 7700 1650
+Connection ~ 5700 1800
+Connection ~ 5600 5600
+Connection ~ 2800 1100
+Connection ~ 2400 1500
+Connection ~ 8100 1650
+Connection ~ 2000 3450
+Connection ~ 2450 3350
+Connection ~ 2850 3250
+Connection ~ 2400 2600
 Connection ~ 2450 3950
 Connection ~ 8550 1650
+Connection ~ 2000 3950
 Connection ~ 2400 1100
-Connection ~ 2000 3950
+Connection ~ 2400 2100
+Connection ~ 5600 1800
 Connection ~ 8100 1150
-Connection ~ 8100 1650
-Connection ~ 2450 3350
-Connection ~ 2000 3450
-Connection ~ 2400 1500
-Connection ~ 2850 3250
-Connection ~ 5700 1800
-Connection ~ 7700 1150
-Connection ~ 2800 1100
-Connection ~ 5600 5600
 Wire Wire Line
 	1750 3250 2850 3250
@@
 	2400 1500 2800 1500
 Wire Wire Line
+	2400 2100 2750 2100
+Wire Wire Line
 	2400 2200 2400 2100
 Wire Wire Line
@@
 	2450 3950 2850 3950
 Wire Wire Line
+	2750 2100 2750 2200
+Wire Wire Line
+	2750 2500 2750 2600
+Wire Wire Line
+	2750 2600 2400 2600
+Wire Wire Line
 	2800 1100 2750 1100
 Wire Wire Line
@@
 	4600 4000 4700 4000
 Wire Wire Line
+	4700 1800 5600 1800
+Wire Wire Line
 	4700 2200 5100 2200
 Wire Wire Line
@@
 Wire Wire Line
 	5100 3500 4700 3500
+Wire Wire Line
+	5600 1800 5600 1900
+Wire Wire Line
+	5600 1800 5700 1800
 Wire Wire Line
 	5600 5600 5600 5500
@@
 U 1 1 5E275587
 P 2400 2350
-F 0 "R7" H 2470 2396 50  0000 L CNN
+AR Path="/5E698B9F/5E275587" Ref="R7"  Part="1"
+AR Path="/5F8D10A3/5F8D1751/5E275587" Ref="R?"  Part="1"
+F 0 "R?" H 2470 2396 50  0000 L CNN
 F 1 "10K" H 2470 2305 50  0000 L CNN
 F 2 "Resistor_SMD:R_0603_1608Metric" V 2330 2350 50  0001 C CNN
@@
 U 1 1 5E2529E7
 P 4900 3200
-F 0 "R8" V 4800 3200 50  0000 C CNN
+AR Path="/5E698B9F/5E2529E7" Ref="R8"  Part="1"
+AR Path="/5F8D10A3/5F8D1751/5E2529E7" Ref="R?"  Part="1"
+F 0 "R?" V 4800 3200 50  0000 C CNN
 F 1 "22R" V 4900 3200 50  0000 C CNN
 F 2 "Resistor_SMD:R_0603_1608Metric" V 4830 3200 50  0001 C CNN
@@
 U 1 1 5E253B05
 P 4900 3300
-F 0 "R9" V 4800 3300 50  0000 C CNN
+AR Path="/5E698B9F/5E253B05" Ref="R9"  Part="1"
+AR Path="/5F8D10A3/5F8D1751/5E253B05" Ref="R?"  Part="1"
+F 0 "R?" V 4800 3300 50  0000 C CNN
 F 1 "22R" V 4900 3300 50  0000 C CNN
 F 2 "Resistor_SMD:R_0603_1608Metric" V 4830 3300 50  0001 C CNN
@@
 U 1 1 5E287281
 P 2000 3700
-F 0 "D1" V 1954 3779 50  0000 L CNN
+AR Path="/5E698B9F/5E287281" Ref="D1"  Part="1"
+AR Path="/5F8D10A3/5F8D1751/5E287281" Ref="D?"  Part="1"
+F 0 "D?" V 1954 3779 50  0000 L CNN
 F 1 "ESD9B5.0ST5G" H 1850 3600 50  0000 L CNN
 F 2 "william_diode:D_SOD-923" H 2000 3700 50  0001 C CNN
@@
 U 1 1 5E2C94B3
 P 2450 3700
-F 0 "D2" V 2404 3779 50  0000 L CNN
+AR Path="/5E698B9F/5E2C94B3" Ref="D2"  Part="1"
+AR Path="/5F8D10A3/5F8D1751/5E2C94B3" Ref="D?"  Part="1"
+F 0 "D?" V 2404 3779 50  0000 L CNN
 F 1 "ESD9B5.0ST5G" H 2300 3600 50  0000 L CNN
 F 2 "william_diode:D_SOD-923" H 2450 3700 50  0001 C CNN
@@
 U 1 1 5E2CCF8B
 P 2850 3700
-F 0 "D3" V 2804 3779 50  0000 L CNN
+AR Path="/5E698B9F/5E2CCF8B" Ref="D3"  Part="1"
+AR Path="/5F8D10A3/5F8D1751/5E2CCF8B" Ref="D?"  Part="1"
+F 0 "D?" V 2804 3779 50  0000 L CNN
 F 1 "ESD9B5.0ST5G" H 2700 3600 50  0000 L CNN
 F 2 "william_diode:D_SOD-923" H 2850 3700 50  0001 C CNN
@@
 U 1 1 5E2F1167
 P 2400 1250
-F 0 "C2" H 2286 1204 50  0000 R CNN
+AR Path="/5E698B9F/5E2F1167" Ref="C2"  Part="1"
+AR Path="/5F8D10A3/5F8D1751/5E2F1167" Ref="C?"  Part="1"
+F 0 "C?" H 2286 1204 50  0000 R CNN
 F 1 "27P" H 2286 1295 50  0000 R CNN
 F 2 "Capacitor_SMD:C_0402_1005Metric" H 2438 1100 50  0001 C CNN
@@
 $EndComp
 $Comp
+L Device:C C3
+U 1 1 5E275A45
+P 2750 2350
+AR Path="/5E698B9F/5E275A45" Ref="C3"  Part="1"
+AR Path="/5F8D10A3/5F8D1751/5E275A45" Ref="C?"  Part="1"
+F 0 "C?" H 2865 2396 50  0000 L CNN
+F 1 "100N" H 2865 2305 50  0000 L CNN
+F 2 "Capacitor_SMD:C_0603_1608Metric" H 2788 2200 50  0001 C CNN
+F 3 "~" H 2750 2350 50  0001 C CNN
+	1    2750 2350
+	1    0    0    -1
+$EndComp
+$Comp
 L Device:C C4
 U 1 1 5E2F1C0C
 P 2800 1250
-F 0 "C4" H 2685 1296 50  0000 R CNN
+AR Path="/5E698B9F/5E2F1C0C" Ref="C4"  Part="1"
+AR Path="/5F8D10A3/5F8D1751/5E2F1C0C" Ref="C?"  Part="1"
+F 0 "C?" H 2685 1296 50  0000 R CNN
 F 1 "27P" H 2685 1205 50  0000 R CNN
 F 2 "Capacitor_SMD:C_0402_1005Metric" H 2838 1100 50  0001 C CNN
@@
 U 1 1 5E203FED
 P 4700 3750
-F 0 "C5" H 4815 3796 50  0000 L CNN
+AR Path="/5E698B9F/5E203FED" Ref="C5"  Part="1"
+AR Path="/5F8D10A3/5F8D1751/5E203FED" Ref="C?"  Part="1"
+F 0 "C?" H 4815 3796 50  0000 L CNN
 F 1 "1U" H 4815 3705 50  0000 L CNN
 F 2 "Capacitor_SMD:C_0603_1608Metric" H 4738 3600 50  0001 C CNN
@@
 U 1 1 5E1FFDB7
 P 7700 1400
-F 0 "C6" H 7815 1446 50  0000 L CNN
+AR Path="/5E698B9F/5E1FFDB7" Ref="C6"  Part="1"
+AR Path="/5F8D10A3/5F8D1751/5E1FFDB7" Ref="C?"  Part="1"
+F 0 "C?" H 7815 1446 50  0000 L CNN
 F 1 "10U" H 7815 1355 50  0000 L CNN
 F 2 "Capacitor_SMD:C_0805_2012Metric" H 7738 1250 50  0001 C CNN
@@
 U 1 1 5E200B40
 P 8100 1400
-F 0 "C7" H 8215 1446 50  0000 L CNN
+AR Path="/5E698B9F/5E200B40" Ref="C7"  Part="1"
+AR Path="/5F8D10A3/5F8D1751/5E200B40" Ref="C?"  Part="1"
+F 0 "C?" H 8215 1446 50  0000 L CNN
 F 1 "100N" H 8215 1355 50  0000 L CNN
 F 2 "Capacitor_SMD:C_0603_1608Metric" H 8138 1250 50  0001 C CNN
@@
 U 1 1 5E200E50
 P 8550 1400
-F 0 "C8" H 8665 1446 50  0000 L CNN
+AR Path="/5E698B9F/5E200E50" Ref="C8"  Part="1"
+AR Path="/5F8D10A3/5F8D1751/5E200E50" Ref="C?"  Part="1"
+F 0 "C?" H 8665 1446 50  0000 L CNN
 F 1 "100N" H 8665 1355 50  0000 L CNN
 F 2 "Capacitor_SMD:C_0603_1608Metric" H 8588 1250 50  0001 C CNN
@@
 U 1 1 5E2011C6
 P 9200 1400
-F 0 "C9" H 9315 1446 50  0000 L CNN
+AR Path="/5E698B9F/5E2011C6" Ref="C9"  Part="1"
+AR Path="/5F8D10A3/5F8D1751/5E2011C6" Ref="C?"  Part="1"
+F 0 "C?" H 9315 1446 50  0000 L CNN
 F 1 "1U" H 9315 1355 50  0000 L CNN
 F 2 "Capacitor_SMD:C_0603_1608Metric" H 9238 1250 50  0001 C CNN
@@
 U 1 1 5E2F04BD
 P 2600 1100
-F 0 "Y1" H 2600 1368 50  0000 C CNN
+AR Path="/5E698B9F/5E2F04BD" Ref="Y1"  Part="1"
+AR Path="/5F8D10A3/5F8D1751/5E2F04BD" Ref="Y?"  Part="1"
+F 0 "Y?" H 2600 1368 50  0000 C CNN
 F 1 "NX5032GA-8MHZ-EXS00A-CG07039" H 2600 1277 50  0000 C CNN
 F 2 "william_crystal:Crystal_SMD_5032-2Pin_5.0x3.2mm" H 2600 1100 50  0001 C CNN
@@
 AR Path="/5E1A8B1B/5E1FC528/5E2F4893" Ref="J8"  Part="1"
 AR Path="/00000000/5E2F4893" Ref="J8"  Part="1"
-F 0 "J8" H 8620 2796 50  0000 R CNN
+AR Path="/5E698B9F/5E2F4893" Ref="J8"  Part="1"
+AR Path="/5F8D10A3/5F8D1751/5E2F4893" Ref="J?"  Part="1"
+F 0 "J?" H 8620 2796 50  0000 R CNN
 F 1 "AVR-ISP-6" H 8620 2705 50  0000 R CNN
 F 2 "Connector_IDC:IDC-Header_2x03_P2.54mm_Vertical" V 8650 2750 50  0001 C CNN
@@
 AR Path="/5E1A8B1B/5E1FC528/5E1FCA92" Ref="U2"  Part="1"
 AR Path="/00000000/5E1FCA92" Ref="U2"  Part="1"
-F 0 "U2" H 6150 5450 50  0000 C CNN
+AR Path="/5E698B9F/5E1FCA92" Ref="U2"  Part="1"
+AR Path="/5F8D10A3/5F8D1751/5E1FCA92" Ref="U?"  Part="1"
+F 0 "U?" H 6150 5450 50  0000 C CNN
 F 1 "ATmega32U4-AU" H 5600 3600 50  0000 C CNN
 F 2 "Package_QFP:TQFP-44_10x10mm_P0.8mm" H 5700 3700 50  0001 C CIN
@@
 	1    0    0    -1
 $EndComp
-Text HLabel 4550 3500 0    50   Input ~ 0
-3V3
-Wire Wire Line
-	4550 3500 4700 3500
-Connection ~ 4700 3500
-Wire Wire Line
-	4700 1800 5700 1800
-NoConn ~ 5600 1900
 $EndSCHEMATC
