File: stspin220.sch (KiCad schematic (older format))
At the start: 13 parts, among them U3 STSPIN220

Commit message: adding milad subs
Parts:
- removed R6: 0R2, symbol Device:R
- added R11: 0R2, Resistor_SMD:R_1020_2550Metric, symbol Device:R
- C3: footprint (none) -> Capacitor_SMD:C_0603_1608Metric
- C4: renamed from C?; footprint (none) -> Capacitor_SMD:C_0603_1608Metric
- C5: renamed from C?; footprint (none) -> Capacitor_SMD:C_0805_2012Metric
- C6: renamed from C?; footprint (none) -> Capacitor_THT:CP_Radial_D6.3mm_P2.50mm
- R10: renamed from R5; footprint (none) -> Resistor_SMD:R_1020_2550Metric; MPN (none) -> RCWE1020R200FKEA
- R5, R6, R7, R8: renamed from R?; footprint (none) -> Resistor_SMD:R_0603_1608Metric
- R9: renamed from R4; footprint (none) -> Resistor_SMD:R_0603_1608Metric
- RV1: renamed from RV?; footprint (none) -> william_potentiometer:Potentiometer_Bourns_TC33X_Vertical; MPN (none) -> TC33X-2-104E
- renumbered U3 to U2
Changed lines of the file:
@@
 $Descr A4 11693 8268
 encoding utf-8
-Sheet 4 6
+Sheet 4 10
 Title ""
 Date ""
@@
 $EndDescr
 $Comp
-L Driver_Motor:STSPIN220 U3
+L Driver_Motor:STSPIN220 U2
 U 1 1 5F76C969
 P 6400 2950
-F 0 "U3" H 6800 3700 50  0000 C CNN
+F 0 "U2" H 6800 3700 50  0000 C CNN
 F 1 "STSPIN220" H 6700 3600 50  0000 C CNN
 F 2 "Package_DFN_QFN:VQFN-16-1EP_3x3mm_P0.5mm_EP1.8x1.8mm" H 6600 3700 50  0001 L CNN
@@
 VMOT
 $Comp
-L Device:R R5
+L Device:R R10
 U 1 1 5F76E303
 P 7350 5400
-F 0 "R5" H 7420 5446 50  0000 L CNN
+F 0 "R10" H 7420 5446 50  0000 L CNN
 F 1 "0R2" H 7420 5355 50  0000 L CNN
-F 2 "" V 7280 5400 50  0001 C CNN
+F 2 "Resistor_SMD:R_1020_2550Metric" V 7280 5400 50  0001 C CNN
 F 3 "~" H 7350 5400 50  0001 C CNN
+F 4 "RCWE1020R200FKEA" H 7350 5400 50  0001 C CNN "MPN"
 	1    7350 5400
-	1    0    0    -1
-$EndComp
-$Comp
-L Device:R R6
-U 1 1 5F76E44D
-P 7750 5400
-F 0 "R6" H 7820 5446 50  0000 L CNN
-F 1 "0R2" H 7820 5355 50  0000 L CNN
-F 2 "" V 7680 5400 50  0001 C CNN
-F 3 "~" H 7750 5400 50  0001 C CNN
-	1    7750 5400
 	1    0    0    -1
 $EndComp
@@
 F 0 "C3" H 1615 1896 50  0000 L CNN
 F 1 "22N" H 1615 1805 50  0000 L CNN
-F 2 "" H 1538 1700 50  0001 C CNN
+F 2 "Capacitor_SMD:C_0603_1608Metric" H 1538 1700 50  0001 C CNN
 F 3 "~" H 1500 1850 50  0001 C CNN
 	1    1500 1850
@@
 	5650 3450 5900 3450
 $Comp
-L Device:R R4
+L Device:R R9
 U 1 1 5F773161
 P 2050 1700
-F 0 "R4" H 2120 1746 50  0000 L CNN
+F 0 "R9" H 2120 1746 50  0000 L CNN
 F 1 "10K" H 2120 1655 50  0000 L CNN
-F 2 "" V 1980 1700 50  0001 C CNN
+F 2 "Resistor_SMD:R_0603_1608Metric" V 1980 1700 50  0001 C CNN
 F 3 "~" H 2050 1700 50  0001 C CNN
 	1    2050 1700
@@
 $EndComp
 $Comp
-L william_potentiometer:TC33X-2-104E RV?
+L william_potentiometer:TC33X-2-104E RV1
 U 1 1 5F77879D
 P 2050 1400
-F 0 "RV?" H 1980 1446 50  0000 R CNN
+F 0 "RV1" H 1980 1446 50  0000 R CNN
 F 1 "TC33X-2-104E" H 1980 1355 50  0000 R CNN
-F 2 "" H 2050 1400 50  0001 C CNN
+F 2 "william_potentiometer:Potentiometer_Bourns_TC33X_Vertical" H 2050 1400 50  0001 C CNN
 F 3 "~" H 2050 1400 50  0001 C CNN
+F 4 "TC33X-2-104E" H 2050 1400 50  0001 C CNN "MPN"
 	1    2050 1400
 	-1   0    0    -1
 $EndComp
 $Comp
-L Device:R R?
+L Device:R R5
 U 1 1 5F779374
 P 1500 1550
-F 0 "R?" H 1570 1596 50  0000 L CNN
+F 0 "R5" H 1570 1596 50  0000 L CNN
 F 1 "1K" H 1570 1505 50  0000 L CNN
-F 2 "" V 1430 1550 50  0001 C CNN
+F 2 "Resistor_SMD:R_0603_1608Metric" V 1430 1550 50  0001 C CNN
 F 3 "~" H 1500 1550 50  0001 C CNN
 	1    1500 1550
@@
 ~FAULT
 $Comp
-L Device:R R?
+L Device:R R6
 U 1 1 5F77EB87
 P 1600 3100
-F 0 "R?" V 1807 3100 50  0000 C CNN
+F 0 "R6" V 1807 3100 50  0000 C CNN
 F 1 "10K" V 1716 3100 50  0000 C CNN
-F 2 "" V 1530 3100 50  0001 C CNN
+F 2 "Resistor_SMD:R_0603_1608Metric" V 1530 3100 50  0001 C CNN
 F 3 "~" H 1600 3100 50  0001 C CNN
 	1    1600 3100
@@
 $EndComp
 $Comp
-L Device:C C?
+L Device:C C4
 U 1 1 5F77EE63
 P 1750 3250
-F 0 "C?" H 1865 3296 50  0000 L CNN
+F 0 "C4" H 1865 3296 50  0000 L CNN
 F 1 "100N" H 1865 3205 50  0000 L CNN
-F 2 "" H 1788 3100 50  0001 C CNN
+F 2 "Capacitor_SMD:C_0603_1608Metric" H 1788 3100 50  0001 C CNN
 F 3 "~" H 1750 3250 50  0001 C CNN
 	1    1750 3250
@@
 	1750 6250 1750 6150
 $Comp
-L Device:R R?
+L Device:R R8
 U 1 1 5F78D338
 P 1750 6000
-F 0 "R?" H 1820 6046 50  0000 L CNN
+F 0 "R8" H 1820 6046 50  0000 L CNN
 F 1 "10K" H 1820 5955 50  0000 L CNN
-F 2 "" V 1680 6000 50  0001 C CNN
+F 2 "Resistor_SMD:R_0603_1608Metric" V 1680 6000 50  0001 C CNN
 F 3 "~" H 1750 6000 50  0001 C CNN
 	1    1750 6000
@@
 $EndComp
 $Comp
-L Device:R R?
+L Device:R R7
 U 1 1 5F78CCBB
 P 1750 5700
-F 0 "R?" H 1820 5746 50  0000 L CNN
+F 0 "R7" H 1820 5746 50  0000 L CNN
 F 1 "100K" H 1820 5655 50  0000 L CNN
-F 2 "" V 1680 5700 50  0001 C CNN
+F 2 "Resistor_SMD:R_0603_1608Metric" V 1680 5700 50  0001 C CNN
 F 3 "~" H 1750 5700 50  0001 C CNN
 	1    1750 5700
@@
 GND
 $Comp
-L Device:C C?
+L Device:C C5
 U 1 1 5F790FDD
 P 4350 1100
-F 0 "C?" H 4465 1146 50  0000 L CNN
+F 0 "C5" H 4465 1146 50  0000 L CNN
 F 1 "2U2" H 4465 1055 50  0000 L CNN
-F 2 "" H 4388 950 50  0001 C CNN
+F 2 "Capacitor_SMD:C_0805_2012Metric" H 4388 950 50  0001 C CNN
 F 3 "~" H 4350 1100 50  0001 C CNN
 	1    4350 1100
@@
 $EndComp
 $Comp
-L Device:CP C?
+L Device:CP C6
 U 1 1 5F791CAE
 P 4800 1100
-F 0 "C?" H 4918 1146 50  0000 L CNN
+F 0 "C6" H 4918 1146 50  0000 L CNN
 F 1 "100UF" H 4918 1055 50  0000 L CNN
-F 2 "" H 4838 950 50  0001 C CNN
+F 2 "Capacitor_THT:CP_Radial_D6.3mm_P2.50mm" H 4838 950 50  0001 C CNN
 F 3 "~" H 4800 1100 50  0001 C CNN
 	1    4800 1100
@@
 Text Notes 6000 2100 0    50   ~ 0
 1.8V - 10V
+$Comp
+L Device:R R11
+U 1 1 5F8E68C6
+P 7750 5400
+F 0 "R11" H 7820 5446 50  0000 L CNN
+F 1 "0R2" H 7820 5355 50  0000 L CNN
+F 2 "Resistor_SMD:R_1020_2550Metric" V 7680 5400 50  0001 C CNN
+F 3 "~" H 7750 5400 50  0001 C CNN
+F 4 "RCWE1020R200FKEA" H 7750 5400 50  0001 C CNN "MPN"
+	1    7750 5400
+	1    0    0    -1
+$EndComp
 $EndSCHEMATC

Commit message: stspin?
Parts:
- C6: value 100UF -> 470U
Changed lines of the file:
@@
 P 4800 1100
 F 0 "C6" H 4918 1146 50  0000 L CNN
-F 1 "100UF" H 4918 1055 50  0000 L CNN
+F 1 "470U" H 4918 1055 50  0000 L CNN
 F 2 "Capacitor_THT:CP_Radial_D6.3mm_P2.50mm" H 4838 950 50  0001 C CNN
 F 3 "~" H 4800 1100 50  0001 C CNN

Commit message: chevelle adds
Parts:
- renumbered C3 to C?, C4 to C?, C5 to C?, C6 to C?, R10 to R?, R9 to R?, R5 to R?, R6 to R?, R7 to R?, R8 to R?, R11 to R?, RV1 to RV?, U2 to U?
Changed lines of the file:
@@
 $Descr A4 11693 8268
 encoding utf-8
-Sheet 4 10
+Sheet 7 10
 Title ""
 Date ""
@@
 $EndDescr
 $Comp
-L Driver_Motor:STSPIN220 U2
+L Driver_Motor:STSPIN220 U?
 U 1 1 5F76C969
 P 6400 2950
-F 0 "U2" H 6800 3700 50  0000 C CNN
+F 0 "U?" H 6800 3700 50  0000 C CNN
 F 1 "STSPIN220" H 6700 3600 50  0000 C CNN
 F 2 "Package_DFN_QFN:VQFN-16-1EP_3x3mm_P0.5mm_EP1.8x1.8mm" H 6600 3700 50  0001 L CNN
@@
 VMOT
 $Comp
-L Device:R R10
+L Device:R R?
 U 1 1 5F76E303
 P 7350 5400
-F 0 "R10" H 7420 5446 50  0000 L CNN
+F 0 "R?" H 7420 5446 50  0000 L CNN
 F 1 "0R2" H 7420 5355 50  0000 L CNN
 F 2 "Resistor_SMD:R_1020_2550Metric" V 7280 5400 50  0001 C CNN
@@
 MODE2
 $Comp
-L Device:C C3
+L Device:C C?
 U 1 1 5F770F3B
 P 1500 1850
-F 0 "C3" H 1615 1896 50  0000 L CNN
+F 0 "C?" H 1615 1896 50  0000 L CNN
 F 1 "22N" H 1615 1805 50  0000 L CNN
 F 2 "Capacitor_SMD:C_0603_1608Metric" H 1538 1700 50  0001 C CNN
@@
 	5650 3450 5900 3450
 $Comp
-L Device:R R9
+L Device:R R?
 U 1 1 5F773161
 P 2050 1700
-F 0 "R9" H 2120 1746 50  0000 L CNN
+F 0 "R?" H 2120 1746 50  0000 L CNN
 F 1 "10K" H 2120 1655 50  0000 L CNN
 F 2 "Resistor_SMD:R_0603_1608Metric" V 1980 1700 50  0001 C CNN
@@
 $EndComp
 $Comp
-L william_potentiometer:TC33X-2-104E RV1
+L william_potentiometer:TC33X-2-104E RV?
 U 1 1 5F77879D
 P 2050 1400
-F 0 "RV1" H 1980 1446 50  0000 R CNN
+F 0 "RV?" H 1980 1446 50  0000 R CNN
 F 1 "TC33X-2-104E" H 1980 1355 50  0000 R CNN
 F 2 "william_potentiometer:Potentiometer_Bourns_TC33X_Vertical" H 2050 1400 50  0001 C CNN
@@
 $EndComp
 $Comp
-L Device:R R5
+L Device:R R?
 U 1 1 5F779374
 P 1500 1550
-F 0 "R5" H 1570 1596 50  0000 L CNN
+F 0 "R?" H 1570 1596 50  0000 L CNN
 F 1 "1K" H 1570 1505 50  0000 L CNN
 F 2 "Resistor_SMD:R_0603_1608Metric" V 1430 1550 50  0001 C CNN
@@
 ~FAULT
 $Comp
-L Device:R R6
+L Device:R R?
 U 1 1 5F77EB87
 P 1600 3100
-F 0 "R6" V 1807 3100 50  0000 C CNN
+F 0 "R?" V 1807 3100 50  0000 C CNN
 F 1 "10K" V 1716 3100 50  0000 C CNN
 F 2 "Resistor_SMD:R_0603_1608Metric" V 1530 3100 50  0001 C CNN
@@
 $EndComp
 $Comp
-L Device:C C4
+L Device:C C?
 U 1 1 5F77EE63
 P 1750 3250
-F 0 "C4" H 1865 3296 50  0000 L CNN
+F 0 "C?" H 1865 3296 50  0000 L CNN
 F 1 "100N" H 1865 3205 50  0000 L CNN
 F 2 "Capacitor_SMD:C_0603_1608Metric" H 1788 3100 50  0001 C CNN
@@
 	1750 6250 1750 6150
 $Comp
-L Device:R R8
+L Device:R R?
 U 1 1 5F78D338
 P 1750 6000
-F 0 "R8" H 1820 6046 50  0000 L CNN
+F 0 "R?" H 1820 6046 50  0000 L CNN
 F 1 "10K" H 1820 5955 50  0000 L CNN
 F 2 "Resistor_SMD:R_0603_1608Metric" V 1680 6000 50  0001 C CNN
@@
 $EndComp
 $Comp
-L Device:R R7
+L Device:R R?
 U 1 1 5F78CCBB
 P 1750 5700
-F 0 "R7" H 1820 5746 50  0000 L CNN
+F 0 "R?" H 1820 5746 50  0000 L CNN
 F 1 "100K" H 1820 5655 50  0000 L CNN
 F 2 "Resistor_SMD:R_0603_1608Metric" V 1680 5700 50  0001 C CNN
@@
 GND
 $Comp
-L Device:C C5
+L Device:C C?
 U 1 1 5F790FDD
 P 4350 1100
-F 0 "C5" H 4465 1146 50  0000 L CNN
+F 0 "C?" H 4465 1146 50  0000 L CNN
 F 1 "2U2" H 4465 1055 50  0000 L CNN
 F 2 "Capacitor_SMD:C_0805_2012Metric" H 4388 950 50  0001 C CNN
@@
 $EndComp
 $Comp
-L Device:CP C6
+L Device:CP C?
 U 1 1 5F791CAE
 P 4800 1100
-F 0 "C6" H 4918 1146 50  0000 L CNN
+F 0 "C?" H 4918 1146 50  0000 L CNN
 F 1 "470U" H 4918 1055 50  0000 L CNN
 F 2 "Capacitor_THT:CP_Radial_D6.3mm_P2.50mm" H 4838 950 50  0001 C CNN
@@
 1.8V - 10V
 $Comp
-L Device:R R11
+L Device:R R?
 U 1 1 5F8E68C6
 P 7750 5400
-F 0 "R11" H 7820 5446 50  0000 L CNN
+F 0 "R?" H 7820 5446 50  0000 L CNN
 F 1 "0R2" H 7820 5355 50  0000 L CNN
 F 2 "Resistor_SMD:R_1020_2550Metric" V 7680 5400 50  0001 C CNN
