File: 32_768KHz.sch (KiCad schematic (older format))
At the start: 3 parts, among them Y2 ECX-.327-CDX-1293

Commit message: fixed some footprints
Parts:
- removed Y2: ECX-.327-CDX-1293, Crystal:Crystal_SMD_3215-2Pin_3.2x1.5mm, symbol Device:Crystal
- added Y2: ECX-.327-CDX-1293, william_crystal:ECX-.327-CDX-1293, symbol william_crystal:ECX-.327-CDX-1293
Changed lines of the file:
@@
 Text Notes 4850 2650 0    50   ~ 0
 Cl = (C1*C2)/(C1 + C2) + Cparasitic\n\nlet C1 = C2\nCl = C1*C1/2*C1 + Cparasitic\nCl = C1/2 + Cparasitic\nCl - Cparasitic = C1/2\n2(Cl - Cparasitic) = C1\nC1 = 2(Cl - Cparasitic)\nCparasitic appx= 2pF - 5pF\n
-$Comp
-L Device:Crystal Y2
-U 1 1 5EEE4FBD
-P 5400 3700
-F 0 "Y2" H 5400 3968 50  0000 C CNN
-F 1 "ECX-.327-CDX-1293" H 5400 3877 50  0000 C CNN
-F 2 "Crystal:Crystal_SMD_3215-2Pin_3.2x1.5mm" H 5400 3700 50  0001 C CNN
-F 3 "~" H 5400 3700 50  0001 C CNN
-	1    5400 3700
-	1    0    0    -1
-$EndComp
 Wire Wire Line
 	5150 4050 5650 4050
@@
 Wire Wire Line
 	5650 3700 5750 3700
+$Comp
+L william_crystal:ECX-.327-CDX-1293 Y2
+U 1 1 5EE21633
+P 5400 3700
+F 0 "Y2" H 5400 3968 50  0000 C CNN
+F 1 "ECX-.327-CDX-1293" H 5400 3877 50  0000 C CNN
+F 2 "william_crystal:ECX-.327-CDX-1293" H 5400 3700 50  0001 C CNN
+F 3 "~" H 5400 3700 50  0001 C CNN
+	1    5400 3700
+	1    0    0    -1
+$EndComp
 $EndSCHEMATC

Commit message: parts for grease board &displays
Changed lines of the file:
@@
 $Descr A4 11693 8268
 encoding utf-8
-Sheet 10 13
+Sheet 13 17
 Title ""
 Date ""
@@
 AR Path="/5EE8C24E/5C241710/5C243448" Ref="C?"  Part="1"
 AR Path="/5EE8C24E/5EECCCAE/5C243448" Ref="C36"  Part="1"
-F 0 "C36" H 4900 3900 50  0000 L CNN
+AR Path="/5F7173C7/5EECCCAE/5C243448" Ref="C36"  Part="1"
+AR Path="/5F7270DA/5EECCCAE/5C243448" Ref="C40"  Part="1"
+AR Path="/5F7429EF/5EECCCAE/5C243448" Ref="C?"  Part="1"
+AR Path="/6030263D/60306C73/6030EB4E/5C243448" Ref="C58"  Part="1"
+AR Path="/6030263D/603F73B7/6030EB4E/5C243448" Ref="C?"  Part="1"
+F 0 "C58" H 4900 3900 50  0000 L CNN
 F 1 "17P" H 4900 3800 50  0000 L CNN
 F 2 "Capacitor_SMD:C_0402_1005Metric" H 5188 3700 50  0001 C CNN
@@
 AR Path="/5EE8C24E/5C241710/5EEE6426" Ref="C?"  Part="1"
 AR Path="/5EE8C24E/5EECCCAE/5EEE6426" Ref="C37"  Part="1"
-F 0 "C37" H 5400 3900 50  0000 L CNN
+AR Path="/5F7173C7/5EECCCAE/5EEE6426" Ref="C37"  Part="1"
+AR Path="/5F7270DA/5EECCCAE/5EEE6426" Ref="C41"  Part="1"
+AR Path="/5F7429EF/5EECCCAE/5EEE6426" Ref="C?"  Part="1"
+AR Path="/6030263D/60306C73/6030EB4E/5EEE6426" Ref="C59"  Part="1"
+AR Path="/6030263D/603F73B7/6030EB4E/5EEE6426" Ref="C?"  Part="1"
+F 0 "C59" H 5400 3900 50  0000 L CNN
 F 1 "17P" H 5400 3800 50  0000 L CNN
 F 2 "Capacitor_SMD:C_0402_1005Metric" H 5688 3700 50  0001 C CNN
@@
 U 1 1 5EE21633
 P 5400 3700
-F 0 "Y2" H 5400 3968 50  0000 C CNN
+AR Path="/5F7173C7/5EECCCAE/5EE21633" Ref="Y2"  Part="1"
+AR Path="/5F7270DA/5EECCCAE/5EE21633" Ref="Y4"  Part="1"
+AR Path="/5F7429EF/5EECCCAE/5EE21633" Ref="Y?"  Part="1"
+AR Path="/6030263D/60306C73/6030EB4E/5EE21633" Ref="Y3"  Part="1"
+AR Path="/6030263D/603F73B7/6030EB4E/5EE21633" Ref="Y?"  Part="1"
+F 0 "Y3" H 5400 3968 50  0000 C CNN
 F 1 "ECX-.327-CDX-1293" H 5400 3877 50  0000 C CNN
 F 2 "william_crystal:ECX-.327-CDX-1293" H 5400 3700 50  0001 C CNN

Commit message: bunch of updates, apparently
Parts:
- renumbered C36 to C45, C37 to C46
Changed lines of the file:
@@
 $Descr A4 11693 8268
 encoding utf-8
-Sheet 13 17
+Sheet 11 18
 Title ""
 Date ""
@@
 AR Path="/5BFEFCBF/5C241710/5C243448" Ref="C?"  Part="1"
 AR Path="/5EE8C24E/5C241710/5C243448" Ref="C?"  Part="1"
-AR Path="/5EE8C24E/5EECCCAE/5C243448" Ref="C36"  Part="1"
-AR Path="/5F7173C7/5EECCCAE/5C243448" Ref="C36"  Part="1"
-AR Path="/5F7270DA/5EECCCAE/5C243448" Ref="C40"  Part="1"
+AR Path="/5EE8C24E/5EECCCAE/5C243448" Ref="C?"  Part="1"
+AR Path="/5F7173C7/5EECCCAE/5C243448" Ref="C?"  Part="1"
+AR Path="/5F7270DA/5EECCCAE/5C243448" Ref="C?"  Part="1"
 AR Path="/5F7429EF/5EECCCAE/5C243448" Ref="C?"  Part="1"
-AR Path="/6030263D/60306C73/6030EB4E/5C243448" Ref="C58"  Part="1"
+AR Path="/6030263D/60306C73/6030EB4E/5C243448" Ref="C45"  Part="1"
 AR Path="/6030263D/603F73B7/6030EB4E/5C243448" Ref="C?"  Part="1"
-F 0 "C58" H 4900 3900 50  0000 L CNN
+F 0 "C45" H 4900 3900 50  0000 L CNN
 F 1 "17P" H 4900 3800 50  0000 L CNN
 F 2 "Capacitor_SMD:C_0402_1005Metric" H 5188 3700 50  0001 C CNN
@@
 AR Path="/5BFEFCBF/5C241710/5EEE6426" Ref="C?"  Part="1"
 AR Path="/5EE8C24E/5C241710/5EEE6426" Ref="C?"  Part="1"
-AR Path="/5EE8C24E/5EECCCAE/5EEE6426" Ref="C37"  Part="1"
-AR Path="/5F7173C7/5EECCCAE/5EEE6426" Ref="C37"  Part="1"
-AR Path="/5F7270DA/5EECCCAE/5EEE6426" Ref="C41"  Part="1"
+AR Path="/5EE8C24E/5EECCCAE/5EEE6426" Ref="C?"  Part="1"
+AR Path="/5F7173C7/5EECCCAE/5EEE6426" Ref="C?"  Part="1"
+AR Path="/5F7270DA/5EECCCAE/5EEE6426" Ref="C?"  Part="1"
 AR Path="/5F7429EF/5EECCCAE/5EEE6426" Ref="C?"  Part="1"
-AR Path="/6030263D/60306C73/6030EB4E/5EEE6426" Ref="C59"  Part="1"
+AR Path="/6030263D/60306C73/6030EB4E/5EEE6426" Ref="C46"  Part="1"
 AR Path="/6030263D/603F73B7/6030EB4E/5EEE6426" Ref="C?"  Part="1"
-F 0 "C59" H 5400 3900 50  0000 L CNN
+F 0 "C46" H 5400 3900 50  0000 L CNN
 F 1 "17P" H 5400 3800 50  0000 L CNN
 F 2 "Capacitor_SMD:C_0402_1005Metric" H 5688 3700 50  0001 C CNN
@@
 	5650 3700 5750 3700
 $Comp
-L william_crystal:ECX-.327-CDX-1293 Y2
+L william_crystal:ECX-.327-CDX-1293 Y?
 U 1 1 5EE21633
 P 5400 3700
-AR Path="/5F7173C7/5EECCCAE/5EE21633" Ref="Y2"  Part="1"
-AR Path="/5F7270DA/5EECCCAE/5EE21633" Ref="Y4"  Part="1"
+AR Path="/5F7173C7/5EECCCAE/5EE21633" Ref="Y?"  Part="1"
+AR Path="/5F7270DA/5EECCCAE/5EE21633" Ref="Y?"  Part="1"
 AR Path="/5F7429EF/5EECCCAE/5EE21633" Ref="Y?"  Part="1"
-AR Path="/6030263D/60306C73/6030EB4E/5EE21633" Ref="Y3"  Part="1"
+AR Path="/6030263D/60306C73/6030EB4E/5EE21633" Ref="Y2"  Part="1"
 AR Path="/6030263D/603F73B7/6030EB4E/5EE21633" Ref="Y?"  Part="1"
-F 0 "Y3" H 5400 3968 50  0000 C CNN
+F 0 "Y2" H 5400 3968 50  0000 C CNN
 F 1 "ECX-.327-CDX-1293" H 5400 3877 50  0000 C CNN
 F 2 "william_crystal:ECX-.327-CDX-1293" H 5400 3700 50  0001 C CNN
