File: STM32F746NGHX.sch (KiCad schematic (older format))
At the start: 31 parts, among them J15 TC2030-IDC, U3 STM32F746NGHx

Commit message: bunch of updates, apparently
Parts:
- renumbered C16 to C14, C17 to C15, C18 to C16, C19 to C17, C20 to C18, C21 to C19, C22 to C20, C23 to C21, C24 to C22, C25 to C23, C26 to C24, C38 to C25, C39 to C26, C40 to C27, C41 to C28, C42 to C29, C43 to C30, C44 to C31, C45 to C32, C46 to C33, C47 to C34, C48 to C35, C49 to C36, C50 to C37, C51 to C38, C52 to C39, C53 to C40, C54 to C41, C55 to C42, J15 to J17, U3 to U2

Commit message: display board updates
Parts:
- C15, C16, C22, C23, C24, C25, C26, C27, C28, C29, C30, C31, C32, C33, C34, C35, C36, C37, C38, C39, C40, C41, C42: footprint Capacitor_SMD:C_0603_1608Metric -> Capacitor_SMD:C_0402_1005Metric
Changed lines of the file:
@@
 F 0 "C23" H 6265 3446 50  0000 L CNN
 F 1 "100N" H 6265 3355 50  0000 L CNN
-F 2 "Capacitor_SMD:C_0603_1608Metric" H 6188 3250 50  0001 C CNN
+F 2 "Capacitor_SMD:C_0402_1005Metric" H 6188 3250 50  0001 C CNN
 F 3 "~" H 6150 3400 50  0001 C CNN
 	1    6150 3400
@@
 F 0 "C24" H 6265 4246 50  0000 L CNN
 F 1 "100N" H 6265 4155 50  0000 L CNN
-F 2 "Capacitor_SMD:C_0603_1608Metric" H 6188 4050 50  0001 C CNN
+F 2 "Capacitor_SMD:C_0402_1005Metric" H 6188 4050 50  0001 C CNN
 F 3 "~" H 6150 4200 50  0001 C CNN
 	1    6150 4200
@@
 F 0 "C15" H 5365 1046 50  0000 L CNN
 F 1 "100N" H 5365 955 50  0000 L CNN
-F 2 "Capacitor_SMD:C_0603_1608Metric" H 5288 850 50  0001 C CNN
+F 2 "Capacitor_SMD:C_0402_1005Metric" H 5288 850 50  0001 C CNN
 F 3 "~" H 5250 1000 50  0001 C CNN
 	1    5250 1000
@@
 F 0 "C16" H 5815 1046 50  0000 L CNN
 F 1 "100N" H 5815 955 50  0000 L CNN
-F 2 "Capacitor_SMD:C_0603_1608Metric" H 5738 850 50  0001 C CNN
+F 2 "Capacitor_SMD:C_0402_1005Metric" H 5738 850 50  0001 C CNN
 F 3 "~" H 5700 1000 50  0001 C CNN
 	1    5700 1000
@@
 F 0 "C22" H 6265 1046 50  0000 L CNN
 F 1 "100N" H 6265 955 50  0000 L CNN
-F 2 "Capacitor_SMD:C_0603_1608Metric" H 6188 850 50  0001 C CNN
+F 2 "Capacitor_SMD:C_0402_1005Metric" H 6188 850 50  0001 C CNN
 F 3 "~" H 6150 1000 50  0001 C CNN
 	1    6150 1000
@@
 F 0 "C26" H 6715 1046 50  0000 L CNN
 F 1 "100N" H 6715 955 50  0000 L CNN
-F 2 "Capacitor_SMD:C_0603_1608Metric" H 6638 850 50  0001 C CNN
+F 2 "Capacitor_SMD:C_0402_1005Metric" H 6638 850 50  0001 C CNN
 F 3 "~" H 6600 1000 50  0001 C CNN
 	1    6600 1000
@@
 F 0 "C27" H 7165 1046 50  0000 L CNN
 F 1 "100N" H 7165 955 50  0000 L CNN
-F 2 "Capacitor_SMD:C_0603_1608Metric" H 7088 850 50  0001 C CNN
+F 2 "Capacitor_SMD:C_0402_1005Metric" H 7088 850 50  0001 C CNN
 F 3 "~" H 7050 1000 50  0001 C CNN
 	1    7050 1000
@@
 F 0 "C28" H 7615 1046 50  0000 L CNN
 F 1 "100N" H 7615 955 50  0000 L CNN
-F 2 "Capacitor_SMD:C_0603_1608Metric" H 7538 850 50  0001 C CNN
+F 2 "Capacitor_SMD:C_0402_1005Metric" H 7538 850 50  0001 C CNN
 F 3 "~" H 7500 1000 50  0001 C CNN
 	1    7500 1000
@@
 F 0 "C29" H 8065 1046 50  0000 L CNN
 F 1 "100N" H 8065 955 50  0000 L CNN
-F 2 "Capacitor_SMD:C_0603_1608Metric" H 7988 850 50  0001 C CNN
+F 2 "Capacitor_SMD:C_0402_1005Metric" H 7988 850 50  0001 C CNN
 F 3 "~" H 7950 1000 50  0001 C CNN
 	1    7950 1000
@@
 F 0 "C30" H 8515 1046 50  0000 L CNN
 F 1 "100N" H 8515 955 50  0000 L CNN
-F 2 "Capacitor_SMD:C_0603_1608Metric" H 8438 850 50  0001 C CNN
+F 2 "Capacitor_SMD:C_0402_1005Metric" H 8438 850 50  0001 C CNN
 F 3 "~" H 8400 1000 50  0001 C CNN
 	1    8400 1000
@@
 F 0 "C31" H 8965 1046 50  0000 L CNN
 F 1 "100N" H 8965 955 50  0000 L CNN
-F 2 "Capacitor_SMD:C_0603_1608Metric" H 8888 850 50  0001 C CNN
+F 2 "Capacitor_SMD:C_0402_1005Metric" H 8888 850 50  0001 C CNN
 F 3 "~" H 8850 1000 50  0001 C CNN
 	1    8850 1000
@@
 F 0 "C32" H 9415 1046 50  0000 L CNN
 F 1 "100N" H 9415 955 50  0000 L CNN
-F 2 "Capacitor_SMD:C_0603_1608Metric" H 9338 850 50  0001 C CNN
+F 2 "Capacitor_SMD:C_0402_1005Metric" H 9338 850 50  0001 C CNN
 F 3 "~" H 9300 1000 50  0001 C CNN
 	1    9300 1000
@@
 F 0 "C33" H 9865 1046 50  0000 L CNN
 F 1 "100N" H 9865 955 50  0000 L CNN
-F 2 "Capacitor_SMD:C_0603_1608Metric" H 9788 850 50  0001 C CNN
+F 2 "Capacitor_SMD:C_0402_1005Metric" H 9788 850 50  0001 C CNN
 F 3 "~" H 9750 1000 50  0001 C CNN
 	1    9750 1000
@@
 F 0 "C34" H 10315 1046 50  0000 L CNN
 F 1 "100N" H 10315 955 50  0000 L CNN
-F 2 "Capacitor_SMD:C_0603_1608Metric" H 10238 850 50  0001 C CNN
+F 2 "Capacitor_SMD:C_0402_1005Metric" H 10238 850 50  0001 C CNN
 F 3 "~" H 10200 1000 50  0001 C CNN
 	1    10200 1000
@@
 F 0 "C35" H 10765 1046 50  0000 L CNN
 F 1 "100N" H 10765 955 50  0000 L CNN
-F 2 "Capacitor_SMD:C_0603_1608Metric" H 10688 850 50  0001 C CNN
+F 2 "Capacitor_SMD:C_0402_1005Metric" H 10688 850 50  0001 C CNN
 F 3 "~" H 10650 1000 50  0001 C CNN
 	1    10650 1000
@@
 F 0 "C36" H 11215 1046 50  0000 L CNN
 F 1 "100N" H 11215 955 50  0000 L CNN
-F 2 "Capacitor_SMD:C_0603_1608Metric" H 11138 850 50  0001 C CNN
+F 2 "Capacitor_SMD:C_0402_1005Metric" H 11138 850 50  0001 C CNN
 F 3 "~" H 11100 1000 50  0001 C CNN
 	1    11100 1000
@@
 F 0 "C37" H 11665 1046 50  0000 L CNN
 F 1 "100N" H 11665 955 50  0000 L CNN
-F 2 "Capacitor_SMD:C_0603_1608Metric" H 11588 850 50  0001 C CNN
+F 2 "Capacitor_SMD:C_0402_1005Metric" H 11588 850 50  0001 C CNN
 F 3 "~" H 11550 1000 50  0001 C CNN
 	1    11550 1000
@@
 F 0 "C38" H 12115 1046 50  0000 L CNN
 F 1 "100N" H 12115 955 50  0000 L CNN
-F 2 "Capacitor_SMD:C_0603_1608Metric" H 12038 850 50  0001 C CNN
+F 2 "Capacitor_SMD:C_0402_1005Metric" H 12038 850 50  0001 C CNN
 F 3 "~" H 12000 1000 50  0001 C CNN
 	1    12000 1000
@@
 F 0 "C39" H 12565 1046 50  0000 L CNN
 F 1 "100N" H 12565 955 50  0000 L CNN
-F 2 "Capacitor_SMD:C_0603_1608Metric" H 12488 850 50  0001 C CNN
+F 2 "Capacitor_SMD:C_0402_1005Metric" H 12488 850 50  0001 C CNN
 F 3 "~" H 12450 1000 50  0001 C CNN
 	1    12450 1000
@@
 F 0 "C40" H 13015 1046 50  0000 L CNN
 F 1 "100N" H 13015 955 50  0000 L CNN
-F 2 "Capacitor_SMD:C_0603_1608Metric" H 12938 850 50  0001 C CNN
+F 2 "Capacitor_SMD:C_0402_1005Metric" H 12938 850 50  0001 C CNN
 F 3 "~" H 12900 1000 50  0001 C CNN
 	1    12900 1000
@@
 F 0 "C41" H 13465 1046 50  0000 L CNN
 F 1 "100N" H 13465 955 50  0000 L CNN
-F 2 "Capacitor_SMD:C_0603_1608Metric" H 13388 850 50  0001 C CNN
+F 2 "Capacitor_SMD:C_0402_1005Metric" H 13388 850 50  0001 C CNN
 F 3 "~" H 13350 1000 50  0001 C CNN
 	1    13350 1000
@@
 F 0 "C42" H 13915 1046 50  0000 L CNN
 F 1 "100N" H 13915 955 50  0000 L CNN
-F 2 "Capacitor_SMD:C_0603_1608Metric" H 13838 850 50  0001 C CNN
+F 2 "Capacitor_SMD:C_0402_1005Metric" H 13838 850 50  0001 C CNN
 F 3 "~" H 13800 1000 50  0001 C CNN
 	1    13800 1000
@@
 F 0 "C25" H 6265 5096 50  0000 L CNN
 F 1 "100N" H 6265 5005 50  0000 L CNN
-F 2 "Capacitor_SMD:C_0603_1608Metric" H 6188 4900 50  0001 C CNN
+F 2 "Capacitor_SMD:C_0402_1005Metric" H 6188 4900 50  0001 C CNN
 F 3 "~" H 6150 5050 50  0001 C CNN
 	1    6150 5050
