File: eve2_display.sch (KiCad schematic (older format))
At the start: 3 parts, among them J13 EVE2_Display_IDC

Commit message: bunch of updates, apparently
Parts:
- renumbered C14 to C12, C15 to C13, J13 to J16
Changed lines of the file:
@@
 $Descr A4 11693 8268
 encoding utf-8
-Sheet 9 17
+Sheet 7 18
 Title ""
 Date ""
@@
 $EndDescr
 $Comp
-L william_display:EVE2_Display_IDC J13
+L william_display:EVE2_Display_IDC J?
 U 1 1 5F871AFC
 P 5550 3300
-AR Path="/5F871AFC" Ref="J13"  Part="1"
-AR Path="/5F861584/5F871AFC" Ref="J13"  Part="1"
-F 0 "J13" H 5800 4100 50  0000 C CNN
+AR Path="/5F871AFC" Ref="J?"  Part="1"
+AR Path="/5F861584/5F871AFC" Ref="J16"  Part="1"
+F 0 "J16" H 5800 4100 50  0000 C CNN
 F 1 "EVE2_Display_IDC" H 6050 4000 50  0000 C CNN
 F 2 "Connector_IDC:IDC-Header_2x10_P2.54mm_Vertical" H 8000 4300 50  0001 C CNN
@@
 I_VDD := 100mA\nI_BL := 375 mA\n\nI_total = 475mA TYP
 $Comp
-L Device:C C14
+L Device:C C12
 U 1 1 5F87E729
 P 3450 1250
-F 0 "C14" H 3565 1296 50  0000 L CNN
+F 0 "C12" H 3565 1296 50  0000 L CNN
 F 1 "22U" H 3565 1205 50  0000 L CNN
 F 2 "Capacitor_SMD:C_0805_2012Metric" H 3488 1100 50  0001 C CNN
@@
 $EndComp
 $Comp
-L Device:C C15
+L Device:C C13
 U 1 1 5F87E997
 P 3800 1250
-F 0 "C15" H 3915 1296 50  0000 L CNN
+F 0 "C13" H 3915 1296 50  0000 L CNN
 F 1 "100N" H 3915 1205 50  0000 L CNN
 F 2 "Capacitor_SMD:C_0603_1608Metric" H 3838 1100 50  0001 C CNN

Commit message: display board updates
Parts:
- C13: footprint Capacitor_SMD:C_0603_1608Metric -> Capacitor_SMD:C_0402_1005Metric
Changed lines of the file:
@@
 F 0 "C13" H 3915 1296 50  0000 L CNN
 F 1 "100N" H 3915 1205 50  0000 L CNN
-F 2 "Capacitor_SMD:C_0603_1608Metric" H 3838 1100 50  0001 C CNN
+F 2 "Capacitor_SMD:C_0402_1005Metric" H 3838 1100 50  0001 C CNN
 F 3 "~" H 3800 1250 50  0001 C CNN
 	1    3800 1250
