File: Nfet.sch (KiCad schematic (older format))
At the start: 3 parts, among them Q1 BSS138LT3G

Commit message: bunch of updates, apparently
Parts:
- renumbered Q1 to Q9, R5 to R14, R6 to R15
Changed lines of the file:
@@
 $Descr A4 11693 8268
 encoding utf-8
-Sheet 15 17
+Sheet 13 18
 Title ""
 Date ""
@@
 	6250 2800 6200 2800
 $Comp
-L Device:Q_NMOS_GSD Q1
+L Device:Q_NMOS_GSD Q?
 U 1 1 5FC32503
 P 6150 3450
-AR Path="/5BE5A530/5FC32503" Ref="Q1"  Part="1"
-AR Path="/5BE5D36F/5FC32503" Ref="Q2"  Part="1"
-AR Path="/5BE5D37A/5FC32503" Ref="Q3"  Part="1"
+AR Path="/5BE5A530/5FC32503" Ref="Q?"  Part="1"
+AR Path="/5BE5D36F/5FC32503" Ref="Q?"  Part="1"
+AR Path="/5BE5D37A/5FC32503" Ref="Q?"  Part="1"
 AR Path="/5BE5D381/5FC32503" Ref="Q?"  Part="1"
 AR Path="/5C3B8390/5FC32503" Ref="Q?"  Part="1"
 AR Path="/5C3C14B8/5FC32503" Ref="Q?"  Part="1"
 AR Path="/5C4D1AE2/5FC32503" Ref="Q?"  Part="1"
-AR Path="/5C4E4A9C/5FC32503" Ref="Q4"  Part="1"
-AR Path="/5C4EE84B/5FC32503" Ref="Q5"  Part="1"
+AR Path="/5C4E4A9C/5FC32503" Ref="Q?"  Part="1"
+AR Path="/5C4EE84B/5FC32503" Ref="Q?"  Part="1"
 AR Path="/5D986736/5FC32503" Ref="Q?"  Part="1"
 AR Path="/5D98C5E1/5FC32503" Ref="Q?"  Part="1"
 AR Path="/5E03117E/5FC32503" Ref="Q?"  Part="1"
-AR Path="/5ED23439/5FC32503" Ref="Q1"  Part="1"
-AR Path="/5EDCBFC6/5FC32503" Ref="Q2"  Part="1"
-AR Path="/5EDD6DCA/5FC32503" Ref="Q3"  Part="1"
+AR Path="/5ED23439/5FC32503" Ref="Q?"  Part="1"
+AR Path="/5EDCBFC6/5FC32503" Ref="Q?"  Part="1"
+AR Path="/5EDD6DCA/5FC32503" Ref="Q?"  Part="1"
 AR Path="/6048BAFD/5F994F1D/5FC32503" Ref="Q9"  Part="1"
 F 0 "Q9" H 6355 3496 50  0000 L CNN
@@
 $EndComp
 $Comp
-L Device:R R6
+L Device:R R?
 U 1 1 5FC32504
 P 5750 3450
-AR Path="/5BE5A530/5FC32504" Ref="R6"  Part="1"
-AR Path="/5BE5D36F/5FC32504" Ref="R8"  Part="1"
-AR Path="/5BE5D37A/5FC32504" Ref="R10"  Part="1"
+AR Path="/5BE5A530/5FC32504" Ref="R?"  Part="1"
+AR Path="/5BE5D36F/5FC32504" Ref="R?"  Part="1"
+AR Path="/5BE5D37A/5FC32504" Ref="R?"  Part="1"
 AR Path="/5BE5D381/5FC32504" Ref="R?"  Part="1"
 AR Path="/5C3B8390/5FC32504" Ref="R?"  Part="1"
 AR Path="/5C3C14B8/5FC32504" Ref="R?"  Part="1"
 AR Path="/5C4D1AE2/5FC32504" Ref="R?"  Part="1"
-AR Path="/5C4E4A9C/5FC32504" Ref="R26"  Part="1"
-AR Path="/5C4EE84B/5FC32504" Ref="R28"  Part="1"
+AR Path="/5C4E4A9C/5FC32504" Ref="R?"  Part="1"
+AR Path="/5C4EE84B/5FC32504" Ref="R?"  Part="1"
 AR Path="/5D986736/5FC32504" Ref="R?"  Part="1"
 AR Path="/5D98C5E1/5FC32504" Ref="R?"  Part="1"
 AR Path="/5E03117E/5FC32504" Ref="R?"  Part="1"
-AR Path="/5ED23439/5FC32504" Ref="R9"  Part="1"
-AR Path="/5EDCBFC6/5FC32504" Ref="R11"  Part="1"
-AR Path="/5EDD6DCA/5FC32504" Ref="R13"  Part="1"
+AR Path="/5ED23439/5FC32504" Ref="R?"  Part="1"
+AR Path="/5EDCBFC6/5FC32504" Ref="R?"  Part="1"
+AR Path="/5EDD6DCA/5FC32504" Ref="R?"  Part="1"
 AR Path="/6048BAFD/5F994F1D/5FC32504" Ref="R15"  Part="1"
 F 0 "R15" V 5543 3450 50  0000 C CNN
@@
 $EndComp
 $Comp
-L Device:R R5
+L Device:R R?
 U 1 1 5BE5AA7F
 P 5450 3650
-AR Path="/5BE5A530/5BE5AA7F" Ref="R5"  Part="1"
-AR Path="/5BE5D36F/5BE5AA7F" Ref="R7"  Part="1"
-AR Path="/5BE5D37A/5BE5AA7F" Ref="R9"  Part="1"
+AR Path="/5BE5A530/5BE5AA7F" Ref="R?"  Part="1"
+AR Path="/5BE5D36F/5BE5AA7F" Ref="R?"  Part="1"
+AR Path="/5BE5D37A/5BE5AA7F" Ref="R?"  Part="1"
 AR Path="/5BE5D381/5BE5AA7F" Ref="R?"  Part="1"
 AR Path="/5C3B8390/5BE5AA7F" Ref="R?"  Part="1"
 AR Path="/5C3C14B8/5BE5AA7F" Ref="R?"  Part="1"
 AR Path="/5C4D1AE2/5BE5AA7F" Ref="R?"  Part="1"
-AR Path="/5C4E4A9C/5BE5AA7F" Ref="R1"  Part="1"
-AR Path="/5C4EE84B/5BE5AA7F" Ref="R27"  Part="1"
+AR Path="/5C4E4A9C/5BE5AA7F" Ref="R?"  Part="1"
+AR Path="/5C4EE84B/5BE5AA7F" Ref="R?"  Part="1"
 AR Path="/5D986736/5BE5AA7F" Ref="R?"  Part="1"
 AR Path="/5D98C5E1/5BE5AA7F" Ref="R?"  Part="1"
 AR Path="/5E03117E/5BE5AA7F" Ref="R?"  Part="1"
-AR Path="/5ED23439/5BE5AA7F" Ref="R8"  Part="1"
-AR Path="/5EDCBFC6/5BE5AA7F" Ref="R10"  Part="1"
-AR Path="/5EDD6DCA/5BE5AA7F" Ref="R12"  Part="1"
-AR Path="/6048BAFD/5F994F1D/5BE5AA7F" Ref="R12"  Part="1"
-F 0 "R12" H 5520 3696 50  0000 L CNN
+AR Path="/5ED23439/5BE5AA7F" Ref="R?"  Part="1"
+AR Path="/5EDCBFC6/5BE5AA7F" Ref="R?"  Part="1"
+AR Path="/5EDD6DCA/5BE5AA7F" Ref="R?"  Part="1"
+AR Path="/6048BAFD/5F994F1D/5BE5AA7F" Ref="R14"  Part="1"
+F 0 "R14" H 5520 3696 50  0000 L CNN
 F 1 "10K" H 5520 3605 50  0000 L CNN
 F 2 "Resistor_SMD:R_0603_1608Metric" V 5380 3650 50  0001 C CNN

Commit message: changes for display board
Parts:
- Q9: value BSS138LT3G -> BSS670S2LH6327XTSA1‎
Changed lines of the file:
@@
 AR Path="/6053E9DE/5F994F1D/5FC32503" Ref="Q9"  Part="1"
 AR Path="/6053E9DE/604F8548/5FC32503" Ref="Q?"  Part="1"
+AR Path="/609185DA/5F994F1D/5FC32503" Ref="Q9"  Part="1"
 F 0 "Q9" H 6355 3496 50  0000 L CNN
-F 1 "BSS138LT3G" H 6355 3405 50  0000 L CNN
+F 1 "BSS670S2LH6327XTSA1‎" H 6355 3405 50  0000 L CNN
 F 2 "Package_TO_SOT_SMD:SC-59" H 6350 3550 50  0001 C CNN
 F 3 "~" H 6150 3450 50  0001 C CNN
@@
 AR Path="/6053E9DE/5F994F1D/5FC32504" Ref="R15"  Part="1"
 AR Path="/6053E9DE/604F8548/5FC32504" Ref="R?"  Part="1"
+AR Path="/609185DA/5F994F1D/5FC32504" Ref="R15"  Part="1"
 F 0 "R15" V 5543 3450 50  0000 C CNN
 F 1 "1K" V 5634 3450 50  0000 C CNN
@@
 AR Path="/6053E9DE/5F994F1D/5BE5AA7F" Ref="R14"  Part="1"
 AR Path="/6053E9DE/604F8548/5BE5AA7F" Ref="R?"  Part="1"
+AR Path="/609185DA/5F994F1D/5BE5AA7F" Ref="R14"  Part="1"
 F 0 "R14" H 5520 3696 50  0000 L CNN
 F 1 "10K" H 5520 3605 50  0000 L CNN
