File: 24V_to_3v3_1A.sch (KiCad schematic (older format))
At the start: 6 parts

Commit message: parts for touchscreen
Parts:
- gave numbers to parts that had none: 6
Changed lines of the file:
@@
 $Descr A4 11693 8268
 encoding utf-8
-Sheet 8 10
+Sheet 14 20
 Title ""
 Date ""
@@
 $EndDescr
 $Comp
-L Regulator_Switching:R-78E3.3-1.0 U?
+L Regulator_Switching:R-78E3.3-1.0 U4
 U 1 1 5FF26201
 P 4800 3150
-AR Path="/5F8F7CE4/5FF26201" Ref="U?"  Part="1"
-AR Path="/5F8F934E/5FF26201" Ref="U?"  Part="1"
-AR Path="/5F8F956C/5FF26201" Ref="U?"  Part="1"
-AR Path="/5F933719/5FF26201" Ref="U?"  Part="1"
-F 0 "U?" H 4800 3392 50  0000 C CNN
+F 0 "U4" H 4800 3392 50  0000 C CNN
 F 1 "R-78E3.3-1.0" H 4800 3301 50  0000 C CNN
 F 2 "Converter_DCDC:Converter_DCDC_RECOM_R-78E-0.5_THT" H 4850 2900 50  0001 L CIN
@@
 $EndComp
 $Comp
-L Device:L L?
+L Device:L L1
 U 1 1 5FF26B66
 P 4000 3150
-AR Path="/5F8F7CE4/5FF26B66" Ref="L?"  Part="1"
-AR Path="/5F8F934E/5FF26B66" Ref="L?"  Part="1"
-AR Path="/5F8F956C/5FF26B66" Ref="L?"  Part="1"
-AR Path="/5F933719/5FF26B66" Ref="L?"  Part="1"
-F 0 "L?" V 4190 3150 50  0000 C CNN
+F 0 "L1" V 4190 3150 50  0000 C CNN
 F 1 "12U" V 4099 3150 50  0000 C CNN
 F 2 "Inductor_THT:L_Radial_D8.7mm_P5.00mm_Fastron_07HCP" H 4000 3150 50  0001 C CNN
@@
 $EndComp
 $Comp
-L Device:C C?
+L Device:C C50
 U 1 1 5FF2748A
 P 4200 3300
-AR Path="/5F8F7CE4/5FF2748A" Ref="C?"  Part="1"
-AR Path="/5F8F934E/5FF2748A" Ref="C?"  Part="1"
-AR Path="/5F8F956C/5FF2748A" Ref="C?"  Part="1"
-AR Path="/5F933719/5FF2748A" Ref="C?"  Part="1"
-F 0 "C?" H 4315 3346 50  0000 L CNN
+F 0 "C50" H 4315 3346 50  0000 L CNN
 F 1 "10U" H 4315 3255 50  0000 L CNN
 F 2 "Capacitor_SMD:C_0805_2012Metric" H 4238 3150 50  0001 C CNN
@@
 $EndComp
 $Comp
-L Device:C C?
+L Device:C C49
 U 1 1 5FF27909
 P 3800 3300
-AR Path="/5F8F7CE4/5FF27909" Ref="C?"  Part="1"
-AR Path="/5F8F934E/5FF27909" Ref="C?"  Part="1"
-AR Path="/5F8F956C/5FF27909" Ref="C?"  Part="1"
-AR Path="/5F933719/5FF27909" Ref="C?"  Part="1"
-F 0 "C?" H 3915 3346 50  0000 L CNN
+F 0 "C49" H 3915 3346 50  0000 L CNN
 F 1 "10U" H 3915 3255 50  0000 L CNN
 F 2 "Capacitor_SMD:C_0805_2012Metric" H 3838 3150 50  0001 C CNN
@@
 	4200 3450 3800 3450
 $Comp
-L Device:C C?
+L Device:C C51
 U 1 1 5FF28D89
 P 5350 3300
-AR Path="/5F8F7CE4/5FF28D89" Ref="C?"  Part="1"
-AR Path="/5F8F934E/5FF28D89" Ref="C?"  Part="1"
-AR Path="/5F8F956C/5FF28D89" Ref="C?"  Part="1"
-AR Path="/5F933719/5FF28D89" Ref="C?"  Part="1"
-F 0 "C?" H 5465 3346 50  0000 L CNN
+F 0 "C51" H 5465 3346 50  0000 L CNN
 F 1 "10U" H 5465 3255 50  0000 L CNN
 F 2 "Capacitor_SMD:C_0805_2012Metric" H 5388 3150 50  0001 C CNN
@@
 Connection ~ 4800 3450
 $Comp
-L Device:C C?
+L Device:C C52
 U 1 1 5FF292C1
 P 5850 3300
-AR Path="/5F8F7CE4/5FF292C1" Ref="C?"  Part="1"
-AR Path="/5F8F934E/5FF292C1" Ref="C?"  Part="1"
-AR Path="/5F8F956C/5FF292C1" Ref="C?"  Part="1"
-AR Path="/5F933719/5FF292C1" Ref="C?"  Part="1"
-F 0 "C?" H 5965 3346 50  0000 L CNN
+F 0 "C52" H 5965 3346 50  0000 L CNN
 F 1 "100N" H 5965 3255 50  0000 L CNN
 F 2 "Capacitor_SMD:C_0402_1005Metric" H 5888 3150 50  0001 C CNN
@@
 U 1 1 6014322A
 P 4300 3150
-AR Path="/5F8F7CE4/6014322A" Ref="#FLG0101"  Part="1"
-AR Path="/5F8F934E/6014322A" Ref="#FLG?"  Part="1"
-AR Path="/5F8F956C/6014322A" Ref="#FLG?"  Part="1"
-AR Path="/5F933719/6014322A" Ref="#FLG?"  Part="1"
 F 0 "#FLG0101" H 4300 3225 50  0001 C CNN
 F 1 "PWR_FLAG" H 4300 3323 50  0000 C CNN

Commit message: changes for display board
Parts:
- renumbered C49 to C12, C50 to C13, C51 to C14, C52 to C15, U4 to U2
Changed lines of the file:
@@
 $Descr A4 11693 8268
 encoding utf-8
-Sheet 7 13
+Sheet 7 11
 Title ""
 Date ""
@@
 $EndDescr
 $Comp
-L Regulator_Switching:R-78E3.3-1.0 U4
+L Regulator_Switching:R-78E3.3-1.0 U2
 U 1 1 5FF26201
 P 4800 3150
-F 0 "U4" H 4800 3392 50  0000 C CNN
+F 0 "U2" H 4800 3392 50  0000 C CNN
 F 1 "R-78E3.3-1.0" H 4800 3301 50  0000 C CNN
 F 2 "Converter_DCDC:Converter_DCDC_RECOM_R-78E-0.5_THT" H 4850 2900 50  0001 L CIN
@@
 $EndComp
 $Comp
-L Device:C C50
+L Device:C C13
 U 1 1 5FF2748A
 P 4200 3300
-F 0 "C50" H 4315 3346 50  0000 L CNN
+F 0 "C13" H 4315 3346 50  0000 L CNN
 F 1 "10U" H 4315 3255 50  0000 L CNN
 F 2 "Capacitor_SMD:C_0805_2012Metric" H 4238 3150 50  0001 C CNN
@@
 $EndComp
 $Comp
-L Device:C C49
+L Device:C C12
 U 1 1 5FF27909
 P 3800 3300
-F 0 "C49" H 3915 3346 50  0000 L CNN
+F 0 "C12" H 3915 3346 50  0000 L CNN
 F 1 "10U" H 3915 3255 50  0000 L CNN
 F 2 "Capacitor_SMD:C_0805_2012Metric" H 3838 3150 50  0001 C CNN
@@
 	4200 3450 3800 3450
 $Comp
-L Device:C C51
+L Device:C C14
 U 1 1 5FF28D89
 P 5350 3300
-F 0 "C51" H 5465 3346 50  0000 L CNN
+F 0 "C14" H 5465 3346 50  0000 L CNN
 F 1 "10U" H 5465 3255 50  0000 L CNN
 F 2 "Capacitor_SMD:C_0805_2012Metric" H 5388 3150 50  0001 C CNN
@@
 Connection ~ 4800 3450
 $Comp
-L Device:C C52
+L Device:C C15
 U 1 1 5FF292C1
 P 5850 3300
-F 0 "C52" H 5965 3346 50  0000 L CNN
+F 0 "C15" H 5965 3346 50  0000 L CNN
 F 1 "100N" H 5965 3255 50  0000 L CNN
 F 2 "Capacitor_SMD:C_0402_1005Metric" H 5888 3150 50  0001 C CNN
@@
 Connection ~ 5850 3150
 $Comp
-L power:PWR_FLAG #FLG0101
+L power:PWR_FLAG #FLG05
 U 1 1 6014322A
 P 4300 3150
-F 0 "#FLG0101" H 4300 3225 50  0001 C CNN
+F 0 "#FLG05" H 4300 3225 50  0001 C CNN
 F 1 "PWR_FLAG" H 4300 3323 50  0000 C CNN
 F 2 "" H 4300 3150 50  0001 C CNN

Commit message: new f446RETx, displays, a4957
Parts:
- C15: footprint Capacitor_SMD:C_0402_1005Metric -> Capacitor_SMD:C_0603_1608Metric
Changed lines of the file:
@@
 F 0 "C15" H 5965 3346 50  0000 L CNN
 F 1 "100N" H 5965 3255 50  0000 L CNN
-F 2 "Capacitor_SMD:C_0402_1005Metric" H 5888 3150 50  0001 C CNN
+F 2 "Capacitor_SMD:C_0603_1608Metric" H 5888 3150 50  0001 C CNN
 F 3 "~" H 5850 3300 50  0001 C CNN
 	1    5850 3300
