File: 24V_to_5V_500mA.sch (KiCad schematic (older format))
At the start: 6 parts

Commit message: parts for touchscreen
Parts:
- gave numbers to parts that had none: 1
Changed lines of the file:
@@
 $Descr A4 11693 8268
 encoding utf-8
-Sheet 10 10
+Sheet 15 20
 Title ""
 Date ""
@@
 AR Path="/5FF1C389/5FF2CBDC" Ref="L?"  Part="1"
 AR Path="/5FF1CD55/5FF2CBDC" Ref="L2"  Part="1"
-AR Path="/5F933719/5FF2CBDC" Ref="L?"  Part="1"
-F 0 "L?" V 5240 3650 50  0000 C CNN
+F 0 "L2" V 5240 3650 50  0000 C CNN
 F 1 "12U" V 5149 3650 50  0000 C CNN
 F 2 "Inductor_THT:L_Radial_D8.7mm_P5.00mm_Fastron_07HCP" H 5050 3650 50  0001 C CNN
@@
 AR Path="/5FF1C389/5FF2CBE2" Ref="C?"  Part="1"
 AR Path="/5FF1CD55/5FF2CBE2" Ref="C54"  Part="1"
-AR Path="/5F933719/5FF2CBE2" Ref="C?"  Part="1"
-F 0 "C?" H 5365 3846 50  0000 L CNN
+F 0 "C54" H 5365 3846 50  0000 L CNN
 F 1 "4U7" H 5365 3755 50  0000 L CNN
 F 2 "Capacitor_SMD:C_0805_2012Metric" H 5288 3650 50  0001 C CNN
@@
 AR Path="/5FF1C389/5FF2CBE8" Ref="C?"  Part="1"
 AR Path="/5FF1CD55/5FF2CBE8" Ref="C53"  Part="1"
-AR Path="/5F933719/5FF2CBE8" Ref="C?"  Part="1"
-F 0 "C?" H 4965 3846 50  0000 L CNN
+F 0 "C53" H 4965 3846 50  0000 L CNN
 F 1 "10U" H 4965 3755 50  0000 L CNN
 F 2 "Capacitor_SMD:C_0805_2012Metric" H 4888 3650 50  0001 C CNN
@@
 AR Path="/5FF1C389/5FF2CBFC" Ref="C?"  Part="1"
 AR Path="/5FF1CD55/5FF2CBFC" Ref="C55"  Part="1"
-AR Path="/5F933719/5FF2CBFC" Ref="C?"  Part="1"
-F 0 "C?" H 6515 3846 50  0000 L CNN
+F 0 "C55" H 6515 3846 50  0000 L CNN
 F 1 "10U" H 6515 3755 50  0000 L CNN
 F 2 "Capacitor_SMD:C_0805_2012Metric" H 6438 3650 50  0001 C CNN
@@
 AR Path="/5FF1C389/5FF2CC04" Ref="C?"  Part="1"
 AR Path="/5FF1CD55/5FF2CC04" Ref="C56"  Part="1"
-AR Path="/5F933719/5FF2CC04" Ref="C?"  Part="1"
-F 0 "C?" H 7015 3846 50  0000 L CNN
+F 0 "C56" H 7015 3846 50  0000 L CNN
 F 1 "100N" H 7015 3755 50  0000 L CNN
 F 2 "Capacitor_SMD:C_0402_1005Metric" H 6938 3650 50  0001 C CNN
@@
 	5250 3950 5850 3950
 $Comp
-L Regulator_Switching:R-78E5.0-0.5 U?
+L Regulator_Switching:R-78E5.0-0.5 U5
 U 1 1 5FF2CFE9
 P 5850 3650
-F 0 "U?" H 5850 3892 50  0000 C CNN
+F 0 "U5" H 5850 3892 50  0000 C CNN
 F 1 "R-78E5.0-0.5" H 5850 3801 50  0000 C CNN
 F 2 "Converter_DCDC:Converter_DCDC_RECOM_R-78E-0.5_THT" H 5900 3400 50  0001 L CIN

Commit message: changes for display board
Parts:
- renumbered C53 to C27, C54 to C28, C55 to C29, C56 to C30, U5 to U4
Changed lines of the file:
@@
 $Descr A4 11693 8268
 encoding utf-8
-Sheet 15 13
+Sheet 11 11
 Title ""
 Date ""
@@
 P 5250 3800
 AR Path="/5FF1C389/5FF2CBE2" Ref="C?"  Part="1"
-AR Path="/5FF1CD55/5FF2CBE2" Ref="C54"  Part="1"
-F 0 "C54" H 5365 3846 50  0000 L CNN
+AR Path="/5FF1CD55/5FF2CBE2" Ref="C28"  Part="1"
+F 0 "C28" H 5365 3846 50  0000 L CNN
 F 1 "4U7" H 5365 3755 50  0000 L CNN
 F 2 "Capacitor_SMD:C_0805_2012Metric" H 5288 3650 50  0001 C CNN
@@
 P 4850 3800
 AR Path="/5FF1C389/5FF2CBE8" Ref="C?"  Part="1"
-AR Path="/5FF1CD55/5FF2CBE8" Ref="C53"  Part="1"
-F 0 "C53" H 4965 3846 50  0000 L CNN
+AR Path="/5FF1CD55/5FF2CBE8" Ref="C27"  Part="1"
+F 0 "C27" H 4965 3846 50  0000 L CNN
 F 1 "10U" H 4965 3755 50  0000 L CNN
 F 2 "Capacitor_SMD:C_0805_2012Metric" H 4888 3650 50  0001 C CNN
@@
 P 6400 3800
 AR Path="/5FF1C389/5FF2CBFC" Ref="C?"  Part="1"
-AR Path="/5FF1CD55/5FF2CBFC" Ref="C55"  Part="1"
-F 0 "C55" H 6515 3846 50  0000 L CNN
+AR Path="/5FF1CD55/5FF2CBFC" Ref="C29"  Part="1"
+F 0 "C29" H 6515 3846 50  0000 L CNN
 F 1 "10U" H 6515 3755 50  0000 L CNN
 F 2 "Capacitor_SMD:C_0805_2012Metric" H 6438 3650 50  0001 C CNN
@@
 P 6900 3800
 AR Path="/5FF1C389/5FF2CC04" Ref="C?"  Part="1"
-AR Path="/5FF1CD55/5FF2CC04" Ref="C56"  Part="1"
-F 0 "C56" H 7015 3846 50  0000 L CNN
+AR Path="/5FF1CD55/5FF2CC04" Ref="C30"  Part="1"
+F 0 "C30" H 7015 3846 50  0000 L CNN
 F 1 "100N" H 7015 3755 50  0000 L CNN
 F 2 "Capacitor_SMD:C_0402_1005Metric" H 6938 3650 50  0001 C CNN
@@
 	5250 3950 5850 3950
 $Comp
-L Regulator_Switching:R-78E5.0-0.5 U5
+L Regulator_Switching:R-78E5.0-0.5 U4
 U 1 1 5FF2CFE9
 P 5850 3650
-F 0 "U5" H 5850 3892 50  0000 C CNN
+F 0 "U4" H 5850 3892 50  0000 C CNN
 F 1 "R-78E5.0-0.5" H 5850 3801 50  0000 C CNN
 F 2 "Converter_DCDC:Converter_DCDC_RECOM_R-78E-0.5_THT" H 5900 3400 50  0001 L CIN
@@
 	5850 3950 6400 3950
 $Comp
-L power:PWR_FLAG #FLG0102
+L power:PWR_FLAG #FLG06
 U 1 1 60144803
 P 5350 3650
-F 0 "#FLG0102" H 5350 3725 50  0001 C CNN
+F 0 "#FLG06" H 5350 3725 50  0001 C CNN
 F 1 "PWR_FLAG" H 5350 3823 50  0000 C CNN
 F 2 "" H 5350 3650 50  0001 C CNN

Commit message: new f446RETx, displays, a4957
Parts:
- C30: footprint Capacitor_SMD:C_0402_1005Metric -> Capacitor_SMD:C_0603_1608Metric
Changed lines of the file:
@@
 F 0 "C30" H 7015 3846 50  0000 L CNN
 F 1 "100N" H 7015 3755 50  0000 L CNN
-F 2 "Capacitor_SMD:C_0402_1005Metric" H 6938 3650 50  0001 C CNN
+F 2 "Capacitor_SMD:C_0603_1608Metric" H 6938 3650 50  0001 C CNN
 F 3 "~" H 6900 3800 50  0001 C CNN
 	1    6900 3800
