File: A4957sch.sch (KiCad schematic (older format))
At the start: 19 parts, among them Q1 Q_NMOS_GSD, Q2 Q_NMOS_GSD, Q3 Q_NMOS_GSD, Q4 Q_NMOS_GSD, U2 A4957

Commit message: bunch of updates, apparently
Parts:
- removed Q1, Q2, Q3, Q4: Q_NMOS_GSD, william_mosfet:SOT669, symbol Device:Q_NMOS_GSD
- added Q1, Q2, Q3, Q4: PSMN1R0-30YLC,115, Package_TO_SOT_SMD:LFPAK56, symbol william_fets:PSMN1R0-30YLC,115
- R10, R11, R8, R9: footprint Resistor_SMD:R_0612_1632Metric -> Resistor_SMD:R_0603_1608Metric
- R7: value R -> 10K
- renumbered C12 to C10, C13 to C11, C5 to C3, C6 to C4, C7 to C5, C8 to C6, C9 to C7, C10 to C8, C11 to C9, U2 to U1
Connections:
- net labels added: ~FAULT~
Changed lines of the file:
@@
 $Descr A4 11693 8268
 encoding utf-8
-Sheet 2 17
+Sheet 2 18
 Title ""
 Date ""
@@
 P 5450 3900
 AR Path="/5F6A7B03" Ref="U?"  Part="1"
-AR Path="/5F6A7917/5F6A7B03" Ref="U2"  Part="1"
-F 0 "U2" H 5450 4000 50  0000 C CNN
+AR Path="/5F6A7917/5F6A7B03" Ref="U1"  Part="1"
+F 0 "U1" H 5450 4000 50  0000 C CNN
 F 1 "A4957" H 5450 3900 50  0000 C CNN
 F 2 "Package_DFN_QFN:QFN-24-1EP_4x4mm_P0.5mm_EP2.65x2.65mm_ThermalVias" H 5450 5050 50  0001 C CNN
@@
 $EndComp
 $Comp
-L Device:Q_NMOS_GSD Q1
-U 1 1 5F6A8E9F
-P 7350 3500
-F 0 "Q1" H 7554 3546 50  0000 L CNN
-F 1 "Q_NMOS_GSD" H 7554 3455 50  0000 L CNN
-F 2 "william_mosfet:SOT669" H 7550 3600 50  0001 C CNN
-F 3 "~" H 7350 3500 50  0001 C CNN
-	1    7350 3500
-	1    0    0    -1
-$EndComp
-$Comp
-L Device:C C10
+L Device:C C8
 U 1 1 5F6A9316
 P 4650 4000
-F 0 "C10" H 4536 3954 50  0000 R CNN
+F 0 "C8" H 4536 3954 50  0000 R CNN
 F 1 "16V 470N" H 4536 4045 50  0000 R CNN
 F 2 "Capacitor_SMD:C_0603_1608Metric" H 4688 3850 50  0001 C CNN
@@
 	4750 4150 4650 4150
 $Comp
-L Device:C C5
+L Device:C C3
 U 1 1 5F6AA958
 P 2950 1400
-F 0 "C5" H 2835 1446 50  0000 R CNN
+F 0 "C3" H 2835 1446 50  0000 R CNN
 F 1 "10U" H 2835 1355 50  0000 R CNN
 F 2 "Capacitor_SMD:C_0603_1608Metric" H 2988 1250 50  0001 C CNN
@@
 Connection ~ 5300 5100
 $Comp
-L Device:C C8
+L Device:C C6
 U 1 1 5F6ACE5A
 P 4400 4850
-F 0 "C8" H 4285 4896 50  0000 R CNN
+F 0 "C6" H 4285 4896 50  0000 R CNN
 F 1 "16V 22U" H 4285 4805 50  0000 R CNN
 F 2 "Capacitor_SMD:C_0603_1608Metric" H 4438 4700 50  0001 C CNN
@@
 P 6250 3000
 F 0 "R7" H 6320 3046 50  0000 L CNN
-F 1 "R" H 6320 2955 50  0000 L CNN
+F 1 "10K" H 6320 2955 50  0000 L CNN
 F 2 "Resistor_SMD:R_0603_1608Metric" V 6180 3000 50  0001 C CNN
 F 3 "~" H 6250 3000 50  0001 C CNN
@@
 Wire Wire Line
 	6350 3650 6150 3650
-Connection ~ 7450 3700
 Text HLabel 5700 2850 2    50   Input ~ 0
 VBB
@@
 Text HLabel 9250 3700 2    50   Output ~ 0
 OUTA
-Wire Wire Line
-	9250 3700 7450 3700
 Text HLabel 7350 4100 0    50   Input ~ 0
 GND
@@
 VBB
 $Comp
-L Device:C C6
+L Device:C C4
 U 1 1 5F6BC98C
 P 3300 1400
-F 0 "C6" H 3185 1446 50  0000 R CNN
+F 0 "C4" H 3185 1446 50  0000 R CNN
 F 1 "100N" H 3185 1355 50  0000 R CNN
 F 2 "Capacitor_SMD:C_0603_1608Metric" H 3338 1250 50  0001 C CNN
@@
 Wire Wire Line
 	6350 3850 6350 3750
-$Comp
-L Device:Q_NMOS_GSD Q2
-U 1 1 5F6B05A9
-P 7350 3900
-F 0 "Q2" H 7554 3946 50  0000 L CNN
-F 1 "Q_NMOS_GSD" H 7554 3855 50  0000 L CNN
-F 2 "william_mosfet:SOT669" H 7550 4000 50  0001 C CNN
-F 3 "~" H 7350 3900 50  0001 C CNN
-	1    7350 3900
-	1    0    0    -1
-$EndComp
 Wire Wire Line
 	7050 3550 7050 3700
-Wire Wire Line
-	7050 3700 7450 3700
 Wire Wire Line
 	6150 3500 6650 3500
@@
 	6500 3850 6350 3850
 $Comp
-L Device:C C12
+L Device:C C10
 U 1 1 5F6AEFCD
 P 6500 3700
-F 0 "C12" H 6615 3746 50  0000 L CNN
+F 0 "C10" H 6615 3746 50  0000 L CNN
 F 1 "10N" H 6615 3655 50  0000 L CNN
 F 2 "Capacitor_SMD:C_0603_1608Metric" H 6538 3550 50  0001 C CNN
@@
 F 0 "R9" V 6593 3900 50  0000 C CNN
 F 1 "1K" V 6684 3900 50  0000 C CNN
-F 2 "Resistor_SMD:R_0612_1632Metric" V 6730 3900 50  0001 C CNN
+F 2 "Resistor_SMD:R_0603_1608Metric" V 6730 3900 50  0001 C CNN
 F 3 "~" H 6800 3900 50  0001 C CNN
 	1    6800 3900
@@
 F 0 "R8" V 6593 3500 50  0000 C CNN
 F 1 "1K" V 6684 3500 50  0000 C CNN
-F 2 "Resistor_SMD:R_0612_1632Metric" V 6730 3500 50  0001 C CNN
+F 2 "Resistor_SMD:R_0603_1608Metric" V 6730 3500 50  0001 C CNN
 F 3 "~" H 6800 3500 50  0001 C CNN
 	1    6800 3500
@@
 Wire Wire Line
 	6950 3900 7150 3900
-$Comp
-L Device:Q_NMOS_GSD Q3
-U 1 1 5F6CC5E4
-P 8550 4200
-F 0 "Q3" H 8754 4246 50  0000 L CNN
-F 1 "Q_NMOS_GSD" H 8754 4155 50  0000 L CNN
-F 2 "william_mosfet:SOT669" H 8750 4300 50  0001 C CNN
-F 3 "~" H 8550 4200 50  0001 C CNN
-	1    8550 4200
-	1    0    0    -1
-$EndComp
 Wire Wire Line
 	6350 4450 6150 4450
@@
 Wire Wire Line
 	6350 4350 6150 4350
-Connection ~ 8650 4400
 Text HLabel 9250 4400 2    50   Output ~ 0
 OUTB
 Wire Wire Line
-	9250 4400 8650 4400
-Wire Wire Line
 	6350 4550 6350 4450
-$Comp
-L Device:Q_NMOS_GSD Q4
-U 1 1 5F6CC5F6
-P 8550 4600
-F 0 "Q4" H 8754 4646 50  0000 L CNN
-F 1 "Q_NMOS_GSD" H 8754 4555 50  0000 L CNN
-F 2 "william_mosfet:SOT669" H 8750 4700 50  0001 C CNN
-F 3 "~" H 8550 4600 50  0001 C CNN
-	1    8550 4600
-	1    0    0    -1
-$EndComp
 Wire Wire Line
 	7050 4250 7050 4400
-Wire Wire Line
-	7050 4400 8650 4400
 Wire Wire Line
 	6150 4200 6650 4200
@@
 	6500 4550 6350 4550
 $Comp
-L Device:C C13
+L Device:C C11
 U 1 1 5F6CC607
 P 6500 4400
-F 0 "C13" H 6615 4446 50  0000 L CNN
+F 0 "C11" H 6615 4446 50  0000 L CNN
 F 1 "10N" H 6615 4355 50  0000 L CNN
 F 2 "Capacitor_SMD:C_0603_1608Metric" H 6538 4250 50  0001 C CNN
@@
 F 0 "R11" V 6593 4600 50  0000 C CNN
 F 1 "1K" V 6684 4600 50  0000 C CNN
-F 2 "Resistor_SMD:R_0612_1632Metric" V 6730 4600 50  0001 C CNN
+F 2 "Resistor_SMD:R_0603_1608Metric" V 6730 4600 50  0001 C CNN
 F 3 "~" H 6800 4600 50  0001 C CNN
 	1    6800 4600
@@
 F 0 "R10" V 6593 4200 50  0000 C CNN
 F 1 "1K" V 6684 4200 50  0000 C CNN
-F 2 "Resistor_SMD:R_0612_1632Metric" V 6730 4200 50  0001 C CNN
+F 2 "Resistor_SMD:R_0603_1608Metric" V 6730 4200 50  0001 C CNN
 F 3 "~" H 6800 4200 50  0001 C CNN
 	1    6800 4200
@@
 	8550 4800 8650 4800
 $Comp
-L Device:C C11
+L Device:C C9
 U 1 1 5F6EE782
 P 4900 1350
-F 0 "C11" H 5015 1396 50  0000 L CNN
+F 0 "C9" H 5015 1396 50  0000 L CNN
 F 1 "50V 10U" H 5015 1305 50  0000 L CNN
 F 2 "Capacitor_SMD:C_0603_1608Metric" H 4938 1200 50  0001 C CNN
@@
 	4200 1100 3850 1100
 $Comp
-L Device:CP C7
+L Device:CP C5
 U 1 1 5F6FFA62
 P 4200 1350
-F 0 "C7" V 4000 1150 50  0000 L CNN
+F 0 "C5" V 4000 1150 50  0000 L CNN
 F 1 "50V 220U" V 4050 1150 50  0000 L CNN
 F 2 "Capacitor_SMD:CP_Elec_10x10" H 4238 1200 50  0001 C CNN
@@
 Wire Wire Line
 	4200 3300 4750 3300
-Wire Wire Line
-	4200 3200 4750 3200
-$Comp
-L Device:CP C9
+$Comp
+L Device:CP C7
 U 1 1 5FA658A1
 P 4550 1350
-F 0 "C9" V 4350 1150 50  0000 L CNN
+F 0 "C7" V 4350 1150 50  0000 L CNN
 F 1 "50V 220U" V 4400 1150 50  0000 L CNN
 F 2 "Capacitor_SMD:CP_Elec_10x10" H 4588 1200 50  0001 C CNN
@@
 Text Notes 7400 2850 0    50   ~ 0
 Let Cboot = Qgate / Vboot\n\nVboot = appx 16V\nQgate for these fets is 15nC\n\nso Cboot = 15nC / 16V = appx 1nF\nUsing 10nF since I won't drive these quickly
+Wire Wire Line
+	7050 3700 7450 3700
+Wire Wire Line
+	7050 4400 8650 4400
+$Comp
+L william_fets:PSMN1R0-30YLC,115 Q1
+U 1 1 60184E58
+P 7350 3500
+F 0 "Q1" H 7556 3591 50  0000 L CNN
+F 1 "PSMN1R0-30YLC,115" H 7556 3500 50  0000 L CNN
+F 2 "Package_TO_SOT_SMD:LFPAK56" H 7200 3700 50  0001 C CNN
+F 3 "https://assets.nexperia.com/documents/data-sheet/PSMN1R0-30YLC.pdf" H 7350 3500 50  0001 C CNN
+F 4 "PSMN1R0-30YLC,115" H 7556 3409 50  0000 L CNN "MPN"
+	1    7350 3500
+	1    0    0    -1
+$EndComp
+Connection ~ 7450 3700
+Wire Wire Line
+	7450 3700 9250 3700
+$Comp
+L william_fets:PSMN1R0-30YLC,115 Q2
+U 1 1 60186BF3
+P 7350 3900
+F 0 "Q2" H 7556 3991 50  0000 L CNN
+F 1 "PSMN1R0-30YLC,115" H 7556 3900 50  0000 L CNN
+F 2 "Package_TO_SOT_SMD:LFPAK56" H 7200 4100 50  0001 C CNN
+F 3 "https://assets.nexperia.com/documents/data-sheet/PSMN1R0-30YLC.pdf" H 7350 3900 50  0001 C CNN
+F 4 "PSMN1R0-30YLC,115" H 7556 3809 50  0000 L CNN "MPN"
+	1    7350 3900
+	1    0    0    -1
+$EndComp
+$Comp
+L william_fets:PSMN1R0-30YLC,115 Q3
+U 1 1 6018D46B
+P 8550 4200
+F 0 "Q3" H 8756 4291 50  0000 L CNN
+F 1 "PSMN1R0-30YLC,115" H 8756 4200 50  0000 L CNN
+F 2 "Package_TO_SOT_SMD:LFPAK56" H 8400 4400 50  0001 C CNN
+F 3 "https://assets.nexperia.com/documents/data-sheet/PSMN1R0-30YLC.pdf" H 8550 4200 50  0001 C CNN
+F 4 "PSMN1R0-30YLC,115" H 8756 4109 50  0000 L CNN "MPN"
+	1    8550 4200
+	1    0    0    -1
+$EndComp
+Connection ~ 8650 4400
+Wire Wire Line
+	8650 4400 9250 4400
+$Comp
+L william_fets:PSMN1R0-30YLC,115 Q4
+U 1 1 601900A3
+P 8550 4600
+F 0 "Q4" H 8756 4691 50  0000 L CNN
+F 1 "PSMN1R0-30YLC,115" H 8756 4600 50  0000 L CNN
+F 2 "Package_TO_SOT_SMD:LFPAK56" H 8400 4800 50  0001 C CNN
+F 3 "https://assets.nexperia.com/documents/data-sheet/PSMN1R0-30YLC.pdf" H 8550 4600 50  0001 C CNN
+F 4 "PSMN1R0-30YLC,115" H 8756 4509 50  0000 L CNN "MPN"
+	1    8550 4600
+	1    0    0    -1
+$EndComp
+Text HLabel 6250 3250 2    50   Output ~ 0
+~FAULT~
+Wire Wire Line
+	4750 3200 4200 3200
 $EndSCHEMATC

Commit message: display board updates
Parts:
- C4: footprint Capacitor_SMD:C_0603_1608Metric -> Capacitor_SMD:C_0402_1005Metric
Changed lines of the file:
@@
 F 0 "C4" H 3185 1446 50  0000 R CNN
 F 1 "100N" H 3185 1355 50  0000 R CNN
-F 2 "Capacitor_SMD:C_0603_1608Metric" H 3338 1250 50  0001 C CNN
+F 2 "Capacitor_SMD:C_0402_1005Metric" H 3338 1250 50  0001 C CNN
 F 3 "~" H 3300 1400 50  0001 C CNN
 	1    3300 1400

Commit message: new f446RETx, displays, a4957
Parts:
- C3, C6, C8, C9: footprint Capacitor_SMD:C_0603_1608Metric -> Capacitor_SMD:C_0805_2012Metric
- C4: footprint Capacitor_SMD:C_0402_1005Metric -> Capacitor_SMD:C_0603_1608Metric
- U1: footprint Package_DFN_QFN:QFN-24-1EP_4x4mm_P0.5mm_EP2.65x2.65mm_ThermalVias -> william_motor:A4957
Changed lines of the file:
@@
 $Descr A4 11693 8268
 encoding utf-8
-Sheet 2 11
+Sheet 2 12
 Title ""
 Date ""
@@
 $EndDescr
 $Comp
-L william_motor:A4957 U?
-U 1 1 5F6A7B03
-P 5450 3900
-AR Path="/5F6A7B03" Ref="U?"  Part="1"
-AR Path="/5F6A7917/5F6A7B03" Ref="U1"  Part="1"
-F 0 "U1" H 5450 4000 50  0000 C CNN
-F 1 "A4957" H 5450 3900 50  0000 C CNN
-F 2 "Package_DFN_QFN:QFN-24-1EP_4x4mm_P0.5mm_EP2.65x2.65mm_ThermalVias" H 5450 5050 50  0001 C CNN
-F 3 "https://www.allegromicro.com/~/media/Files/Datasheets/A4957-Datasheet.ashx" H 5450 5050 50  0001 C CNN
-	1    5450 3900
-	1    0    0    -1
-$EndComp
-$Comp
 L Device:C C8
 U 1 1 5F6A9316
@@
 F 0 "C8" H 4536 3954 50  0000 R CNN
 F 1 "16V 470N" H 4536 4045 50  0000 R CNN
-F 2 "Capacitor_SMD:C_0603_1608Metric" H 4688 3850 50  0001 C CNN
+F 2 "Capacitor_SMD:C_0805_2012Metric" H 4688 3850 50  0001 C CNN
 F 3 "~" H 4650 4000 50  0001 C CNN
 	1    4650 4000
@@
 F 0 "C3" H 2835 1446 50  0000 R CNN
 F 1 "10U" H 2835 1355 50  0000 R CNN
-F 2 "Capacitor_SMD:C_0603_1608Metric" H 2988 1250 50  0001 C CNN
+F 2 "Capacitor_SMD:C_0805_2012Metric" H 2988 1250 50  0001 C CNN
 F 3 "~" H 2950 1400 50  0001 C CNN
 	1    2950 1400
@@
 F 0 "C6" H 4285 4896 50  0000 R CNN
 F 1 "16V 22U" H 4285 4805 50  0000 R CNN
-F 2 "Capacitor_SMD:C_0603_1608Metric" H 4438 4700 50  0001 C CNN
+F 2 "Capacitor_SMD:C_0805_2012Metric" H 4438 4700 50  0001 C CNN
 F 3 "~" H 4400 4850 50  0001 C CNN
 	1    4400 4850
@@
 F 0 "C4" H 3185 1446 50  0000 R CNN
 F 1 "100N" H 3185 1355 50  0000 R CNN
-F 2 "Capacitor_SMD:C_0402_1005Metric" H 3338 1250 50  0001 C CNN
+F 2 "Capacitor_SMD:C_0603_1608Metric" H 3338 1250 50  0001 C CNN
 F 3 "~" H 3300 1400 50  0001 C CNN
 	1    3300 1400
@@
 F 0 "C9" H 5015 1396 50  0000 L CNN
 F 1 "50V 10U" H 5015 1305 50  0000 L CNN
-F 2 "Capacitor_SMD:C_0603_1608Metric" H 4938 1200 50  0001 C CNN
+F 2 "Capacitor_SMD:C_0805_2012Metric" H 4938 1200 50  0001 C CNN
 F 3 "~" H 4900 1350 50  0001 C CNN
 	1    4900 1350
@@
 Wire Wire Line
 	4750 3200 4200 3200
+$Comp
+L william_motor:A4957 U1
+U 1 1 60DDB714
+P 5450 3900
+F 0 "U1" H 5450 5031 50  0000 C CNN
+F 1 "A4957" H 5450 4940 50  0000 C CNN
+F 2 "william_motor:A4957" H 5450 5050 50  0001 C CNN
+F 3 "https://www.allegromicro.com/~/media/Files/Datasheets/A4957-Datasheet.ashx" H 5450 5050 50  0001 C CNN
+	1    5450 3900
+	1    0    0    -1
+$EndComp
 $EndSCHEMATC
