File: LT1161.kicad_sch (KiCad schematic)
At the start: 16 parts, among them Q6 Q_NMOS_GDSD, Q7 Q_NMOS_GDSD, Q8 Q_NMOS_GDSD, Q9 Q_NMOS_GDSD, U4 LT1161

Commit message: fix LT1161 symbol/sch
Parts:
- removed Q6, Q7, Q8, Q9: Q_NMOS_GDSD, Package_TO_SOT_SMD:TO-252-3_TabPin4, symbol Device:Q_NMOS_GDSD
- added fNT1, fNT2, fNT3, fNT4: NetTie_2, william_fab:NetTie-2_SMD_Pad0.5mm, symbol Device:NetTie_2
- added fQ1, fQ2, fQ4, fQ6: Q_NMOS_GDS, Package_TO_SOT_SMD:TO-252-2, symbol Device:Q_NMOS_GDS
- fC1: renamed from C14; footprint Capacitor_SMD:C_Elec_10x10.2 -> Capacitor_SMD:C_Elec_8x10.2
- renumbered C17 to bC14, C15 to bC15, C16 to bC16, C19 to bC17, C20 to bC18, C18 to bC19, R11 to fR1, R8 to fR2, R9 to fR3, R10 to fR4, U4 to fU4
Connections:
- net OUTPUT 1: now also fQ4.3 (S)
- net OUTPUT 2: now also fQ6.3 (S)
- net OUTPUT 3: now also fQ2.3 (S)
- net OUTPUT 4: now also fQ1.3 (S)
- net at fU4.12 (GATE_4): now also fQ1.1 (G); no longer fR1.2
- net at fU4.13 (SENSE_4): now also fNT1.1
- net at fU4.14 (GATE_3): now also fQ2.1 (G); no longer fR4.2
- net at fU4.15 (SENSE_3): now also fNT2.1
- net at fU4.16 (GATE_2): now also fQ6.1 (G); no longer fR3.2
- net at fU4.17 (SENSE_2): now also fNT4.1
- net at fU4.18 (GATE_1): now also fQ4.1 (G); no longer fR2.2
- net at fU4.19 (SENSE_1): now also fNT3.1
- new net SENSE_1: fNT1.2, fQ1.2 (D), fR1.2
- new net SENSE_2: fNT2.2, fQ2.2 (D), fR4.2
- new net SENSE_3: fNT4.2, fQ6.2 (D), fR3.2
- new net SENSE_4: fNT3.2, fQ4.2 (D), fR2.2
