File: Nfet_PWR_noPD.kicad_sch (KiCad schematic)
At the start: 3 parts, among them Q8 SIRA24DP

Commit message: nfets
Parts:
- removed Q8: SIRA24DP, Package_SO:PowerPAK_SO-8_Single, symbol william_fets:SIRA24DP
- removed R10: 10K, Resistor_SMD:R_0603_1608Metric, symbol Device:R
- removed R11: 1K, Resistor_SMD:R_0603_1608Metric, symbol Device:R
- added Q11: IRF7458TRPBF, william_mosfet:SO-8_3.9x4.9mm_P1.27mm, symbol william_fets:IRF7458TRPBF
- added R50: 1K, Resistor_SMD:R_0603_1608Metric, symbol Device:R
Connections:
- net GND: now also Q11.1 (S), Q11.2 (S), Q11.3 (S)
- net LOAD-: now also Q11.5 (D), Q11.6 (D), Q11.7 (D), Q11.8 (D)
- net SIG: now also R50.2
- new net: Q11.4 (G), R50.1
Changed lines of the file:
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@@
 (kicad_sch (version 20211123) (generator eeschema)
   (paper "A4")
-  (junction (at 138.43 87.63) (diameter 0) (color 0 0 0 0)
-  )
-  (junction (at 138.43 97.79) (diameter 0) (color 0 0 0 0)
-  )
-  (wire (pts (xy 138.43 96.52) (xy 138.43 97.79))
+  (wire (pts (xy 158.75 97.79) (xy 158.75 92.71))
     (stroke (width 0) (type default) (color 0 0 0 0))
   )
-  (wire (pts (xy 133.35 97.79) (xy 138.43 97.79))
+  (wire (pts (xy 158.75 74.93) (xy 158.75 71.12))
     (stroke (width 0) (type default) (color 0 0 0 0))
   )
@@
     (stroke (width 0) (type default) (color 0 0 0 0))
   )
-  (wire (pts (xy 158.75 97.79) (xy 158.75 92.71))
+  (wire (pts (xy 158.75 77.47) (xy 158.75 82.55))
+    (stroke (width 0) (type default) (color 0 0 0 0))
+  )
+  (wire (pts (xy 133.35 97.79) (xy 158.75 97.79))
+    (stroke (width 0) (type default) (color 0 0 0 0))
+  )
+  (wire (pts (xy 133.35 87.63) (xy 142.24 87.63))
+    (stroke (width 0) (type default) (color 0 0 0 0))
+  )
+  (wire (pts (xy 163.83 77.47) (xy 158.75 77.47))
     (stroke (width 0) (type default) (color 0 0 0 0))
   )
@@
     (stroke (width 0) (type default) (color 0 0 0 0))
   )
-  (wire (pts (xy 138.43 97.79) (xy 158.75 97.79))
-    (stroke (width 0) (type default) (color 0 0 0 0))
-  )
-  (wire (pts (xy 138.43 87.63) (xy 142.24 87.63))
-    (stroke (width 0) (type default) (color 0 0 0 0))
-  )
   (wire (pts (xy 158.75 71.12) (xy 157.48 71.12))
     (stroke (width 0) (type default) (color 0 0 0 0))
   )
-  (wire (pts (xy 133.35 87.63) (xy 138.43 87.63))
-    (stroke (width 0) (type default) (color 0 0 0 0))
-  )
-  (wire (pts (xy 158.75 74.93) (xy 158.75 71.12))
-    (stroke (width 0) (type default) (color 0 0 0 0))
-  )
-  (wire (pts (xy 158.75 77.47) (xy 158.75 82.55))
-    (stroke (width 0) (type default) (color 0 0 0 0))
-  )
-  (wire (pts (xy 163.83 77.47) (xy 158.75 77.47))
-    (stroke (width 0) (type default) (color 0 0 0 0))
-  )
-  (wire (pts (xy 138.43 88.9) (xy 138.43 87.63))
-    (stroke (width 0) (type default) (color 0 0 0 0))
+  (hierarchical_label "V_power" (shape input) (at 157.48 71.12 180)
+    (effects (font (size 1.27 1.27)) (justify right))
   )
   (hierarchical_label "LOAD-" (shape input) (at 163.83 77.47 0)
     (effects (font (size 1.27 1.27)) (justify left))
   )
-  (hierarchical_label "GND" (shape input) (at 133.35 97.79 180)
+  (hierarchical_label "SIG" (shape input) (at 133.35 87.63 180)
     (effects (font (size 1.27 1.27)) (justify right))
   )
-  (hierarchical_label "V_power" (shape input) (at 157.48 71.12 180)
-    (effects (font (size 1.27 1.27)) (justify right))
-  )
-  (hierarchical_label "SIG" (shape input) (at 133.35 87.63 180)
+  (hierarchical_label "GND" (shape input) (at 133.35 97.79 180)
     (effects (font (size 1.27 1.27)) (justify right))
   )
@@
     (effects (font (size 1.27 1.27)) (justify left))
   )
+  (symbol (lib_id "william_fets:IRF7458TRPBF") (at 156.21 87.63 0) (unit 1)
+    (in_bom yes) (on_board yes)
+    (property "Reference" "Q11" (id 0) (at 161.4424 86.4616 0)
+      (effects (font (size 1.27 1.27)) (justify left))
+    )
+    (property "Value" "IRF7458TRPBF" (id 1) (at 161.4424 88.773 0)
+      (effects (font (size 1.27 1.27)) (justify left))
+    )
+    (property "Footprint" "william_mosfet:SO-8_3.9x4.9mm_P1.27mm" (id 2) (at 152.4 82.55 0)
+      (effects (font (size 1.27 1.27)) hide)
+    )
+    (property "Datasheet" "https://www.infineon.com/dgdl/irf7458pbf.pdf?fileId=5546d462533600a4015355fecb231bfe" (id 3) (at 156.21 87.63 0)
+      (effects (font (size 1.27 1.27)) hide)
+    )
+    (pin "1")
+    (pin "2")
+    (pin "3")
+    (pin "4")
+    (pin "5")
+    (pin "6")
+    (pin "7")
+    (pin "8")
+  )
   (symbol (lib_id "Device:R") (at 146.05 87.63 270) (unit 1)
     (in_bom yes) (on_board yes)
-    (property "Reference" "R11" (id 0) (at 146.05 82.3722 90))
+    (property "Reference" "R50" (id 0) (at 146.05 82.3722 90))
     (property "Value" "1K" (id 1) (at 146.05 84.6836 90))
     (property "Footprint" "Resistor_SMD:R_0603_1608Metric" (id 2) (at 146.05 85.852 90)
@@
     (pin "2")
   )
-  (symbol (lib_id "Device:R") (at 138.43 92.71 0) (unit 1)
-    (in_bom yes) (on_board yes)
-    (property "Reference" "R10" (id 0) (at 140.208 91.5416 0)
-      (effects (font (size 1.27 1.27)) (justify left))
-    )
-    (property "Value" "10K" (id 1) (at 140.208 93.853 0)
-      (effects (font (size 1.27 1.27)) (justify left))
-    )
-    (property "Footprint" "Resistor_SMD:R_0603_1608Metric" (id 2) (at 136.652 92.71 90)
-      (effects (font (size 1.27 1.27)) hide)
-    )
-    (property "Datasheet" "~" (id 3) (at 138.43 92.71 0)
-      (effects (font (size 1.27 1.27)) hide)
-    )
-    (pin "1")
-    (pin "2")
-  )
-  (symbol (lib_id "william_fets:SIRA24DP") (at 156.21 87.63 0) (unit 1)
-    (in_bom yes) (on_board yes) (fields_autoplaced)
-    (property "Reference" "Q8" (id 0) (at 162.56 86.3599 0)
-      (effects (font (size 1.27 1.27)) (justify left))
-    )
-    (property "Value" "SIRA24DP" (id 1) (at 162.56 88.8999 0)
-      (effects (font (size 1.27 1.27)) (justify left))
-    )
-    (property "Footprint" "Package_SO:PowerPAK_SO-8_Single" (id 2) (at 152.4 82.55 0)
-      (effects (font (size 1.27 1.27)) hide)
-    )
-    (property "Datasheet" "http://aosmd.com/res/data_sheets/AON7524.pdf" (id 3) (at 156.21 87.63 0)
-      (effects (font (size 1.27 1.27)) hide)
-    )
-    (pin "1")
-    (pin "2")
-    (pin "3")
-    (pin "4")
-    (pin "5")
-  )
 )
