File: analog_front_end.kicad_sch (KiCad schematic)
At the start: 12 parts, among them Q1 MS23P05, Q2 MS23N06A, Q3 MS23P05, Q4 MS23N06A

Commit message: loadcell parts
Parts:
- C20, C21: footprint (none) -> Capacitor_SMD:C_0603_1608Metric
- D5: footprint (none) -> Package_TO_SOT_SMD:SOT-23-6
- Q1, Q2, Q3, Q4: footprint (none) -> Package_TO_SOT_SMD:SOT-23
- R8, R9: footprint (none) -> Resistor_SMD:R_0603_1608Metric
Changed lines of the file:
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@@
       (effects (font (size 1.27 1.27)))
     )
-    (property "Footprint" "" (at 45.72 33.528 90)
+    (property "Footprint" "Resistor_SMD:R_0603_1608Metric" (at 45.72 33.528 90)
       (effects (font (size 1.27 1.27)) hide)
     )
@@
       (effects (font (size 1.27 1.27)) (justify left))
     )
-    (property "Footprint" "" (at 106.68 35.56 0)
+    (property "Footprint" "Package_TO_SOT_SMD:SOT-23" (at 106.68 35.56 0)
       (effects (font (size 1.27 1.27)) hide)
     )
@@
       (effects (font (size 1.27 1.27)) (justify left))
     )
-    (property "Footprint" "" (at 158.75 35.56 0)
+    (property "Footprint" "Package_TO_SOT_SMD:SOT-23" (at 158.75 35.56 0)
       (effects (font (size 1.27 1.27)) hide)
     )
@@
       (effects (font (size 1.27 1.27)) (justify left))
     )
-    (property "Footprint" "" (at 122.8852 62.23 0)
+    (property "Footprint" "Capacitor_SMD:C_0603_1608Metric" (at 122.8852 62.23 0)
       (effects (font (size 1.27 1.27)) hide)
     )
@@
       (effects (font (size 1.27 1.27)) (justify left))
     )
-    (property "Footprint" "" (at 178.7652 62.23 0)
+    (property "Footprint" "Capacitor_SMD:C_0603_1608Metric" (at 178.7652 62.23 0)
       (effects (font (size 1.27 1.27)) hide)
     )
@@
       (effects (font (size 1.27 1.27)) (justify left))
     )
-    (property "Footprint" "" (at 54.61 120.65 0)
-      (effects (font (size 1.27 1.27)) hide)
-    )
-    (property "Datasheet" "https://www.ti.com/general/docs/suppproductinfo.tsp?distId=10&gotoUrl=https%3A%2F%2Fwww.ti.com%2Flit%2Fgpn%2Ftpd4e1u06" (at 63.5 111.76 0)
+    (property "Footprint" "Package_TO_SOT_SMD:SOT-23-6" (at 54.61 120.65 0)
+      (effects (font (size 1.27 1.27)) hide)
+    )
+    (property "Datasheet" "https://www.ti.com/lit/ds/symlink/tpd4e1u06.pdf" (at 63.5 111.76 0)
       (effects (font (size 1.27 1.27)) hide)
     )
@@
       (effects (font (size 1.27 1.27)) (justify left))
     )
-    (property "Footprint" "" (at 158.75 54.61 0)
+    (property "Footprint" "Package_TO_SOT_SMD:SOT-23" (at 158.75 54.61 0)
       (effects (font (size 1.27 1.27)) hide)
     )
@@
       (effects (font (size 1.27 1.27)))
     )
-    (property "Footprint" "" (at 45.72 52.832 90)
+    (property "Footprint" "Resistor_SMD:R_0603_1608Metric" (at 45.72 52.832 90)
       (effects (font (size 1.27 1.27)) hide)
     )
@@
       (effects (font (size 1.27 1.27)) (justify left))
     )
-    (property "Footprint" "" (at 106.68 54.61 0)
-      (effects (font (size 1.27 1.27)) hide)
-    )
+    (property "Footprint" "Package_TO_SOT_SMD:SOT-23" (at 106.68 54.61 0)
+      (effects (font (size 1.27 1.27)) hide)
+    )

Commit message: force frontend
Connections:
- net SIG+_{EXTERNAL}: now also D5.6 (NC); no longer D5.4 (D2+)
- net VEXC+_{EXTERNAL}: now also C21.1, Q3.2 (S), Q4.3 (D); no longer C20.1, Q1.2 (S), Q2.3 (D)
- net VEXC-_{EXTERNAL}: now also C20.1, D5.4 (D2+), Q1.2 (S), Q2.3 (D); no longer C21.1, D5.6 (NC), Q3.2 (S), Q4.3 (D)
- net VLOW: now reaches C20.2, C21.2, C24.1, C25.2, Q2.2 (S), Q4.2 (S), R9.1
Changed lines of the file:
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@@
     (effects (font (size 1.27 1.27)) (justify left bottom))
   )
-  (label "EXC_{B}" (at 177.8 46.99 0) (fields_autoplaced)
+  (label "EXC_{B}" (at 121.92 45.72 0) (fields_autoplaced)
     (effects (font (size 1.27 1.27)) (justify left bottom))
   )
@@
     (effects (font (size 1.27 1.27)) (justify left bottom))
   )
-  (label "EXC_{A}" (at 121.92 45.72 0) (fields_autoplaced)
+  (label "EXC_{A}" (at 177.8 46.99 0) (fields_autoplaced)
     (effects (font (size 1.27 1.27)) (justify left bottom))
   )
   (label "VCCA" (at 139.7 92.71 0) (fields_autoplaced)
+    (effects (font (size 1.27 1.27)) (justify left bottom))
+  )
+  (label "VLOW" (at 78.74 67.31 0) (fields_autoplaced)
     (effects (font (size 1.27 1.27)) (justify left bottom))
   )
@@
     (effects (font (size 1.27 1.27)) (justify right))
   )
-  (hierarchical_label "VEXC-_{EXTERNAL}" (shape input) (at 44.45 102.87 180) (fields_autoplaced)
+  (hierarchical_label "VEXC-_{EXTERNAL}" (shape input) (at 44.45 106.68 180) (fields_autoplaced)
     (effects (font (size 1.27 1.27)) (justify right))
   )
-  (hierarchical_label "SIG+_{EXTERNAL}" (shape input) (at 44.45 106.68 180) (fields_autoplaced)
+  (hierarchical_label "SIG+_{EXTERNAL}" (shape input) (at 44.45 102.87 180) (fields_autoplaced)
     (effects (font (size 1.27 1.27)) (justify right))
   )
