File: can.kicad_sch (KiCad schematic)
At the start: 10 parts, among them U2 TCAN1044V

Commit message: force frontend
Parts:
- U2: value TCAN1044V -> TCAN1044VDDFR
Changed lines of the file:
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@@
       (effects (font (size 1.27 1.27)) (justify left))
     )
-    (property "Value" "TCAN1044V" (at 130.81 109.22 90)
+    (property "Value" "TCAN1044VDDFR" (at 133.35 111.76 90)
       (effects (font (size 1.27 1.27)) (justify left))
     )
